Commit message: pnp

File: robotican_armadillo/description/models/armadillo_arm.xacro (robot description, xacro)
@@ -444,7 +444,8 @@
     <limit
       effort="3.1"
-      lower="-0.4"
-      upper="1.0"
+      lower="-1.57"
+      upper="1.57"
       velocity="7.016223585" />
+      <dynamics friction ="1000" damping="100"/>
   </joint>
   <link
@@ -502,7 +503,8 @@
     <limit
       effort="3.1"
-      lower="-1.0"
-      upper="0.4"
+      lower="-1.57"
+      upper="1.57"
       velocity="7.016223585" />
+      <dynamics friction ="1000" damping="100"/>
   </joint>
   <link

File: robotican_armadillo/description/models/armadillo_base.xacro (robot description, xacro)
@@ -15,5 +15,5 @@
         rpy="0 0 0" />
       <mass
-        value="100.6548" />
+        value="30.6548" />
       <inertia
         ixx="0.61639"

File: robotican_armadillo/description/models/armadillo_gazebo.xacro (robot description, xacro)
@@ -560,7 +560,28 @@
     </gazebo>
   </xacro:if>
+ <gazebo reference="left_wheel_link">
+    <!-- kp and kd for rubber -->
+    <kp>1000000.0</kp>
+    <kd>100.0</kd>
+    <mu1>1.5</mu1>
+    <mu2>1.5</mu2>
+    <fdir1>1 0 0</fdir1>
+    <maxVel>1.0</maxVel>
+    <minDepth>0.00</minDepth>
+  </gazebo>
+   <gazebo reference="right_wheel_link">
+    <!-- kp and kd for rubber -->
+    <kp>1000000.0</kp>
+    <kd>100.0</kd>
+    <mu1>1.5</mu1>
+    <mu2>1.5</mu2>
+    <fdir1>1 0 0</fdir1>
+    <maxVel>1.0</maxVel>
+    <minDepth>0.00</minDepth>
+  </gazebo>
+<!--
   <gazebo reference="left_wheel_link">
-    <mu1>1.0</mu1>
-    <mu2>1.0</mu2>
+    <mu1>10.0</mu1>
+    <mu2>10.0</mu2>
     <kp>1000000.0</kp>
     <kd>100.0</kd>
@@ -568,7 +589,7 @@
     <maxVel>1.0</maxVel>
   </gazebo>
-  <gazebo reference="right_wheel_link">
-    <mu1>1.0</mu1>
-    <mu2>1.0</mu2>
+    <gazebo reference="right_wheel_link">
+    <mu1>10.0</mu1>
+    <mu2>10.0</mu2>
     <kp>1000000.0</kp>
     <kd>100.0</kd>
@@ -576,4 +597,5 @@
     <maxVel>1.0</maxVel>
   </gazebo>
+  -->
   <!--
   <gazebo reference="base_link">
@@ -640,4 +662,7 @@
     <material>Gazebo/Grey</material>
   </gazebo>
+    <gazebo reference="right_finger_link">
+    <material>Gazebo/Grey</material>
+  </gazebo>
   <gazebo reference="base_arm_link">
     <material>Gazebo/Grey</material>

Commit message: fixes

File: robotican_armadillo/description/models/armadillo_arm.xacro (robot description, xacro)
@@ -390,4 +390,10 @@
       velocity="3.455751915" />
   </joint>
+   <link name="gripper_link"/>
+<joint name="gripper_joint" type="fixed">
+    <origin xyz="0 0 0.06" rpy="0 ${-M_PI/2} 0"/>
+    <parent link="wrist_link"/>
+    <child link="gripper_link"/>
+ </joint>
   <link
     name="left_finger_link">

Commit message: calibrations

File: robotican_armadillo/description/models/armadillo_arm.xacro (robot description, xacro)
@@ -515,5 +515,5 @@
   </joint>
   <link
-    name="f200_link">
+    name="sr300_link">
     <inertial>
       <origin
@@ -536,5 +536,5 @@
       <geometry>
         <mesh
-          filename="package://robotican_armadillo/description/meshes/f200_optical_link.STL" />
+          filename="package://robotican_armadillo/description/meshes/sr300_optical_link.STL" />
       </geometry>
       <material
@@ -549,10 +549,10 @@
         rpy="0 0 0" />
       <geometry>
-        <mesh filename="package://robotican_armadillo/description/meshes/f200_optical_link.STL" />
-      </geometry>
-    </collision>
-  </link>
-  <joint
-    name="f200_joint"
+        <mesh filename="package://robotican_armadillo/description/meshes/sr300_optical_link.STL" />
+      </geometry>
+    </collision>
+  </link>
+  <joint
+    name="sr300_joint"
     type="fixed">
     <origin
@@ -562,31 +562,31 @@
       link="wrist_link" />
     <child
-      link="f200_link" />
+      link="sr300_link" />
     <axis
       xyz="0 0 0" />
   </joint>
-  		<link name="f200_rgb_frame" />
-		<joint name="f200_rgb_joint" type="fixed">
+  		<link name="sr300_rgb_frame" />
+		<joint name="sr300_rgb_joint" type="fixed">
 		  <origin xyz="0 0 0" rpy="0 0 0" />
-		  <parent link="f200_link" />
-		  <child link="f200_rgb_frame" />
+		  <parent link="sr300_link" />
+		  <child link="sr300_rgb_frame" />
 		</joint>
-		 <link name="f200_rgb_optical_frame" />
-		<joint name="f200_rgb_optical_joint" type="fixed">
+		 <link name="sr300_rgb_optical_frame" />
+		<joint name="sr300_rgb_optical_joint" type="fixed">
 		  <origin xyz="0 0 0" rpy="${-M_PI/2} 0 ${-M_PI/2}" />
-		  <parent link="f200_rgb_frame" />
-		  <child link="f200_rgb_optical_frame" />
+		  <parent link="sr300_rgb_frame" />
+		  <child link="sr300_rgb_optical_frame" />
 		</joint>
-		<link name="f200_depth_frame" />
-		<joint name="f200_depth_joint" type="fixed">
+		<link name="sr300_depth_frame" />
+		<joint name="sr300_depth_joint" type="fixed">
 		  <origin xyz="0 -0.0235 0" rpy="0 0 0" />
-		  <parent link="f200_link" />
-		  <child link="f200_depth_frame" />
+		  <parent link="sr300_link" />
+		  <child link="sr300_depth_frame" />
 		</joint>
-		<link name="f200_depth_optical_frame" />
-		<joint name="f200_depth_optical_joint" type="fixed">
+		<link name="sr300_depth_optical_frame" />
+		<joint name="sr300_depth_optical_joint" type="fixed">
 		  <origin xyz="0 0 0" rpy="${-M_PI/2} 0 ${-M_PI/2}" />
-		  <parent link="f200_depth_frame" />
-		  <child link="f200_depth_optical_frame" />
+		  <parent link="sr300_depth_frame" />
+		  <child link="sr300_depth_optical_frame" />
 		</joint>
 </robot>

File: robotican_armadillo/description/models/armadillo_gazebo.xacro (robot description, xacro)
@@ -15,6 +15,6 @@
   <xacro:arg name="gps" default="false"/>
   <xacro:arg name="lidar" default="false"/>
-  <xacro:arg name="f200" default="false"/>
-  <xacro:arg name="f200_hz" default="10.0"/>
+  <xacro:arg name="sr300" default="false"/>
+  <xacro:arg name="sr300_hz" default="10.0"/>
   <gazebo>
     <gripper name="gripper">
@@ -63,9 +63,9 @@
   <axis xyz="0 0 0" />
   </joint>-->
-  <xacro:if value="$(arg f200)">
-    <gazebo reference="f200_rgb_frame">
-      <sensor type="depth" name="f200">
+  <xacro:if value="$(arg sr300)">
+    <gazebo reference="sr300_rgb_frame">
+      <sensor type="depth" name="sr300">
 	<always_on>true</always_on>
-	<update_rate>$(arg f200_hz)</update_rate>
+	<update_rate>$(arg sr300_hz)</update_rate>
 	<camera>
 	  <horizontal_fov>1.20772254</horizontal_fov>
@@ -80,9 +80,9 @@
 	  </clip>
 	</camera>
-	<plugin name="f200_camera_controller" filename="libgazebo_ros_openni_kinect.so">
+	<plugin name="sr300_camera_controller" filename="libgazebo_ros_openni_kinect.so">
 	  <alwaysOn>true</alwaysOn>
 	  <!--  <baseline>0.11</baseline> -->
-	  <updateRate>$(arg f200_hz)</updateRate>
-	  <cameraName>f200</cameraName>
+	  <updateRate>$(arg sr300_hz)</updateRate>
+	  <cameraName>sr300</cameraName>
 	  <imageTopicName>color/image_raw</imageTopicName>
 	  <cameraInfoTopicName>color/camera_info</cameraInfoTopicName>
@@ -90,5 +90,5 @@
 	  <depthImageCameraInfoTopicName>depth/camera_info</depthImageCameraInfoTopicName>
 	  <pointCloudTopicName>depth/points</pointCloudTopicName>
-	  <frameName>f200_depth_optical_frame</frameName>
+	  <frameName>sr300_depth_optical_frame</frameName>
 	  <pointCloudCutoff>0.2</pointCloudCutoff>
 	  <pointCloudCutoffMax>1.2</pointCloudCutoffMax>
@@ -626,5 +626,5 @@
     <material>Gazebo/Black</material>
   </gazebo>
-  <gazebo reference="f200_link">
+  <gazebo reference="sr300_link">
     <material>Gazebo/Black</material>
   </gazebo>
