Commit message: update;

File: robotican_armadillo/description/models/armadillo.xacro (robot description, xacro)
@@ -18,5 +18,5 @@
 		<axis xyz="0 0 1" />
 		<dynamics damping="1000.0" friction="100000.0"/>
-		<limit effort="1.765196" velocity="0.1" lower="0.0125" upper="0.4" />
+		<limit effort="1.765196" velocity="0.1" lower="0.0125" upper="0.35" />
 	</joint>
 	<joint name="base_arm_joint" type="fixed">

File: robotican_armadillo/description/models/armadillo_torso.xacro (robot description, xacro)
@@ -254,6 +254,6 @@
       xyz="0 0 1" />
     <limit
-      upper="${M_PI/2}"
-	  lower="${-M_PI/2}"
+      upper="${M_PI/4}"
+	  lower="${-M_PI/4}"
       effort="1.11"
       velocity="5.3" />

Commit message: hi

File: robotican_armadillo/description/models/armadillo.xacro (robot description, xacro)
@@ -13,10 +13,10 @@
 	<!--    LOAD JOINTS    -->
 	<joint name="torso_joint" type="prismatic">
-		<origin xyz="-0.1403 0 0.49381" rpy="0 0 0" />
+		<origin xyz="-0.1403 0 0.51381" rpy="0 0 0" />
 		<parent link="base_link" />
 		<child link="torso_link" />
 		<axis xyz="0 0 1" />
 		<dynamics damping="1000.0" friction="100000.0"/>
-		<limit effort="1.765196" velocity="0.1" lower="0.0125" upper="0.35" />
+		<limit effort="1.765196" velocity="0.1" lower="0.1" upper="0.35" />
 	</joint>
 	<joint name="base_arm_joint" type="fixed">

Commit message: update

File: robotican_armadillo/description/models/armadillo.xacro (robot description, xacro)
@@ -18,5 +18,5 @@
 		<axis xyz="0 0 1" />
 		<dynamics damping="1000.0" friction="100000.0"/>
-		<limit effort="1.765196" velocity="0.1" lower="0.1" upper="0.35" />
+		<limit effort="1.765196" velocity="0.1" lower="0.00" upper="0.32" />
 	</joint>
 	<joint name="base_arm_joint" type="fixed">

Commit message: change offset torso armadillo

File: robotican_armadillo/description/models/armadillo.xacro (robot description, xacro)
@@ -13,5 +13,5 @@
 	<!--    LOAD JOINTS    -->
 	<joint name="torso_joint" type="prismatic">
-		<origin xyz="-0.1403 0 0.51381" rpy="0 0 0" />
+		<origin xyz="-0.1403 0 0.54381" rpy="0 0 0" />
 		<parent link="base_link" />
 		<child link="torso_link" />

Commit message: calibrations

File: robotican_armadillo/description/models/armadillo.xacro (robot description, xacro)
@@ -13,5 +13,5 @@
 	<!--    LOAD JOINTS    -->
 	<joint name="torso_joint" type="prismatic">
-		<origin xyz="-0.1403 0 0.54381" rpy="0 0 0" />
+		<origin xyz="-0.1403 0 0.49381" rpy="0 0 0" />
 		<parent link="base_link" />
 		<child link="torso_link" />

File: robotican_armadillo/description/models/armadillo_base.xacro (robot description, xacro)
@@ -6,5 +6,5 @@
     <parent link="base_footprint"/>
     <child link="base_link"/>
-    <origin xyz="0.00 0.00 0.1" rpy="0.0 0.0 0.0"/>
+    <origin xyz="0.00 0.00 0.095" rpy="0.0 0.0 0.0"/>
   </joint>
   <link
@@ -40,8 +40,8 @@
       <collision name='caster_collision'>
       <origin
-        xyz="-0.30 0 -0.05"
+        xyz="-0.30 0 -0.0475"
         rpy="0 0 0" />
             <geometry>
-              <sphere radius="0.05"/>
+              <sphere radius="0.0475"/>
             </geometry>
             <surface>
@@ -58,8 +58,8 @@
 	<!--  <visual name='caster_visual'>
 	 <origin
-        xyz="-0.30 0 -0.05"
+        xyz="-0.30 0 -0.0475"
         rpy="0 0 0" />
             <geometry>
-	    <sphere radius="0.05"/>
+	    <sphere radius="0.0475"/>
             </geometry>
 	  </visual> -->
@@ -299,5 +299,5 @@
       <geometry>
     <!--  <mesh filename="package://robotican_armadillo/description/meshes/left_wheel_link.STL" /> -->
-                 <cylinder  length="0.05" radius="0.1"/>
+                 <cylinder  length="0.05" radius="0.095"/>
       </geometry>
       <material
@@ -313,5 +313,5 @@
       <geometry>
     <!--  <mesh filename="package://robotican_armadillo/description/meshes/left_wheel_link.STL" /> -->
-                 <cylinder  length="0.05" radius="0.1"/>
+                 <cylinder  length="0.05" radius="0.095"/>
       </geometry>
     </collision>
@@ -352,5 +352,5 @@
       <geometry>
     <!--  <mesh filename="package://robotican_armadillo/description/meshes/right_wheel_link.STL" /> -->
-      <cylinder  length="0.05" radius="0.1"/>
+      <cylinder  length="0.05" radius="0.095"/>
       </geometry>
       <material
@@ -366,5 +366,5 @@
       <geometry>
      <!--  <mesh filename="package://robotican_armadillo/description/meshes/right_wheel_link.STL" /> -->
-      <cylinder  length="0.05" radius="0.1"/>
+      <cylinder  length="0.05" radius="0.095"/>
       </geometry>
     </collision>

Commit message: komodo, ikfast, manipulator_h

File: robotican_armadillo/description/models/armadillo.xacro (robot description, xacro)
@@ -1,13 +1,13 @@
 <?xml version="1.0"?>
-	<robot xmlns:xacro="http://www.ros.org/wiki/xacro" name="armadillo_with_arm" description="Armadillo robot">
+	<robot xmlns:xacro="http://www.ros.org/wiki/xacro" name="armadillo_robot" description="ARMadillo Robot">
 	<xacro:property name="M_PI" value="3.1415926535897931" />
-	<!--    BASE ROBOT     -->
+	<!--    BASE      -->
 	<xacro:include filename="$(find robotican_armadillo)/description/models/armadillo_base.xacro" />
 	<!--      END          -->
-	<!--    ELEV ROBOT     -->
+	<!--   TORSO     -->
 	<xacro:include filename="$(find robotican_armadillo)/description/models/armadillo_torso.xacro" />
 	<!--      END          -->
-	<!--    ELEV ROBOT     -->
-	<xacro:include filename="$(find robotican_armadillo)/description/models/armadillo_arm.xacro" />
+	<!--    ARM     -->
+	<xacro:include filename="$(find robotican_manipulator_h)/models/manipulator_h.xacro" />
 	<!--      END          -->
 	<!--    LOAD JOINTS    -->

File: robotican_komodo/description/models/komodo_base.xacro (robot description, xacro)
@@ -76,5 +76,5 @@
       <origin
         xyz="0 0 0"
-        rpy="0 0 0" />
+        rpy="0 0 1.57" />
       <geometry>
         <mesh
@@ -129,5 +129,5 @@
       <origin
         xyz="0 0 0"
-        rpy="0 0 0" />
+        rpy="0 0 1.57" />
       <geometry>
         <mesh
@@ -182,5 +182,5 @@
       <origin
         xyz="0 0 0"
-        rpy="0 0 0" />
+        rpy="0 0 1.57" />
       <geometry>
         <mesh
@@ -235,5 +235,5 @@
       <origin
         xyz="0 0 0"
-        rpy="0 0 0" />
+        rpy="0 0 1.57" />
       <geometry>
         <mesh
@@ -602,56 +602,3 @@
       xyz="0 0 0" />
   </joint>
-  <link
-    name="arm_link">
-    <inertial>
-      <origin
-        xyz="-0.022197 -1.9122E-07 0.044251"
-        rpy="0 0 0" />
-      <mass
-        value="1.3188" />
-      <inertia
-        ixx="0.0049508"
-        ixy="-6.559E-09"
-        ixz="-0.0011709"
-        iyy="0.0084361"
-        iyz="1.3268E-08"
-        izz="0.010567" />
-    </inertial>
-    <visual>
-      <origin
-        xyz="0 0 0"
-        rpy="0 0 0" />
-      <geometry>
-        <mesh
-          filename="package://robotican_komodo/description/meshes/arm_link.STL" />
-      </geometry>
-      <material
-        name="">
-        <color
-          rgba="0.27843 0.2902 0.31765 1" />
-      </material>
-    </visual>
-    <collision>
-      <origin
-        xyz="0 0 0"
-        rpy="0 0 0" />
-      <geometry>
-        <mesh
-          filename="package://robotican_komodo/description/meshes/arm_link.STL" />
-      </geometry>
-    </collision>
-  </link>
-  <joint
-    name="arm_joint"
-    type="fixed">
-    <origin
-      xyz="-0.11925 0 0.16716"
-      rpy="9.68E-16 -2.5959E-15 -1.3587E-14" />
-    <parent
-      link="base_link" />
-    <child
-      link="arm_link" />
-    <axis
-      xyz="0 0 0" />
-  </joint>
 </robot>
