Commit message: speed up

File: robotican_armadillo/description/models/armadillo_base.xacro (robot description, xacro)
@@ -2,4 +2,10 @@
 <robot
   name="armadillo_base_urdf" description="Armadillo robot base">
+    <link name="base_footprint"/>
+ <joint name="base_footprint_joint" type="fixed">
+    <parent link="base_footprint"/>
+    <child link="base_link"/>
+    <origin xyz="0.00 0.00 0.1" rpy="0.0 0.0 0.0"/>
+  </joint>
   <link
     name="base_link">
@@ -34,8 +40,8 @@
       <collision name='caster_collision'>
       <origin
-        xyz="-0.35 0 0"
+        xyz="-0.30 0 -0.05"
         rpy="0 0 0" />
             <geometry>
-              <sphere radius="0.1"/>
+              <sphere radius="0.05"/>
             </geometry>
             <surface>
@@ -52,17 +58,11 @@
 	<!--  <visual name='caster_visual'>
 	 <origin
-        xyz="-0.35 0 0"
+        xyz="-0.30 0 -0.05"
         rpy="0 0 0" />
             <geometry>
-	    <sphere radius="0.1"/>
+	    <sphere radius="0.05"/>
             </geometry>
 	  </visual> -->
   </link>
-  <link name="base_footprint"/>
- <joint name="base_link_to_base_footprint" type="fixed">
-    <parent link="base_link"/>
-    <child link="base_footprint"/>
-    <origin xyz="0.00 0.00 -0.1" rpy="0.0 0.0 0.0"/>
-  </joint>
   <link
     name="front_cam_link">

File: robotican_armadillo/description/models/armadillo_gazebo.xacro (robot description, xacro)
@@ -107,10 +107,10 @@
   <!-- kinect 2 -->
   <xacro:if value="$(arg kinect2)">
-     <xacro:property name="kinect2_hz" value="$(arg kinect2_hz)"/>
+    <xacro:property name="kinect2_hz" value="$(arg kinect2_hz)"/>
     <xacro:property name="kinect2_hd" value="$(arg kinect2_hd)"/>
-     <xacro:property name="kinect2_qhd" value="$(arg kinect2_qhd)"/>
-      <xacro:property name="kinect2_sd" value="$(arg kinect2_sd)"/>
-        -->
-	  <xacro:include filename="$(find robotican_common)/gazebo/kinect2.xacro" />
+    <xacro:property name="kinect2_qhd" value="$(arg kinect2_qhd)"/>
+    <xacro:property name="kinect2_sd" value="$(arg kinect2_sd)"/>
+    -->
+    <xacro:include filename="$(find robotican_common)/gazebo/kinect2.xacro" />
   </xacro:if>
   <!-- Sonars -->
@@ -576,12 +576,14 @@
     <maxVel>1.0</maxVel>
   </gazebo>
+  <!--
   <gazebo reference="base_link">
-    <mu1>1.0</mu1>
-    <mu2>1.0</mu2>
-    <kp>1000000.0</kp>
-    <kd>100.0</kd>
-    <minDepth>0.001</minDepth>
-    <maxVel>1.0</maxVel>
-  </gazebo>
+  <mu1>1.0</mu1>
+  <mu2>1.0</mu2>
+  <kp>1000000.0</kp>
+  <kd>100.0</kd>
+  <minDepth>0.000</minDepth>
+  <maxVel>1.0</maxVel>
+  </gazebo>
+  -->
   <gazebo reference="base_link">
     <material>Gazebo/Grey</material>
@@ -603,5 +605,41 @@
   </gazebo>
   <gazebo reference="f200_link">
+    <material>Gazebo/Black</material>
+  </gazebo>
+  <gazebo reference="front_cam_link">
+    <material>Gazebo/Black</material>
+  </gazebo>
+  <gazebo reference="rear_cam_link">
+    <material>Gazebo/Black</material>
+  </gazebo>
+  <gazebo reference="arm_link">
+    <material>Gazebo/DarkGrey</material>
+  </gazebo>
+  <gazebo reference="base_arm_link">
+    <material>Gazebo/DarkGrey</material>
+  </gazebo>
+  <gazebo reference="rotation1_link">
+    <material>Gazebo/DarkGrey</material>
+  </gazebo>
+    <gazebo reference="rotation2_link">
+    <material>Gazebo/DarkGrey</material>
+  </gazebo>
+  <gazebo reference="shoulder1_link">
+    <material>Gazebo/DarkGrey</material>
+  </gazebo>
+  <gazebo reference="shoulder2_link">
+    <material>Gazebo/DarkGrey</material>
+  </gazebo>
+  <gazebo reference="shoulder3_link">
+    <material>Gazebo/DarkGrey</material>
+  </gazebo>
+  <gazebo reference="wrist_link">
+    <material>Gazebo/DarkGrey</material>
+  </gazebo>
+  <gazebo reference="left_finger_link">
     <material>Gazebo/Grey</material>
   </gazebo>
+  <gazebo reference="base_arm_link">
+    <material>Gazebo/Grey</material>
+  </gazebo>
 </robot>

File: robotican_armadillo/description/models/armadillo_torso.xacro (robot description, xacro)
@@ -9,5 +9,5 @@
         rpy="0 0 0" />
       <mass
-        value="3.5511" />
+        value="0.035511" />
       <inertia
         ixx="0.19579"
@@ -49,5 +49,5 @@
         rpy="0 0 0" />
       <mass
-        value="0.01942" />
+        value="0.001942" />
       <inertia
         ixx="3.9185E-06"
@@ -102,5 +102,5 @@
         rpy="0 0 0" />
       <mass
-        value="0.51572" />
+        value="0.0051572" />
       <inertia
         ixx="0.0028549"

Commit message: komodo gazebo

File: robotican_armadillo/description/models/armadillo_base.xacro (robot description, xacro)
@@ -1,5 +1,5 @@
 <?xml version="1.0"?>
 <robot
-  name="armadillo_base_urdf" description="Armadillo robot base">
+  name="armadillo_base" description="ARMadillo robot base">
     <link name="base_footprint"/>
  <joint name="base_footprint_joint" type="fixed">

File: robotican_komodo/description/models/komodo_base.xacro (robot description, xacro)
@@ -1,5 +1,11 @@
 <?xml version="1.0"?>
 <robot
-  name="robotican_komodo">
+  name="robotican_komodo" description="Komodo robot base>">
+      <link name="base_footprint"/>
+ <joint name="base_footprint_joint" type="fixed">
+    <parent link="base_footprint"/>
+    <child link="base_link"/>
+    <origin xyz="0.00 0.00 0.1275" rpy="0.0 0.0 0.0"/>
+  </joint>
   <link
     name="base_link">
@@ -9,5 +15,5 @@
         rpy="0 0 0" />
       <mass
-        value="2.0058" />
+        value="20.0058" />
       <inertia
         ixx="0.025582"
@@ -43,19 +49,4 @@
   </link>
   <link
-    name="base_footprint" />
-  <joint
-    name="footprint_joint"
-    type="fixed">
-    <origin
-      xyz="0 0 -0.1275"
-      rpy="0 0 0" />
-    <parent
-      link="base_link" />
-    <child
-      link="base_footprint" />
-    <axis
-      xyz="0 0 0" />
-  </joint>
-  <link
     name="RL_wheel_link">
     <inertial>

Commit message: gazebo fixes

File: robotican_armadillo/description/models/armadillo_base.xacro (robot description, xacro)
@@ -192,5 +192,4 @@
         rpy="0 ${M_PI/2} 0" />
       <geometry>
-  <!--      <mesh filename="package://robotican_armadillo/description/meshes/right_urf_link.STL" /> -->
 	<cylinder  length="0.005" radius="0.008"/>
       </geometry>
@@ -206,5 +205,4 @@
          rpy="0 ${M_PI/2} 0" />
       <geometry>
-  <!--      <mesh filename="package://robotican_armadillo/description/meshes/right_urf_link.STL" /> -->
 	<cylinder  length="0.005" radius="0.008"/>
       </geometry>

File: robotican_komodo/description/models/komodo.xacro (robot description, xacro)
@@ -10,5 +10,7 @@
  <link
     name="arm_link">
-    <inertial>
+    <inertial>  <gazebo reference="base_arm_link">
+    <material>Gazebo/Grey</material>
+  </gazebo>
       <origin
         xyz="-0.022197 -1.9122E-07 0.044251"

File: robotican_komodo/description/models/komodo_base.xacro (robot description, xacro)
@@ -264,5 +264,5 @@
     <visual>
       <origin
-        xyz="-0.22 0.0 -0.165"
+        xyz="0 0 0.02291"
         rpy="0 0 0" />
       <material
@@ -284,5 +284,5 @@
     type="fixed">
     <origin
-      xyz="0.2205 0 0.16233"
+      xyz="0.2205 0 0.145"
       rpy="0 0 0" />
     <parent

File: robotican_komodo/description/models/komodo_gazebo.xacro (robot description, xacro)
@@ -10,43 +10,6 @@
   <xacro:arg name="lidar" default="false"/>
   <xacro:arg name="sr300" default="false"/>
-  <gazebo>
-    <gripper name="gripper">
-      <grasp_check>
-	<attach_steps>1</attach_steps>
-	<detach_steps>2</detach_steps>
-	<min_contact_count>2</min_contact_count>
-      </grasp_check>
-      <gripper_link>left_finger_link</gripper_link>
-      <gripper_link>right_finger_link</gripper_link>
-      <palm_link>wrist_link</palm_link>
-    </gripper>
-  </gazebo>
-  <gazebo reference="left_finger_link">
-    <kp>1000000.0</kp>
-    <kd>100.0</kd>
-    <mu1>1.0</mu1>
-    <mu2>1.0</mu2>
-    <fdir1>0 0 1</fdir1>
-    <maxVel>1.0</maxVel>
-    <minDepth>0.00</minDepth>
-  </gazebo>
-  <gazebo reference="left_finger_joint">
-    <implicitSpringDamper>1</implicitSpringDamper>
-    <provideFeedback>1</provideFeedback>
-  </gazebo>
-  <gazebo reference="right_finger_link">
-    <kp>1000000.0</kp>
-    <kd>100.0</kd>
-    <mu1>1.0</mu1>
-    <mu2>1.0</mu2>
-    <fdir1>0 0 1</fdir1>
-    <maxVel>1.0</maxVel>
-    <minDepth>0.00</minDepth>
-  </gazebo>
-  <gazebo reference="right_finger_joint">
-    <implicitSpringDamper>1</implicitSpringDamper>
-    <provideFeedback>1</provideFeedback>
-  </gazebo>
-  <!-- SR300 -->
+  <xacro:include filename="$(find robotican_manipulator_h)/models/manipulator_h_gazebo_plugins.xacro" />
+  	    <!-- SR300 -->
   <xacro:if value="$(arg sr300)">
     <xacro:include filename="$(find robotican_common)/gazebo/sr300.xacro" />
@@ -60,8 +23,8 @@
     <xacro:urf name="rear" link="rear_urf_link" topic="URF/rear" />
   </xacro:if>
-  <!-- hokuyo URG-04LX-UG01   -->
+  <!-- hokuyo URG-30LX   -->
   <xacro:if value="$(arg lidar)">
     <xacro:include filename="$(find robotican_common)/gazebo/hokuyo.xacro" />
-    <xacro:lidar link="laser_link" topic="scan" samples="667" resolution="1" min_angle="-1.81" max_angle="1.81" range_min="0.02" range_max="5.6" range_resolution="0.01" />
+    <xacro:lidar link="laser_link" topic="scan" samples="720" resolution="1" min_angle="-1.5707" max_angle="1.5707" range_min="0.1" range_max="30.0" range_resolution="0.01" />
   </xacro:if>
   <!-- GPS   -->
@@ -128,76 +91,4 @@
       </actuator>
     </transmission>
-    <transmission name="rotation1_joint_trans">
-      <type>transmission_interface/SimpleTransmission</type>
-      <joint name="rotation1_joint">
-	<hardwareInterface>PosVelJointInterface</hardwareInterface>
-      </joint>
-      <actuator name="rotation1_joint_motor">
-	<mechanicalReduction>1</mechanicalReduction>
-      </actuator>
-    </transmission>
-    <transmission name="shoulder1_joint_trans">
-      <type>transmission_interface/SimpleTransmission</type>
-      <joint name="shoulder1_joint">
-	<hardwareInterface>PosVelJointInterface</hardwareInterface>
-      </joint>
-      <actuator name="shoulder1_joint_motor">
-	<mechanicalReduction>1</mechanicalReduction>
-      </actuator>
-    </transmission>
-    <transmission name="shoulder2_joint_trans">
-      <type>transmission_interface/SimpleTransmission</type>
-      <joint name="shoulder2_joint">
-	<hardwareInterface>PosVelJointInterface</hardwareInterface>
-      </joint>
-      <actuator name="shoulder2_joint_motor">
-	<mechanicalReduction>1</mechanicalReduction>
-      </actuator>
-    </transmission>
-    <transmission name="rotation2_joint_trans">
-      <type>transmission_interface/SimpleTransmission</type>
-      <joint name="rotation2_joint">
-	<hardwareInterface>PosVelJointInterface</hardwareInterface>
-      </joint>
-      <actuator name="rotation2_joint_motor">
-	<mechanicalReduction>1</mechanicalReduction>
-      </actuator>
-    </transmission>
-    <transmission name="shoulder3_joint_trans">
-      <type>transmission_interface/SimpleTransmission</type>
-      <joint name="shoulder3_joint">
-	<hardwareInterface>PosVelJointInterface</hardwareInterface>
-      </joint>
-      <actuator name="shoulder3_joint_motor">
-	<mechanicalReduction>1</mechanicalReduction>
-      </actuator>
-    </transmission>
-    <transmission name="wrist_joint_trans">
-      <type>transmission_interface/SimpleTransmission</type>
-      <joint name="wrist_joint">
-	<hardwareInterface>PosVelJointInterface</hardwareInterface>
-      </joint>
-      <actuator name="wrist_joint_motor">
-	<mechanicalReduction>1</mechanicalReduction>
-      </actuator>
-    </transmission>
-    <transmission name="left_finger_joint_trans">
-      <type>transmission_interface/SimpleTransmission</type>
-      <joint name="left_finger_joint">
-	<hardwareInterface>PositionJointInterface</hardwareInterface>
-      </joint>
-      <actuator name="left_finger_joint_motor">
-	<mechanicalReduction>1</mechanicalReduction>
-      </actuator>
-    </transmission>
-    <transmission name="right_finger_joint_trans">
-      <type>transmission_interface/SimpleTransmission</type>
-      <joint name="right_finger_joint">
-	<hardwareInterface>PositionJointInterface</hardwareInterface>
-      </joint>
-      <actuator name="right_finger_joint_motor">
-	<mechanicalReduction>1</mechanicalReduction>
-      </actuator>
-    </transmission>
   </xacro:if>
  <gazebo reference="FL_wheel_link">
@@ -210,4 +101,5 @@
     <maxVel>1.0</maxVel>
     <minDepth>0.00</minDepth>
+        <material>Gazebo/Black</material>
   </gazebo>
    <gazebo reference="FR_wheel_link">
@@ -220,4 +112,5 @@
     <maxVel>1.0</maxVel>
     <minDepth>0.00</minDepth>
+        <material>Gazebo/Black</material>
   </gazebo>
    <gazebo reference="RL_wheel_link">
@@ -230,4 +123,5 @@
     <maxVel>1.0</maxVel>
     <minDepth>0.00</minDepth>
+        <material>Gazebo/Black</material>
   </gazebo>
    <gazebo reference="RR_wheel_link">
@@ -240,4 +134,5 @@
     <maxVel>1.0</maxVel>
     <minDepth>0.00</minDepth>
+        <material>Gazebo/Black</material>
   </gazebo>
   <gazebo reference="base_link">
@@ -262,36 +157,3 @@
     <material>Gazebo/Black</material>
   </gazebo>
-  <gazebo reference="arm_link">
-    <material>Gazebo/DarkGrey</material>
-  </gazebo>
-  <gazebo reference="base_arm_link">
-    <material>Gazebo/DarkGrey</material>
-  </gazebo>
-  <gazebo reference="rotation1_link">
-    <material>Gazebo/DarkGrey</material>
-  </gazebo>
-    <gazebo reference="rotation2_link">
-    <material>Gazebo/DarkGrey</material>
-  </gazebo>
-  <gazebo reference="shoulder1_link">
-    <material>Gazebo/DarkGrey</material>
-  </gazebo>
-  <gazebo reference="shoulder2_link">
-    <material>Gazebo/DarkGrey</material>
-  </gazebo>
-  <gazebo reference="shoulder3_link">
-    <material>Gazebo/DarkGrey</material>
-  </gazebo>
-  <gazebo reference="wrist_link">
-    <material>Gazebo/DarkGrey</material>
-  </gazebo>
-  <gazebo reference="left_finger_link">
-    <material>Gazebo/Grey</material>
-  </gazebo>
-    <gazebo reference="right_finger_link">
-    <material>Gazebo/Grey</material>
-  </gazebo>
-  <gazebo reference="base_arm_link">
-    <material>Gazebo/Grey</material>
-  </gazebo>
 </robot>

File: robotican_manipulator_h/models/manipulator_h_gazebo.xacro (robot description, xacro)
@@ -1,8 +1,19 @@
 <?xml version="1.0"?>
-<robot xmlns:xacro="http://www.ros.org/wiki/xacro" name="Armadillo" description="Armadillo robot">
+<robot xmlns:xacro="http://www.ros.org/wiki/xacro" name="Manipulator_h_gazebo" description="Manipulator_h_gazebo">
 	<xacro:include filename="$(find robotican_manipulator_h)/models/manipulator_h.xacro" />
-	<link name="world" />
-  <joint name="fixed" type="fixed">
+	<xacro:include filename="$(find robotican_manipulator_h)/models/manipulator_h_gazebo_plugins.xacro" />
+	  <xacro:arg name="sr300" default="false"/>
+	    <!-- SR300 -->
+  <xacro:if value="$(arg sr300)">
+    <xacro:include filename="$(find robotican_common)/gazebo/sr300.xacro" />
+  </xacro:if>
+   <link name="world" />
+  <joint name="world_joint" type="fixed">
     <parent link="world"/>
+    <child link="map"/>
+  </joint>
+  <link name="map" />
+    <joint name="map_joint" type="fixed">
+    <parent link="map"/>
     <child link="arm_link"/>
   </joint>
@@ -41,135 +52,11 @@
     <axis xyz="0 0 0" />
   </joint>
- 	<gazebo>
-    	<gripper name="gripper">
-      		<grasp_check>
-				<attach_steps>1</attach_steps>
-				<detach_steps>2</detach_steps>
-				<min_contact_count>2</min_contact_count>
-      		</grasp_check>
-      			<gripper_link>left_finger_link</gripper_link>
-      			<gripper_link>right_finger_link</gripper_link>
-      			<palm_link>wrist_link</palm_link>
-    		</gripper>
-	</gazebo>
-  	<gazebo reference="left_finger_link">
-		<kp>1000000.0</kp>
-	    <kd>100.0</kd>
-	    <mu1>1.0</mu1>
-	    <mu2>1.0</mu2>
-	    <fdir1>0 0 1</fdir1>
-	    <maxVel>1.0</maxVel>
-	    <minDepth>0.00</minDepth>
-  	</gazebo>
-  	<gazebo reference="left_finger_joint">
-	    <implicitSpringDamper>1</implicitSpringDamper>
-	    <provideFeedback>1</provideFeedback>
-  	</gazebo>
-	<gazebo reference="right_finger_link">
-		<kp>1000000.0</kp>
-		<kd>100.0</kd>
-		<mu1>1.0</mu1>
-		<mu2>1.0</mu2>
-		<fdir1>0 0 1</fdir1>
-		<maxVel>1.0</maxVel>
-		<minDepth>0.00</minDepth>
-	</gazebo>
-	<gazebo reference="right_finger_joint">
-		<implicitSpringDamper>1</implicitSpringDamper>
-		<provideFeedback>1</provideFeedback>
-	</gazebo>
-	<gazebo reference="arm_link">
-		<gravity>true</gravity>
-	</gazebo>
-	<gazebo reference="right_finger_link">
-		<kp>1000000.0</kp>
-		<kd>100.0</kd>
-		<mu1>1.0</mu1>
-		<mu2>1.0</mu2>
-		<fdir1>0 0 1</fdir1>
-		<maxVel>1.0</maxVel>
-		<minDepth>0.00</minDepth>
-	</gazebo>
-  	<gazebo reference="right_finger_joint">
-	    <implicitSpringDamper>1</implicitSpringDamper>
-	    <provideFeedback>1</provideFeedback>
-  	</gazebo>
-	<xacro:include filename="$(find robotican_common)/gazebo/sr300.xacro" />
-    <gazebo>
+     <gazebo>
   		<plugin name="gazebo_ros_control" filename="libgazebo_ros_control.so">
     		<robotSimType>gazebo_ros_control/RoboticanRobotHWSim</robotSimType>
       	</plugin>
     </gazebo>
-	<transmission name="rotation1_joint_trans">
-		<type>transmission_interface/SimpleTransmission</type>
-		<joint name="rotation1_joint">
-			<hardwareInterface>PosVelJointInterface</hardwareInterface>
-		</joint>
-		<actuator name="rotation1_joint_motor">
-			<mechanicalReduction>1</mechanicalReduction>
-		</actuator>
-	</transmission>
-	<transmission name="shoulder1_joint_trans">
-		<type>transmission_interface/SimpleTransmission</type>
-		<joint name="shoulder1_joint">
-			<hardwareInterface>PosVelJointInterface</hardwareInterface>
-		</joint>
-		<actuator name="shoulder1_joint_motor">
-			<mechanicalReduction>1</mechanicalReduction>
-		</actuator>
-	</transmission>
-	<transmission name="shoulder2_joint_trans">
-		<type>transmission_interface/SimpleTransmission</type>
-		<joint name="shoulder2_joint">
-			<hardwareInterface>PosVelJointInterface</hardwareInterface>
-		</joint>
-		<actuator name="shoulder2_joint_motor">
-			<mechanicalReduction>1</mechanicalReduction>
-		</actuator>
-	</transmission>
-	<transmission name="rotation2_joint_trans">
-		<type>transmission_interface/SimpleTransmission</type>
-		<joint name="rotation2_joint">
-			<hardwareInterface>PosVelJointInterface</hardwareInterface>
-		</joint>
-		<actuator name="rotation2_joint_motor">
-			<mechanicalReduction>1</mechanicalReduction>
-		</actuator>
-	</transmission>
-	<transmission name="shoulder3_joint_trans">
-		<type>transmission_interface/SimpleTransmission</type>
-		<joint name="shoulder3_joint">
-			<hardwareInterface>PosVelJointInterface</hardwareInterface>
-		</joint>
-		<actuator name="shoulder3_joint_motor">
-			<mechanicalReduction>1</mechanicalReduction>
-		</actuator>
-	</transmission>
-	<transmission name="wrist_joint_trans">
-		<type>transmission_interface/SimpleTransmission</type>
-		<joint name="wrist_joint">
-			<hardwareInterface>PosVelJointInterface</hardwareInterface>
-		</joint>
-		<actuator name="wrist_joint_motor">
-			<mechanicalReduction>1</mechanicalReduction>
-		</actuator>
-	</transmission>
-	<transmission name="left_finger_joint_trans">
-		<type>transmission_interface/SimpleTransmission</type>
-		<joint name="left_finger_joint">
-			<hardwareInterface>PositionJointInterface</hardwareInterface>
-		</joint>
-		<actuator name="left_finger_joint_motor">
-			<mechanicalReduction>1</mechanicalReduction>
-		</actuator>
-	</transmission>
-	<transmission name="right_finger_joint_trans">
-		<type>transmission_interface/SimpleTransmission</type>
-		<joint name="right_finger_joint">
-			<hardwareInterface>PositionJointInterface</hardwareInterface>
-		</joint>
-		<actuator name="right_finger_joint_motor">
-			<mechanicalReduction>1</mechanicalReduction>
-		</actuator>
-	</transmission>
+	 <gazebo reference="arm_link">
+    <material>Gazebo/DarkGrey</material>
+  </gazebo>
 </robot>

Commit message: added: base_link collision

File: robotican_armadillo/description/models/armadillo_base.xacro (robot description, xacro)
@@ -38,4 +38,13 @@
       </material>
     </visual>
+     <collision name='base_collision'>
+       <origin
+        xyz="0 0 0"
+        rpy="0 0 0" />
+      <geometry>
+        <mesh
+          filename="package://robotican_armadillo/description/meshes/base_link.STL" />
+      </geometry>
+          </collision>
       <collision name='caster_collision'>
       <origin
