Commit message: find objects

File: robotican_armadillo/description/models/armadillo_gazebo.xacro (robot description, xacro)
@@ -3,8 +3,12 @@
   <xacro:include filename="$(find robotican_armadillo)/description/models/armadillo.xacro" />
   <xacro:property name="URF_FOV" value="${10.0*M_PI/180}" />
- <xacro:arg name="controllers" default="true"/>
+  <xacro:arg name="controllers" default="true"/>
   <xacro:arg name="front_camera" default="false"/>
   <xacro:arg name="rear_camera" default="false"/>
   <xacro:arg name="kinect2" default="false"/>
+  <xacro:arg name="kinect2_hz" default="30.0"/>
+  <xacro:arg name="kinect2_hd" default="true"/>
+  <xacro:arg name="kinect2_qhd" default="false"/>
+  <xacro:arg name="kinect2_sd" default="false"/>
   <xacro:arg name="urf" default="false"/>
   <xacro:arg name="imu" default="false"/>
@@ -12,62 +16,43 @@
   <xacro:arg name="lidar" default="false"/>
   <xacro:arg name="f200" default="false"/>
-  <xacro:arg name="kinect2_hz" default="10.0"/>
   <xacro:arg name="f200_hz" default="10.0"/>
   <gazebo>
-	  <gripper name="gripper">
-		<grasp_check>
-	     <attach_steps>1</attach_steps>
-	     <detach_steps>2</detach_steps>
-	     <min_contact_count>2</min_contact_count>
-		</grasp_check>
-		<gripper_link>left_finger_link</gripper_link>
-		<gripper_link>right_finger_link</gripper_link>
-		<palm_link>wrist_link</palm_link>
-	  </gripper>
-	</gazebo>
-	<!--
-	<gazebo reference="wrist_link">
-      <kp>1000000.0</kp>
-      <kd>100.0</kd>
-      <mu1>1.0</mu1>
-      <mu2>1.0</mu2>
-      <fdir1>0 0 1</fdir1>
-      <maxVel>1.0</maxVel>
-      <minDepth>0.00</minDepth>
-      <material>Gazebo/Grey</material>
-    </gazebo>
-    <gazebo reference="wrist_joint">
-      <implicitSpringDamper>1</implicitSpringDamper>
-      <provideFeedback>1</provideFeedback>
-    </gazebo>
-	-->
-    	<gazebo reference="left_finger_link">
-      <kp>1000000.0</kp>
-      <kd>100.0</kd>
-      <mu1>1.0</mu1>
-      <mu2>1.0</mu2>
-      <fdir1>0 0 1</fdir1>
-      <maxVel>1.0</maxVel>
-      <minDepth>0.00</minDepth>
-      <material>Gazebo/Grey</material>
-    </gazebo>
-    <gazebo reference="left_finger_joint">
-      <implicitSpringDamper>1</implicitSpringDamper>
-      <provideFeedback>1</provideFeedback>
-    </gazebo>
-     	<gazebo reference="right_finger_link">
-      <kp>1000000.0</kp>
-      <kd>100.0</kd>
-      <mu1>1.0</mu1>
-      <mu2>1.0</mu2>
-      <fdir1>0 0 1</fdir1>
-      <maxVel>1.0</maxVel>
-      <minDepth>0.00</minDepth>
-      <material>Gazebo/Grey</material>
-    </gazebo>
-    <gazebo reference="right_finger_joint">
-      <implicitSpringDamper>1</implicitSpringDamper>
-      <provideFeedback>1</provideFeedback>
-    </gazebo>
+    <gripper name="gripper">
+      <grasp_check>
+	<attach_steps>1</attach_steps>
+	<detach_steps>2</detach_steps>
+	<min_contact_count>2</min_contact_count>
+      </grasp_check>
+      <gripper_link>left_finger_link</gripper_link>
+      <gripper_link>right_finger_link</gripper_link>
+      <palm_link>wrist_link</palm_link>
+    </gripper>
+  </gazebo>
+  <gazebo reference="left_finger_link">
+    <kp>1000000.0</kp>
+    <kd>100.0</kd>
+    <mu1>1.0</mu1>
+    <mu2>1.0</mu2>
+    <fdir1>0 0 1</fdir1>
+    <maxVel>1.0</maxVel>
+    <minDepth>0.00</minDepth>
+  </gazebo>
+  <gazebo reference="left_finger_joint">
+    <implicitSpringDamper>1</implicitSpringDamper>
+    <provideFeedback>1</provideFeedback>
+  </gazebo>
+  <gazebo reference="right_finger_link">
+    <kp>1000000.0</kp>
+    <kd>100.0</kd>
+    <mu1>1.0</mu1>
+    <mu2>1.0</mu2>
+    <fdir1>0 0 1</fdir1>
+    <maxVel>1.0</maxVel>
+    <minDepth>0.00</minDepth>
+  </gazebo>
+  <gazebo reference="right_finger_joint">
+    <implicitSpringDamper>1</implicitSpringDamper>
+    <provideFeedback>1</provideFeedback>
+  </gazebo>
   <!--  <link name="dummy_link">
   </link>
@@ -78,560 +63,529 @@
   <axis xyz="0 0 0" />
   </joint>-->
-     <xacro:if value="$(arg f200)">
-		<gazebo reference="f200_rgb_frame">
-		  <sensor type="depth" name="f200">
-			<always_on>true</always_on>
-			<update_rate>$(arg f200_hz)</update_rate>
-			<camera>
-			  <horizontal_fov>1.20772254</horizontal_fov>
-			  <image>
-				<format>B8G8R8</format>
-				<width>640</width>
-				<height>480</height>
-			  </image>
-			  <clip>
-				<near>0.2</near>
-				<far>1.2</far>
-			  </clip>
-			</camera>
-			<plugin name="f200_camera_controller" filename="libgazebo_ros_openni_kinect.so">
-			  <alwaysOn>true</alwaysOn>
-			  <!--  <baseline>0.11</baseline> -->
-			  <updateRate>$(arg f200_hz)</updateRate>
-			  <cameraName>f200</cameraName>
-			  <imageTopicName>color/image_raw</imageTopicName>
-			  <cameraInfoTopicName>color/camera_info</cameraInfoTopicName>
-			  <depthImageTopicName>depth/image_raw</depthImageTopicName>
-			  <depthImageCameraInfoTopicName>depth/camera_info</depthImageCameraInfoTopicName>
-			  <pointCloudTopicName>depth/points</pointCloudTopicName>
-			  <frameName>f200_depth_optical_frame</frameName>
-			  <pointCloudCutoff>0.2</pointCloudCutoff>
-			  <pointCloudCutoffMax>1.2</pointCloudCutoffMax>
-			  <distortionK1>0.0</distortionK1>
-			  <distortionK2>0.0</distortionK2>
-			  <distortionK3>0.0</distortionK3>
-			  <distortionT1>0.0</distortionT1>
-			  <distortionT2>0.0</distortionT2>
-			 <!-- <Cx>320</Cx>
-			  <Cy>240</Cy>
-			  <focalLength>463.888592</focalLength> -->
-			</plugin>
-		  </sensor>
-		</gazebo>
-    </xacro:if>
+  <xacro:if value="$(arg f200)">
+    <gazebo reference="f200_rgb_frame">
+      <sensor type="depth" name="f200">
+	<always_on>true</always_on>
+	<update_rate>$(arg f200_hz)</update_rate>
+	<camera>
+	  <horizontal_fov>1.20772254</horizontal_fov>
+	  <image>
+	    <format>B8G8R8</format>
+	    <width>640</width>
+	    <height>480</height>
+	  </image>
+	  <clip>
+	    <near>0.2</near>
+	    <far>1.2</far>
+	  </clip>
+	</camera>
+	<plugin name="f200_camera_controller" filename="libgazebo_ros_openni_kinect.so">
+	  <alwaysOn>true</alwaysOn>
+	  <!--  <baseline>0.11</baseline> -->
+	  <updateRate>$(arg f200_hz)</updateRate>
+	  <cameraName>f200</cameraName>
+	  <imageTopicName>color/image_raw</imageTopicName>
+	  <cameraInfoTopicName>color/camera_info</cameraInfoTopicName>
+	  <depthImageTopicName>depth/image_raw</depthImageTopicName>
+	  <depthImageCameraInfoTopicName>depth/camera_info</depthImageCameraInfoTopicName>
+	  <pointCloudTopicName>depth/points</pointCloudTopicName>
+	  <frameName>f200_depth_optical_frame</frameName>
+	  <pointCloudCutoff>0.2</pointCloudCutoff>
+	  <pointCloudCutoffMax>1.2</pointCloudCutoffMax>
+	  <distortionK1>0.0</distortionK1>
+	  <distortionK2>0.0</distortionK2>
+	  <distortionK3>0.0</distortionK3>
+	  <distortionT1>0.0</distortionT1>
+	  <distortionT2>0.0</distortionT2>
+	  <!-- <Cx>320</Cx>
+	  <Cy>240</Cy>
+	  <focalLength>463.888592</focalLength> -->
+	</plugin>
+      </sensor>
+    </gazebo>
+  </xacro:if>
   <!-- kinect 2 -->
   <xacro:if value="$(arg kinect2)">
- <gazebo reference="kinect2_rgb_frame">
-      <sensor type="depth" name="kinect2">
-        <always_on>true</always_on>
-        <update_rate>$(arg kinect2_hz)</update_rate>
-      <camera>
-        <horizontal_fov>1.09606677025</horizontal_fov>
-        <image>
-          <format>B8G8R8</format>
-          <height>1080</height>
-          <width>1920</width>
-        </image>
-        <clip>
-          <near>0.5</near>
-          <far>9</far>
-        </clip>
-      </camera>
-        <plugin name="kinect2_camera_controller" filename="libgazebo_ros_openni_kinect.so">
-          <cameraName>kinect2</cameraName>
-          <alwaysOn>true</alwaysOn>
-          <updateRate>$(arg kinect2_hz)</updateRate>
-	      <imageTopicName>hd/image_color</imageTopicName>
-	      <cameraInfoTopicName>hd/camera_info</cameraInfoTopicName>
-	      <depthImageTopicName>hd/image_depth_rect</depthImageTopicName>
-	      <depthImageCameraInfoTopicName>hd/camera_info</depthImageCameraInfoTopicName>
-	      <pointCloudTopicName>hd/points</pointCloudTopicName>
-		  <frameName>kinect2_depth_optical_frame</frameName>
-          <baseline>0.1</baseline>
-          <distortion_k1>0.0</distortion_k1>
-          <distortion_k2>0.0</distortion_k2>
-          <distortion_k3>0.0</distortion_k3>
-          <distortion_t1>0.0</distortion_t1>
-          <distortion_t2>0.0</distortion_t2>
-       	  <pointCloudCutoff>0.4</pointCloudCutoff>
-		  <pointCloudCutoffMax>8.0</pointCloudCutoffMax>
-        </plugin>
+     <xacro:property name="kinect2_hz" value="$(arg kinect2_hz)"/>
+    <xacro:property name="kinect2_hd" value="$(arg kinect2_hd)"/>
+     <xacro:property name="kinect2_qhd" value="$(arg kinect2_qhd)"/>
+      <xacro:property name="kinect2_sd" value="$(arg kinect2_sd)"/>
+        -->
+	  <xacro:include filename="$(find robotican_common)/gazebo/kinect2.xacro" />
+  </xacro:if>
+  <!-- Sonars -->
+  <xacro:if value="$(arg urf)">
+    <gazebo reference="left_urf_link">
+      <material>Gazebo/Black</material>
+      <sensor type="ray" name="range">
+	<always_on>true</always_on>
+	<update_rate>10</update_rate>
+	<pose>0 0 0 0 0 0</pose>
+	<visualize>false</visualize>
+	<ray>
+	  <scan>
+	    <horizontal>
+	      <samples>10</samples>
+	      <resolution>1</resolution>
+	      <min_angle>${-URF_FOV/2.0}</min_angle>
+	      <max_angle>${URF_FOV/2.0}</max_angle>
+	    </horizontal>
+	    <vertical>
+	      <samples>10</samples>
+	      <resolution>1</resolution>
+	      <min_angle>${-URF_FOV/2.0}</min_angle>
+	      <max_angle>${URF_FOV/2.0}</max_angle>
+	    </vertical>
+	  </scan>
+	  <range>
+	    <min>0.01</min>
+	    <max>5.0</max>
+	    <resolution>0.001</resolution>
+	  </range>
+	</ray>
+	<plugin name="gazebo_ros_left_urf_controller" filename="libhector_gazebo_ros_sonar.so">
+	  <gaussianNoise>0.0001</gaussianNoise>
+	  <topicName>URF/left</topicName>
+	  <frameId>left_urf_link</frameId>
+	</plugin>
       </sensor>
     </gazebo>
-	</xacro:if>
-	<!-- Sonars -->
-	<xacro:if value="$(arg urf)">
-	  <gazebo reference="left_urf_link">
-	     <material>Gazebo/Black</material>
-	    <sensor type="ray" name="range">
-	      <always_on>true</always_on>
-	      <update_rate>10</update_rate>
-	      <pose>0 0 0 0 0 0</pose>
-	      <visualize>false</visualize>
-	      <ray>
-		<scan>
-		  <horizontal>
-		    <samples>10</samples>
-		    <resolution>1</resolution>
-		    <min_angle>${-URF_FOV/2.0}</min_angle>
-		    <max_angle>${URF_FOV/2.0}</max_angle>
-		  </horizontal>
-		  <vertical>
-		    <samples>10</samples>
-		    <resolution>1</resolution>
-		    <min_angle>${-URF_FOV/2.0}</min_angle>
-		    <max_angle>${URF_FOV/2.0}</max_angle>
-		  </vertical>
-		</scan>
-		<range>
-		  <min>0.01</min>
-		  <max>5.0</max>
-		  <resolution>0.001</resolution>
-		</range>
-	      </ray>
-	      <plugin name="gazebo_ros_left_urf_controller" filename="libhector_gazebo_ros_sonar.so">
-		<gaussianNoise>0.0001</gaussianNoise>
-		<topicName>URF/left</topicName>
-		<frameId>left_urf_link</frameId>
-	      </plugin>
-	    </sensor>
-	  </gazebo>
-	  <gazebo reference="right_urf_link">
-	    <sensor type="ray" name="range">
-	      <always_on>true</always_on>
-	      <update_rate>10</update_rate>
-	      <pose>0 0 0 0 0 0</pose>
-	      <visualize>false</visualize>
-	      <ray>
-		<scan>
-		  <horizontal>
-		    <samples>10</samples>
-		    <resolution>1</resolution>
-		    <min_angle>${-URF_FOV/2.0}</min_angle>
-		    <max_angle>${URF_FOV/2.0}</max_angle>
-		  </horizontal>
-		  <vertical>
-		    <samples>10</samples>
-		    <resolution>1</resolution>
-		    <min_angle>${-URF_FOV/2.0}</min_angle>
-		    <max_angle>${URF_FOV/2.0}</max_angle>
-		  </vertical>
-		</scan>
-		<range>
-		  <min>0.01</min>
-		  <max>5.0</max>
-		  <resolution>0.01</resolution>
-		</range>
-	      </ray>
-	      <plugin name="gazebo_ros_left_urf_controller" filename="libhector_gazebo_ros_sonar.so">
-		<gaussianNoise>0.001</gaussianNoise>
-		<topicName>URF/right</topicName>
-		<frameId>right_urf_link</frameId>
-	      </plugin>
-	    </sensor>
-	  </gazebo>
-	  <gazebo reference="rear_urf_link">
-	    <sensor type="ray" name="range">
-	      <always_on>true</always_on>
-	      <update_rate>10</update_rate>
-	      <pose>0 0 0 0 0 0</pose>
-	      <visualize>false</visualize>
-	      <ray>
-		<scan>
-		  <horizontal>
-		    <samples>10</samples>
-		    <resolution>1</resolution>
-		    <min_angle>${-URF_FOV/2.0}</min_angle>
-		    <max_angle>${URF_FOV/2.0}</max_angle>
-		  </horizontal>
-		  <vertical>
-		    <samples>10</samples>
-		    <resolution>1</resolution>
-		    <min_angle>${-URF_FOV/2.0}</min_angle>
-		    <max_angle>${URF_FOV/2.0}</max_angle>
-		  </vertical>
-		</scan>
-		<range>
-		  <min>0.01</min>
-		  <max>5.0</max>
-		  <resolution>0.01</resolution>
-		</range>
-	      </ray>
-	      <plugin name="gazebo_ros_left_urf_controller" filename="libhector_gazebo_ros_sonar.so">
-		<gaussianNoise>0.0001</gaussianNoise>
-		<topicName>URF/rear</topicName>
-		<frameId>rear_urf_link</frameId>
-	      </plugin>
-	    </sensor>
-	  </gazebo>
-	</xacro:if>
-	<!-- hokuyo URG-04LX-UG01   -->
-	<xacro:if value="$(arg lidar)">
-	  <gazebo reference="laser_link">
-	    <sensor type="ray" name="head_hokuyo_sensor">
-	      <pose>0 0 0 0 0 0</pose>
-	      <visualize>false</visualize>
-	      <update_rate>10</update_rate>
-	      <ray>
-		<scan>
-		  <horizontal>
-		    <samples>667</samples>
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