Commit message: update fix launchs

File: robotican_armadillo/description/models/armadillo_gazebo.xacro (robot description, xacro)
@@ -16,42 +16,5 @@
   <xacro:arg name="lidar" default="false"/>
   <xacro:arg name="sr300" default="false"/>
-  <gazebo>
-    <gripper name="gripper">
-      <grasp_check>
-	<attach_steps>1</attach_steps>
-	<detach_steps>1</detach_steps>
-	<min_contact_count>1</min_contact_count>
-      </grasp_check>
-      <gripper_link>left_finger_link</gripper_link>
-      <gripper_link>right_finger_link</gripper_link>
-      <palm_link>wrist_link</palm_link>
-    </gripper>
-  </gazebo>
-  <gazebo reference="left_finger_link">
-    <kp>1000000.0</kp>
-    <kd>100.0</kd>
-    <mu1>1.0</mu1>
-    <mu2>1.0</mu2>
-    <fdir1>0 0 1</fdir1>
-    <maxVel>1.0</maxVel>
-    <minDepth>0.00</minDepth>
-  </gazebo>
-  <gazebo reference="left_finger_joint">
-    <implicitSpringDamper>1</implicitSpringDamper>
-    <provideFeedback>1</provideFeedback>
-  </gazebo>
-  <gazebo reference="right_finger_link">
-    <kp>1000000.0</kp>
-    <kd>100.0</kd>
-    <mu1>1.0</mu1>
-    <mu2>1.0</mu2>
-    <fdir1>0 0 1</fdir1>
-    <maxVel>1.0</maxVel>
-    <minDepth>0.00</minDepth>
-  </gazebo>
-  <gazebo reference="right_finger_joint">
-    <implicitSpringDamper>1</implicitSpringDamper>
-    <provideFeedback>1</provideFeedback>
-  </gazebo>
+  <xacro:include filename="$(find robotican_manipulator_h)/models/manipulator_h_gazebo_plugins.xacro" />
   <!-- SR300 -->
   <xacro:if value="$(arg sr300)">
@@ -68,5 +31,5 @@
   <!-- Sonars -->
   <xacro:if value="$(arg urf)">
-  	<xacro:include filename="$(find robotican_common)/gazebo/urf.xacro" />
+    <xacro:include filename="$(find robotican_common)/gazebo/urf.xacro" />
     <xacro:urf name="left" link="left_urf_link" topic="URF/left" />
     <xacro:urf name="right" link="right_urf_link" topic="URF/right" />
@@ -90,224 +53,128 @@
       imu_offset_yaw="0" mag_offset_x="0"
       mag_offset_y="0" mag_offset_z="0" />
-  </xacro:if>
-  <!-- cameras  -->
-  <xacro:include filename="$(find robotican_common)/gazebo/camera.xacro" />
-  <xacro:if value="$(arg front_camera)">
-    <xacro:Camera name="front_camera" link="front_cam_link" image_width="640" image_height="480"
-      image_format="R8G8B8" clip_near="0.02" clip_far="300" />
-  </xacro:if>
-  <xacro:if value="$(arg rear_camera)">
-    <xacro:Camera name="rear_camera" link="rear_cam_link" image_width="640" image_height="480"
-      image_format="R8G8B8" clip_near="0.02" clip_far="300" />
-  </xacro:if>
-  <!-- controller manager and hardware interfaces -->
-  <xacro:if value="$(arg controllers)">
-    <gazebo>
-      <plugin name="gazebo_ros_control" filename="libgazebo_ros_control.so">
-    <robotSimType>gazebo_ros_control/RoboticanRobotHWSim</robotSimType>
-      </plugin>
-    </gazebo>
-    <!-- joints -->
-    <transmission name="left_wheel_joint_trans">
-      <type>transmission_interface/SimpleTransmission</type>
-      <joint name="left_wheel_joint">
-	<hardwareInterface>VelocityJointInterface</hardwareInterface>
-      </joint>
-      <actuator name="left_wheel_joint_motor">
-	<mechanicalReduction>1</mechanicalReduction>
-      </actuator>
-    </transmission>
-    <transmission name="right_wheel_joint_trans">
-      <type>transmission_interface/SimpleTransmission</type>
-      <joint name="right_wheel_joint">
-	<hardwareInterface>VelocityJointInterface</hardwareInterface>
-      </joint>
-      <actuator name="right_wheel_joint_motor">
-	<mechanicalReduction>1</mechanicalReduction>
-      </actuator>
-    </transmission>
-    <transmission name="torso_joint_trans">
-      <type>transmission_interface/SimpleTransmission</type>
-      <joint name="torso_joint">
-	<hardwareInterface>PositionJointInterface</hardwareInterface>
-      </joint>
-      <actuator name="torso_joint_motor">
-	<mechanicalReduction>1</mechanicalReduction>
-      </actuator>
-    </transmission>
-    <transmission name="rotation1_joint_trans">
-      <type>transmission_interface/SimpleTransmission</type>
-      <joint name="rotation1_joint">
-	<hardwareInterface>PosVelJointInterface</hardwareInterface>
-      </joint>
-      <actuator name="rotation1_joint_motor">
-	<mechanicalReduction>1</mechanicalReduction>
-      </actuator>
-    </transmission>
-    <transmission name="shoulder1_joint_trans">
-      <type>transmission_interface/SimpleTransmission</type>
-      <joint name="shoulder1_joint">
-	<hardwareInterface>PosVelJointInterface</hardwareInterface>
-      </joint>
-      <actuator name="shoulder1_joint_motor">
-	<mechanicalReduction>1</mechanicalReduction>
-      </actuator>
-    </transmission>
-    <transmission name="shoulder2_joint_trans">
-      <type>transmission_interface/SimpleTransmission</type>
-      <joint name="shoulder2_joint">
-	<hardwareInterface>PosVelJointInterface</hardwareInterface>
-      </joint>
-      <actuator name="shoulder2_joint_motor">
-	<mechanicalReduction>1</mechanicalReduction>
-      </actuator>
-    </transmission>
-    <transmission name="rotation2_joint_trans">
-      <type>transmission_interface/SimpleTransmission</type>
-      <joint name="rotation2_joint">
-	<hardwareInterface>PosVelJointInterface</hardwareInterface>
-      </joint>
-      <actuator name="rotation2_joint_motor">
-	<mechanicalReduction>1</mechanicalReduction>
-      </actuator>
-    </transmission>
-    <transmission name="shoulder3_joint_trans">
-      <type>transmission_interface/SimpleTransmission</type>
-      <joint name="shoulder3_joint">
-	<hardwareInterface>PosVelJointInterface</hardwareInterface>
-      </joint>
-      <actuator name="shoulder3_joint_motor">
-	<mechanicalReduction>1</mechanicalReduction>
-      </actuator>
-    </transmission>
-    <transmission name="wrist_joint_trans">
-      <type>transmission_interface/SimpleTransmission</type>
-      <joint name="wrist_joint">
-	<hardwareInterface>PosVelJointInterface</hardwareInterface>
-      </joint>
-      <actuator name="wrist_joint_motor">
-	<mechanicalReduction>1</mechanicalReduction>
-      </actuator>
-    </transmission>
-    <transmission name="left_finger_joint_trans">
-      <type>transmission_interface/SimpleTransmission</type>
-      <joint name="left_finger_joint">
-	<hardwareInterface>PositionJointInterface</hardwareInterface>
-      </joint>
-      <actuator name="left_finger_joint_motor">
-	<mechanicalReduction>1</mechanicalReduction>
-      </actuator>
-    </transmission>
-    <transmission name="right_finger_joint_trans">
-      <type>transmission_interface/SimpleTransmission</type>
-      <joint name="right_finger_joint">
-	<hardwareInterface>PositionJointInterface</hardwareInterface>
-      </joint>
-      <actuator name="right_finger_joint_motor">
-	<mechanicalReduction>1</mechanicalReduction>
-      </actuator>
-    </transmission>
-    <transmission name="head_pan_joint_trans">
-      <type>transmission_interface/SimpleTransmission</type>
-      <joint name="head_pan_joint">
-	<hardwareInterface>PositionJointInterface</hardwareInterface>
-      </joint>
-      <actuator name="head_pan_joint_motor">
-	<mechanicalReduction>1</mechanicalReduction>
-      </actuator>
-    </transmission>
-    <!-- HS-5685MH -->
-    <transmission name="head_tilt_joint_trans">
-      <type>transmission_interface/SimpleTransmission</type>
-      <joint name="head_tilt_joint">
-	<hardwareInterface>PositionJointInterface</hardwareInterface>
-      </joint>
-      <actuator name="head_tilt_joint_motor">
-	<mechanicalReduction>1</mechanicalReduction>
-      </actuator>
-    </transmission>
-    <gazebo reference="torso_joint_link">
-      <turnGravityOff>true</turnGravityOff>
-    </gazebo>
-  </xacro:if>
- <gazebo reference="left_wheel_link">
-    <!-- kp and kd for rubber -->
-    <kp>1000000.0</kp>
-    <kd>100.0</kd>
-    <mu1>1.5</mu1>
-    <mu2>1.5</mu2>
-    <fdir1>1 0 0</fdir1>
-    <maxVel>1.0</maxVel>
-    <minDepth>0.00</minDepth>
-  </gazebo>
-   <gazebo reference="right_wheel_link">
-    <!-- kp and kd for rubber -->
-    <kp>1000000.0</kp>
-    <kd>100.0</kd>
-    <mu1>1.5</mu1>
-    <mu2>1.5</mu2>
-    <fdir1>1 0 0</fdir1>
-    <maxVel>1.0</maxVel>
-    <minDepth>0.00</minDepth>
-  </gazebo>
-  <gazebo reference="base_link">
-    <material>Gazebo/Grey</material>
-  </gazebo>
-  <gazebo reference="right_urf_link">
-    <material>Gazebo/Black</material>
-  </gazebo>
-  <gazebo reference="left_urf_link">
-    <material>Gazebo/Black</material>
-  </gazebo>
-  <gazebo reference="rear_urf_link">
-    <material>Gazebo/Black</material>
-  </gazebo>
-  <gazebo reference="kinect2_link">
-    <material>Gazebo/Black</material>
-  </gazebo>
-  <gazebo reference="laser_link">
-    <material>Gazebo/Black</material>
-  </gazebo>
-  <gazebo reference="sr300_link">
-    <material>Gazebo/Black</material>
-  </gazebo>
-  <gazebo reference="front_cam_link">
-    <material>Gazebo/Black</material>
-  </gazebo>
-  <gazebo reference="rear_cam_link">
-    <material>Gazebo/Black</material>
-  </gazebo>
-  <gazebo reference="arm_link">
-    <material>Gazebo/DarkGrey</material>
-  </gazebo>
-  <gazebo reference="base_arm_link">
-    <material>Gazebo/DarkGrey</material>
-  </gazebo>
-  <gazebo reference="rotation1_link">
-    <material>Gazebo/DarkGrey</material>
-  </gazebo>
-    <gazebo reference="rotation2_link">
-    <material>Gazebo/DarkGrey</material>
-  </gazebo>
-  <gazebo reference="shoulder1_link">
-    <material>Gazebo/DarkGrey</material>
-  </gazebo>
-  <gazebo reference="shoulder2_link">
-    <material>Gazebo/DarkGrey</material>
-  </gazebo>
-  <gazebo reference="shoulder3_link">
-    <material>Gazebo/DarkGrey</material>
-  </gazebo>
-  <gazebo reference="wrist_link">
-    <material>Gazebo/DarkGrey</material>
-  </gazebo>
-  <gazebo reference="left_finger_link">
-    <material>Gazebo/Grey</material>
-  </gazebo>
-    <gazebo reference="right_finger_link">
-    <material>Gazebo/Grey</material>
-  </gazebo>
-  <gazebo reference="base_arm_link">
-    <material>Gazebo/Grey</material>
-  </gazebo>
-</robot>
+    </xacro:if>
+    <!-- cameras  -->
+    <xacro:include filename="$(find robotican_common)/gazebo/camera.xacro" />
+    <xacro:if value="$(arg front_camera)">
+      <xacro:Camera name="front_camera" link="front_cam_link" image_width="640" image_height="480"
+        image_format="R8G8B8" clip_near="0.02" clip_far="300" />
+      </xacro:if>
+      <xacro:if value="$(arg rear_camera)">
+        <xacro:Camera name="rear_camera" link="rear_cam_link" image_width="640" image_height="480"
+          image_format="R8G8B8" clip_near="0.02" clip_far="300" />
+        </xacro:if>
+        <!-- controller manager and hardware interfaces -->
+        <xacro:if value="$(arg controllers)">
+          <gazebo>
+            <plugin name="gazebo_ros_control" filename="libgazebo_ros_control.so">
+              <robotSimType>gazebo_ros_control/RoboticanRobotHWSim</robotSimType>
+            </plugin>
+          </gazebo>
+          <!-- joints -->
+          <transmission name="left_wheel_joint_trans">
+            <type>transmission_interface/SimpleTransmission</type>
+            <joint name="left_wheel_joint">
+              <hardwareInterface>VelocityJointInterface</hardwareInterface>
+            </joint>
+            <actuator name="left_wheel_joint_motor">
+              <mechanicalReduction>1</mechanicalReduction>
+            </actuator>
+          </transmission>
+          <transmission name="right_wheel_joint_trans">
+            <type>transmission_interface/SimpleTransmission</type>
+            <joint name="right_wheel_joint">
+              <hardwareInterface>VelocityJointInterface</hardwareInterface>
+            </joint>
+            <actuator name="right_wheel_joint_motor">
+              <mechanicalReduction>1</mechanicalReduction>
+            </actuator>
+          </transmission>
+          <transmission name="torso_joint_trans">
+            <type>transmission_interface/SimpleTransmission</type>
+            <joint name="torso_joint">
+              <hardwareInterface>PositionJointInterface</hardwareInterface>
+            </joint>
+            <actuator name="torso_joint_motor">
+              <mechanicalReduction>1</mechanicalReduction>
+            </actuator>
+          </transmission>
+          <transmission name="head_pan_joint_trans">
+            <type>transmission_interface/SimpleTransmission</type>
+            <joint name="head_pan_joint">
+              <hardwareInterface>PositionJointInterface</hardwareInterface>
+            </joint>
+            <actuator name="head_pan_joint_motor">
+              <mechanicalReduction>1</mechanicalReduction>
+            </actuator>
+          </transmission>
+          <!-- HS-5685MH -->
+          <transmission name="head_tilt_joint_trans">
+            <type>transmission_interface/SimpleTransmission</type>
+            <joint name="head_tilt_joint">
+              <hardwareInterface>PositionJointInterface</hardwareInterface>
+            </joint>
+            <actuator name="head_tilt_joint_motor">
+              <mechanicalReduction>1</mechanicalReduction>
+            </actuator>
+          </transmission>
+          <gazebo reference="torso_joint_link">
+            <turnGravityOff>true</turnGravityOff>
+          </gazebo>
+        </xacro:if>
+        <gazebo reference="left_wheel_link">
+          <!-- kp and kd for rubber -->
+          <kp>1000000.0</kp>
+          <kd>100.0</kd>
+          <mu1>1.5</mu1>
+          <mu2>1.5</mu2>
+          <fdir1>1 0 0</fdir1>
+          <maxVel>1.0</maxVel>
+          <minDepth>0.00</minDepth>
+        </gazebo>
+        <gazebo reference="right_wheel_link">
+          <!-- kp and kd for rubber -->
+          <kp>1000000.0</kp>
+          <kd>100.0</kd>
+          <mu1>1.5</mu1>
+          <mu2>1.5</mu2>
+          <fdir1>1 0 0</fdir1>
+          <maxVel>1.0</maxVel>
+          <minDepth>0.00</minDepth>
+        </gazebo>
+        <gazebo reference="base_link">
+          <material>Gazebo/Grey</material>
+        </gazebo>
+        <gazebo reference="right_urf_link">
+          <material>Gazebo/Black</material>
+        </gazebo>
+        <gazebo reference="left_urf_link">
+          <material>Gazebo/Black</material>
+        </gazebo>
+        <gazebo reference="rear_urf_link">
+          <material>Gazebo/Black</material>
+        </gazebo>
+        <gazebo reference="kinect2_link">
+          <material>Gazebo/Black</material>
+        </gazebo>
+        <gazebo reference="laser_link">
+          <material>Gazebo/Black</material>
+        </gazebo>
+        <gazebo reference="sr300_link">
+          <material>Gazebo/Black</material>
+        </gazebo>
+        <gazebo reference="front_cam_link">
+          <material>Gazebo/Black</material>
+        </gazebo>
+        <gazebo reference="rear_cam_link">
+          <material>Gazebo/Black</material>
+        </gazebo>
+        <gazebo reference="arm_link">
+          <material>Gazebo/DarkGrey</material>
+        </gazebo>
+        <gazebo reference="base_arm_link">
+          <material>Gazebo/DarkGrey</material>
+        </gazebo>
+        <gazebo reference="base_arm_link">
+          <material>Gazebo/Grey</material>
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