Commit message: update fix launchs

File: robotican_komodo/description/models/komodo_gazebo.xacro (robot description, xacro)
@@ -12,5 +12,5 @@
   <xacro:arg name="depth_camera" default="false"/>
   <xacro:include filename="$(find robotican_manipulator_h)/models/manipulator_h_gazebo_plugins.xacro" />
-  	    <!-- SR300 -->
+  <!-- SR300 -->
   <xacro:if value="$(arg sr300)">
     <xacro:include filename="$(find robotican_common)/gazebo/sr300.xacro" />
@@ -22,5 +22,5 @@
   <!-- Sonars -->
   <xacro:if value="$(arg urf)">
-  	<xacro:include filename="$(find robotican_common)/gazebo/urf.xacro" />
+    <xacro:include filename="$(find robotican_common)/gazebo/urf.xacro" />
     <xacro:urf name="left" link="left_urf_link" topic="URF/left" />
     <xacro:urf name="right" link="right_urf_link" topic="URF/right" />
@@ -44,120 +44,120 @@
       imu_offset_yaw="0" mag_offset_x="0"
       mag_offset_y="0" mag_offset_z="0" />
-  </xacro:if>
-  <!-- cameras  -->
-  <xacro:include filename="$(find robotican_common)/gazebo/camera.xacro" />
-  <xacro:if value="$(arg front_camera)">
-    <xacro:Camera name="front_camera" link="front_cam_link" image_width="640" image_height="480"
-      image_format="R8G8B8" clip_near="0.02" clip_far="300" />
-  </xacro:if>
-  <!-- controller manager and hardware interfaces -->
-  <xacro:if value="$(arg controllers)">
-    <gazebo>
-      <plugin name="gazebo_ros_control" filename="libgazebo_ros_control.so">
-    <robotSimType>gazebo_ros_control/RoboticanRobotHWSim</robotSimType>
-      </plugin>
-    </gazebo>
-    <!-- joints -->
-    <transmission name="FL_wheel_joint_trans">
-      <type>transmission_interface/SimpleTransmission</type>
-      <joint name="FL_wheel_joint">
-	<hardwareInterface>VelocityJointInterface</hardwareInterface>
-      </joint>
-      <actuator name="FL_wheel_joint_motor">
-	<mechanicalReduction>1</mechanicalReduction>
-      </actuator>
-    </transmission>
-    <transmission name="FR_wheel_joint_trans">
-      <type>transmission_interface/SimpleTransmission</type>
-      <joint name="FR_wheel_joint">
-	<hardwareInterface>VelocityJointInterface</hardwareInterface>
-      </joint>
-      <actuator name="FR_wheel_joint_motor">
-	<mechanicalReduction>1</mechanicalReduction>
-      </actuator>
-    </transmission>
+    </xacro:if>
+    <!-- cameras  -->
+    <xacro:include filename="$(find robotican_common)/gazebo/camera.xacro" />
+    <xacro:if value="$(arg front_camera)">
+      <xacro:Camera name="front_camera" link="front_cam_link" image_width="640" image_height="480"
+        image_format="R8G8B8" clip_near="0.02" clip_far="300" />
+      </xacro:if>
+      <!-- controller manager and hardware interfaces -->
+      <xacro:if value="$(arg controllers)">
+        <gazebo>
+          <plugin name="gazebo_ros_control" filename="libgazebo_ros_control.so">
+            <robotSimType>gazebo_ros_control/RoboticanRobotHWSim</robotSimType>
+          </plugin>
+        </gazebo>
+        <!-- joints -->
+        <transmission name="FL_wheel_joint_trans">
+          <type>transmission_interface/SimpleTransmission</type>
+          <joint name="FL_wheel_joint">
+            <hardwareInterface>VelocityJointInterface</hardwareInterface>
+          </joint>
+          <actuator name="FL_wheel_joint_motor">
+            <mechanicalReduction>1</mechanicalReduction>
+          </actuator>
+        </transmission>
+        <transmission name="FR_wheel_joint_trans">
+          <type>transmission_interface/SimpleTransmission</type>
+          <joint name="FR_wheel_joint">
+            <hardwareInterface>VelocityJointInterface</hardwareInterface>
+          </joint>
+          <actuator name="FR_wheel_joint_motor">
+            <mechanicalReduction>1</mechanicalReduction>
+          </actuator>
+        </transmission>
         <transmission name="RL_wheel_joint_trans">
-      <type>transmission_interface/SimpleTransmission</type>
-      <joint name="RL_wheel_joint">
-	<hardwareInterface>VelocityJointInterface</hardwareInterface>
-      </joint>
-      <actuator name="RL_wheel_joint_motor">
-	<mechanicalReduction>1</mechanicalReduction>
-      </actuator>
-    </transmission>
-    <transmission name="RR_wheel_joint_trans">
-      <type>transmission_interface/SimpleTransmission</type>
-      <joint name="RR_wheel_joint">
-	<hardwareInterface>VelocityJointInterface</hardwareInterface>
-      </joint>
-      <actuator name="RR_wheel_joint_motor">
-	<mechanicalReduction>1</mechanicalReduction>
-      </actuator>
-    </transmission>
-  </xacro:if>
- <gazebo reference="FL_wheel_link">
-    <!-- kp and kd for rubber -->
-    <kp>1000000.0</kp>
-    <kd>100.0</kd>
-    <mu1>1.5</mu1>
-    <mu2>1.5</mu2>
-    <fdir1>1 0 0</fdir1>
-    <maxVel>1.0</maxVel>
-    <minDepth>0.00</minDepth>
+          <type>transmission_interface/SimpleTransmission</type>
+          <joint name="RL_wheel_joint">
+            <hardwareInterface>VelocityJointInterface</hardwareInterface>
+          </joint>
+          <actuator name="RL_wheel_joint_motor">
+            <mechanicalReduction>1</mechanicalReduction>
+          </actuator>
+        </transmission>
+        <transmission name="RR_wheel_joint_trans">
+          <type>transmission_interface/SimpleTransmission</type>
+          <joint name="RR_wheel_joint">
+            <hardwareInterface>VelocityJointInterface</hardwareInterface>
+          </joint>
+          <actuator name="RR_wheel_joint_motor">
+            <mechanicalReduction>1</mechanicalReduction>
+          </actuator>
+        </transmission>
+      </xacro:if>
+      <gazebo reference="FL_wheel_link">
+        <!-- kp and kd for rubber -->
+        <kp>1000000.0</kp>
+        <kd>100.0</kd>
+        <mu1>1.5</mu1>
+        <mu2>1.5</mu2>
+        <fdir1>1 0 0</fdir1>
+        <maxVel>1.0</maxVel>
+        <minDepth>0.00</minDepth>
         <material>Gazebo/Black</material>
-  </gazebo>
-   <gazebo reference="FR_wheel_link">
-    <!-- kp and kd for rubber -->
-    <kp>1000000.0</kp>
-    <kd>100.0</kd>
-    <mu1>1.5</mu1>
-    <mu2>1.5</mu2>
-    <fdir1>1 0 0</fdir1>
-    <maxVel>1.0</maxVel>
-    <minDepth>0.00</minDepth>
+      </gazebo>
+      <gazebo reference="FR_wheel_link">
+        <!-- kp and kd for rubber -->
+        <kp>1000000.0</kp>
+        <kd>100.0</kd>
+        <mu1>1.5</mu1>
+        <mu2>1.5</mu2>
+        <fdir1>1 0 0</fdir1>
+        <maxVel>1.0</maxVel>
+        <minDepth>0.00</minDepth>
         <material>Gazebo/Black</material>
-  </gazebo>
-   <gazebo reference="RL_wheel_link">
-    <!-- kp and kd for rubber -->
-    <kp>1000000.0</kp>
-    <kd>100.0</kd>
-    <mu1>1.5</mu1>
-    <mu2>1.5</mu2>
-    <fdir1>1 0 0</fdir1>
-    <maxVel>1.0</maxVel>
-    <minDepth>0.00</minDepth>
+      </gazebo>
+      <gazebo reference="RL_wheel_link">
+        <!-- kp and kd for rubber -->
+        <kp>1000000.0</kp>
+        <kd>100.0</kd>
+        <mu1>1.5</mu1>
+        <mu2>1.5</mu2>
+        <fdir1>1 0 0</fdir1>
+        <maxVel>1.0</maxVel>
+        <minDepth>0.00</minDepth>
         <material>Gazebo/Black</material>
-  </gazebo>
-   <gazebo reference="RR_wheel_link">
-    <!-- kp and kd for rubber -->
-    <kp>1000000.0</kp>
-    <kd>100.0</kd>
-    <mu1>1.5</mu1>
-    <mu2>1.5</mu2>
-    <fdir1>1 0 0</fdir1>
-    <maxVel>1.0</maxVel>
-    <minDepth>0.00</minDepth>
+      </gazebo>
+      <gazebo reference="RR_wheel_link">
+        <!-- kp and kd for rubber -->
+        <kp>1000000.0</kp>
+        <kd>100.0</kd>
+        <mu1>1.5</mu1>
+        <mu2>1.5</mu2>
+        <fdir1>1 0 0</fdir1>
+        <maxVel>1.0</maxVel>
+        <minDepth>0.00</minDepth>
         <material>Gazebo/Black</material>
-  </gazebo>
-  <gazebo reference="base_link">
-    <material>Gazebo/Grey</material>
-  </gazebo>
-  <gazebo reference="FR_urf_link">
-    <material>Gazebo/Black</material>
-  </gazebo>
-  <gazebo reference="FL_urf_link">
-    <material>Gazebo/Black</material>
-  </gazebo>
-    <gazebo reference="RR_urf_link">
-    <material>Gazebo/Black</material>
-  </gazebo>
-  <gazebo reference="RL_urf_link">
-    <material>Gazebo/Black</material>
-  </gazebo>
-  <gazebo reference="rear_urf_link">
-    <material>Gazebo/Black</material>
-  </gazebo>
-  <gazebo reference="sr300_link">
-    <material>Gazebo/Black</material>
-  </gazebo>
+      </gazebo>
+      <gazebo reference="base_link">
+        <material>Gazebo/Grey</material>
+      </gazebo>
+      <gazebo reference="FR_urf_link">
+        <material>Gazebo/Black</material>
+      </gazebo>
+      <gazebo reference="FL_urf_link">
+        <material>Gazebo/Black</material>
+      </gazebo>
+      <gazebo reference="RR_urf_link">
+        <material>Gazebo/Black</material>
+      </gazebo>
+      <gazebo reference="RL_urf_link">
+        <material>Gazebo/Black</material>
+      </gazebo>
+      <gazebo reference="rear_urf_link">
+        <material>Gazebo/Black</material>
+      </gazebo>
+      <gazebo reference="sr300_link">
+        <material>Gazebo/Black</material>
+      </gazebo>
 </robot>

File: robotican_manipulator_h/models/manipulator_h_gazebo_plugins.xacro (robot description, xacro)
@@ -1,131 +1,131 @@
 <?xml version="1.0"?>
 <robot xmlns:xacro="http://www.ros.org/wiki/xacro" name="Manipulator_h_gazebo_plugins" description="Manipulator_h_gazebo_plugins">
- 	<gazebo>
-    	<gripper name="gripper">
-      		<grasp_check>
-				<attach_steps>1</attach_steps>
-				<detach_steps>2</detach_steps>
-				<min_contact_count>2</min_contact_count>
-      		</grasp_check>
-      			<gripper_link>left_finger_link</gripper_link>
-      			<gripper_link>right_finger_link</gripper_link>
-      			<palm_link>wrist_link</palm_link>
-    		</gripper>
-	</gazebo>
-  	<gazebo reference="left_finger_link">
-		<kp>1000000.0</kp>
-	    <kd>100.0</kd>
-	    <mu1>1.0</mu1>
-	    <mu2>1.0</mu2>
-	    <fdir1>0 0 1</fdir1>
-	    <maxVel>1.0</maxVel>
-	    <minDepth>0.00</minDepth>
-  	</gazebo>
-  	<gazebo reference="left_finger_joint">
-	    <implicitSpringDamper>1</implicitSpringDamper>
-	    <provideFeedback>1</provideFeedback>
-  	</gazebo>
-	<gazebo reference="right_finger_link">
-		<kp>1000000.0</kp>
-		<kd>100.0</kd>
-		<mu1>1.0</mu1>
-		<mu2>1.0</mu2>
-		<fdir1>0 0 1</fdir1>
-		<maxVel>1.0</maxVel>
-		<minDepth>0.00</minDepth>
-	</gazebo>
-	<gazebo reference="right_finger_joint">
-		<implicitSpringDamper>1</implicitSpringDamper>
-		<provideFeedback>1</provideFeedback>
-	</gazebo>
-	<gazebo reference="arm_link">
-		<gravity>true</gravity>
-	</gazebo>
-	<gazebo reference="right_finger_link">
-		<kp>1000000.0</kp>
-		<kd>100.0</kd>
-		<mu1>1.0</mu1>
-		<mu2>1.0</mu2>
-		<fdir1>0 0 1</fdir1>
-		<maxVel>1.0</maxVel>
-		<minDepth>0.00</minDepth>
-	</gazebo>
-  	<gazebo reference="right_finger_joint">
-	    <implicitSpringDamper>1</implicitSpringDamper>
-	    <provideFeedback>1</provideFeedback>
-  	</gazebo>
-	<transmission name="rotation1_joint_trans">
-		<type>transmission_interface/SimpleTransmission</type>
-		<joint name="rotation1_joint">
-			<hardwareInterface>PosVelJointInterface</hardwareInterface>
-		</joint>
-		<actuator name="rotation1_joint_motor">
-			<mechanicalReduction>1</mechanicalReduction>
-		</actuator>
-	</transmission>
-	<transmission name="shoulder1_joint_trans">
-		<type>transmission_interface/SimpleTransmission</type>
-		<joint name="shoulder1_joint">
-			<hardwareInterface>PosVelJointInterface</hardwareInterface>
-		</joint>
-		<actuator name="shoulder1_joint_motor">
-			<mechanicalReduction>1</mechanicalReduction>
-		</actuator>
-	</transmission>
-	<transmission name="shoulder2_joint_trans">
-		<type>transmission_interface/SimpleTransmission</type>
-		<joint name="shoulder2_joint">
-			<hardwareInterface>PosVelJointInterface</hardwareInterface>
-		</joint>
-		<actuator name="shoulder2_joint_motor">
-			<mechanicalReduction>1</mechanicalReduction>
-		</actuator>
-	</transmission>
-	<transmission name="rotation2_joint_trans">
-		<type>transmission_interface/SimpleTransmission</type>
-		<joint name="rotation2_joint">
-			<hardwareInterface>PosVelJointInterface</hardwareInterface>
-		</joint>
-		<actuator name="rotation2_joint_motor">
-			<mechanicalReduction>1</mechanicalReduction>
-		</actuator>
-	</transmission>
-	<transmission name="shoulder3_joint_trans">
-		<type>transmission_interface/SimpleTransmission</type>
-		<joint name="shoulder3_joint">
-			<hardwareInterface>PosVelJointInterface</hardwareInterface>
-		</joint>
-		<actuator name="shoulder3_joint_motor">
-			<mechanicalReduction>1</mechanicalReduction>
-		</actuator>
-	</transmission>
-	<transmission name="wrist_joint_trans">
-		<type>transmission_interface/SimpleTransmission</type>
-		<joint name="wrist_joint">
-			<hardwareInterface>PosVelJointInterface</hardwareInterface>
-		</joint>
-		<actuator name="wrist_joint_motor">
-			<mechanicalReduction>1</mechanicalReduction>
-		</actuator>
-	</transmission>
-	<transmission name="left_finger_joint_trans">
-		<type>transmission_interface/SimpleTransmission</type>
-		<joint name="left_finger_joint">
-			<hardwareInterface>PositionJointInterface</hardwareInterface>
-		</joint>
-		<actuator name="left_finger_joint_motor">
-			<mechanicalReduction>1</mechanicalReduction>
-		</actuator>
-	</transmission>
-	<transmission name="right_finger_joint_trans">
-		<type>transmission_interface/SimpleTransmission</type>
-		<joint name="right_finger_joint">
-			<hardwareInterface>PositionJointInterface</hardwareInterface>
-		</joint>
-		<actuator name="right_finger_joint_motor">
-			<mechanicalReduction>1</mechanicalReduction>
-		</actuator>
-	</transmission>
-	 <gazebo reference="arm_link">
+  <gazebo>
+    <gripper name="gripper">
+      <grasp_check>
+        <attach_steps>1</attach_steps>
+        <detach_steps>2</detach_steps>
+        <min_contact_count>2</min_contact_count>
+      </grasp_check>
+      <gripper_link>left_finger_link</gripper_link>
+      <gripper_link>right_finger_link</gripper_link>
+      <palm_link>wrist_link</palm_link>
+    </gripper>
+  </gazebo>
+  <gazebo reference="left_finger_link">
+    <kp>1000000.0</kp>
+    <kd>100.0</kd>
+    <mu1>1.0</mu1>
+    <mu2>1.0</mu2>
+    <fdir1>0 0 1</fdir1>
+    <maxVel>1.0</maxVel>
+    <minDepth>0.00</minDepth>
+  </gazebo>
+  <gazebo reference="left_finger_joint">
+    <implicitSpringDamper>1</implicitSpringDamper>
+    <provideFeedback>1</provideFeedback>
+  </gazebo>
+  <gazebo reference="right_finger_link">
+    <kp>1000000.0</kp>
+    <kd>100.0</kd>
+    <mu1>1.0</mu1>
+    <mu2>1.0</mu2>
+    <fdir1>0 0 1</fdir1>
+    <maxVel>1.0</maxVel>
+    <minDepth>0.00</minDepth>
+  </gazebo>
+  <gazebo reference="right_finger_joint">
+    <implicitSpringDamper>1</implicitSpringDamper>
+    <provideFeedback>1</provideFeedback>
+  </gazebo>
+  <gazebo reference="arm_link">
+    <gravity>true</gravity>
+  </gazebo>
+  <gazebo reference="right_finger_link">
+    <kp>1000000.0</kp>
+    <kd>100.0</kd>
+    <mu1>1.0</mu1>
+    <mu2>1.0</mu2>
+    <fdir1>0 0 1</fdir1>
+    <maxVel>1.0</maxVel>
+    <minDepth>0.00</minDepth>
+  </gazebo>
+  <gazebo reference="right_finger_joint">
+    <implicitSpringDamper>1</implicitSpringDamper>
+    <provideFeedback>1</provideFeedback>
+  </gazebo>
+  <transmission name="rotation1_joint_trans">
+    <type>transmission_interface/SimpleTransmission</type>
+    <joint name="rotation1_joint">
+      <hardwareInterface>PosVelJointInterface</hardwareInterface>
+    </joint>
+    <actuator name="rotation1_joint_motor">
+      <mechanicalReduction>1</mechanicalReduction>
+    </actuator>
+  </transmission>
+  <transmission name="shoulder1_joint_trans">
+    <type>transmission_interface/SimpleTransmission</type>
+    <joint name="shoulder1_joint">
+      <hardwareInterface>PosVelJointInterface</hardwareInterface>
+    </joint>
+    <actuator name="shoulder1_joint_motor">
+      <mechanicalReduction>1</mechanicalReduction>
+    </actuator>
+  </transmission>
+  <transmission name="shoulder2_joint_trans">
+    <type>transmission_interface/SimpleTransmission</type>
+    <joint name="shoulder2_joint">
+      <hardwareInterface>PosVelJointInterface</hardwareInterface>
+    </joint>
+    <actuator name="shoulder2_joint_motor">
+      <mechanicalReduction>1</mechanicalReduction>
+    </actuator>
+  </transmission>
+  <transmission name="rotation2_joint_trans">
+    <type>transmission_interface/SimpleTransmission</type>
+    <joint name="rotation2_joint">
+      <hardwareInterface>PosVelJointInterface</hardwareInterface>
+    </joint>
+    <actuator name="rotation2_joint_motor">
+      <mechanicalReduction>1</mechanicalReduction>
+    </actuator>
+  </transmission>
+  <transmission name="shoulder3_joint_trans">
+    <type>transmission_interface/SimpleTransmission</type>
+    <joint name="shoulder3_joint">
+      <hardwareInterface>PosVelJointInterface</hardwareInterface>
+    </joint>
+    <actuator name="shoulder3_joint_motor">
+      <mechanicalReduction>1</mechanicalReduction>
+    </actuator>
+  </transmission>
+  <transmission name="wrist_joint_trans">
+    <type>transmission_interface/SimpleTransmission</type>
+    <joint name="wrist_joint">
+      <hardwareInterface>PosVelJointInterface</hardwareInterface>
+    </joint>
+    <actuator name="wrist_joint_motor">
+      <mechanicalReduction>1</mechanicalReduction>
+    </actuator>
+  </transmission>
+  <transmission name="left_finger_joint_trans">
+    <type>transmission_interface/SimpleTransmission</type>
+    <joint name="left_finger_joint">
+      <hardwareInterface>PositionJointInterface</hardwareInterface>
+    </joint>
+    <actuator name="left_finger_joint_motor">
+      <mechanicalReduction>1</mechanicalReduction>
+    </actuator>
+  </transmission>
+  <transmission name="right_finger_joint_trans">
+    <type>transmission_interface/SimpleTransmission</type>
+    <joint name="right_finger_joint">
+      <hardwareInterface>PositionJointInterface</hardwareInterface>
+    </joint>
+    <actuator name="right_finger_joint_motor">
+      <mechanicalReduction>1</mechanicalReduction>
+    </actuator>
+  </transmission>
+  <gazebo reference="arm_link">
     <material>Gazebo/DarkGrey</material>
   </gazebo>
@@ -136,5 +136,5 @@
     <material>Gazebo/DarkGrey</material>
   </gazebo>
-    <gazebo reference="rotation2_link">
+  <gazebo reference="rotation2_link">
     <material>Gazebo/DarkGrey</material>
   </gazebo>
@@ -154,5 +154,5 @@
     <material>Gazebo/Grey</material>
   </gazebo>
-    <gazebo reference="right_finger_link">
+  <gazebo reference="right_finger_link">
     <material>Gazebo/Grey</material>
   </gazebo>

Commit message: update: softkinetics camera for armadillo

File: robotican_armadillo/description/models/armadillo_gazebo.xacro (robot description, xacro)
@@ -2,4 +2,5 @@
 <robot xmlns:xacro="http://www.ros.org/wiki/xacro" name="Armadillo" description="Armadillo robot">
   <xacro:include filename="$(find robotican_armadillo)/description/models/armadillo.xacro" />
+  <xacro:include filename="$(find robotican_common)/gazebo/softkinetic_camera_ds325.xacro" />
   <xacro:property name="URF_FOV" value="${10.0*M_PI/180}" />
   <xacro:arg name="controllers" default="true"/>
@@ -15,9 +16,15 @@
   <xacro:arg name="gps" default="false"/>
   <xacro:arg name="lidar" default="false"/>
-  <xacro:arg name="sr300" default="false"/>
+  <xacro:arg name="softkinetic" default="false"/>
+  <!--<xacro:arg name="sr300" default="false"/>-->
   <xacro:include filename="$(find robotican_manipulator_h)/models/manipulator_h_gazebo_plugins.xacro" />
   <!-- SR300 -->
-  <xacro:if value="$(arg sr300)">
+  <!--<xacro:if value="$(arg sr300)">
     <xacro:include filename="$(find robotican_common)/gazebo/sr300.xacro" />
+  </xacro:if> -->
+  <!-- Softkinetic -->
+    <!-- softkinetic -->
+  <xacro:if value="$(arg softkinetic)">
+     <xacro:softkinetic_gazebo name="softkinetic_camera_rgb" ros_topic="softkinetic_camera"/>
   </xacro:if>
   <!-- kinect 2 -->
@@ -160,5 +167,8 @@
           <material>Gazebo/Black</material>
         </gazebo>
-        <gazebo reference="sr300_link">
+        <!--<gazebo reference="sr300_link">
+          <material>Gazebo/Black</material>
+        </gazebo> -->
+        <gazebo reference="softkinetic_camera_link">
           <material>Gazebo/Black</material>
         </gazebo>
