Commit message: fix conflict

File: robotican_lizi/description/models/lizi_gazebo.xacro (robot description, xacro)
@@ -9,8 +9,47 @@
   <xacro:arg name="lidar" default="false"/>
   <xacro:arg name="sr300" default="false"/>
+  <xacro:arg name="pan_tilt" default='false'/>
   <xacro:arg name="asus_hz" default="10.0"/>
   <xacro:property name="URF_FOV" value="${10.0*M_PI/180}" />
- <xacro:if value="$(arg urf)">
-      <gazebo reference="left_urf_link">
+  <xacro:if value="$(arg pan_tilt)">
+    <gazebo reference="asus_camera_rgb_frame">
+      <sensor type="depth" name="asus_camera">
+        <always_on>true</always_on>
+        <update_rate>$(arg asus_hz)</update_rate>
+      <camera>
+        <horizontal_fov>${57.0*M_PI/180.0}</horizontal_fov>
+        <image>
+          <format>R8G8B8</format>
+          <height>640</height>
+          <width>480</width>
+        </image>
+        <clip>
+          <near>0.01</near>
+          <far>5.0</far>
+        </clip>
+      </camera>
+        <plugin name="asus_camera_controller" filename="libgazebo_ros_openni_kinect.so">
+          <cameraName>asus_camera</cameraName>
+          <alwaysOn>true</alwaysOn>
+          <updateRate>$(arg asus_hz)</updateRate>
+            <imageTopicName>rgb/image_raw</imageTopicName>
+            <cameraInfoTopicName>rgb/camera_info</cameraInfoTopicName>
+            <depthImageTopicName>depth/image_raw</depthImageTopicName>
+            <depthImageCameraInfoTopicName>depth/camera_info</depthImageCameraInfoTopicName>
+            <pointCloudTopicName>depth/points</pointCloudTopicName>
+          <frameName>asus_camera_depth_optical_frame</frameName>
+    <distortion_k1>-0.02</distortion_k1>
+            <distortion_k2>0.04</distortion_k2>
+            <distortion_k3>-0.06</distortion_k3>
+            <distortion_t1>0.0</distortion_t1>
+            <distortion_t2>0.0</distortion_t2>
+          <pointCloudCutoff>0.01</pointCloudCutoff>
+    <pointCloudCutoffMax>5.0</pointCloudCutoffMax>
+        </plugin>
+      </sensor>
+    </gazebo>
+  </xacro:if>
+  <xacro:if value="$(arg urf)">
+    <gazebo reference="left_urf_link">
        <material>Gazebo/Black</material>
       <sensor type="ray" name="range">
@@ -115,6 +154,6 @@
       </sensor>
     </gazebo>
- </xacro:if>
- <xacro:if value="$(arg lidar)">
+  </xacro:if>
+  <xacro:if value="$(arg lidar)">
     <gazebo reference="laser_link">
       <sensor type="ray" name="head_hokuyo_sensor">
@@ -273,7 +312,25 @@
       </actuator>
     </transmission>
-  <gazebo reference="sr300_link">
-    <material>Gazebo/FlatBlack</material>
-   </gazebo>
+    <xacro:if value="$(arg pan_tilt)">
+      <transmission name="pan_joint_trans">
+        <type>transmission_interface/SimpleTransmission</type>
+        <joint name="pan_joint">
+          <hardwareInterface>PositionJointInterface</hardwareInterface>
+        </joint>
+        <actuator name="pan_joint_motor">
+          <mechanicalReduction>1</mechanicalReduction>
+        </actuator>
+      </transmission>
+      <transmission name="tilt_joint_trans">
+        <type>transmission_interface/SimpleTransmission</type>
+        <joint name="tilt_joint">
+          <hardwareInterface>PositionJointInterface</hardwareInterface>
+        </joint>
+        <actuator name="tilt_joint_motor">
+          <mechanicalReduction>1</mechanicalReduction>
+        </actuator>
+      </transmission>
+    </xacro:if>
+  </xacro:if>
 <gazebo reference="right_urf_link">
     <material>Gazebo/Black</material>
@@ -306,4 +363,12 @@
     <material>Gazebo/FlatBlack</material>
    </gazebo>
+   <xacro:if value="$(arg pan_tilt)">
+     <gazebo reference="asus_camera_link">
+    <material>Gazebo/FlatBlack</material>
+     </gazebo>
+     <gazebo reference="pan_link">
+    <material>Gazebo/Grey</material>
+     </gazebo>
+   </xacro:if>
   <gazebo reference="FR_wheel_link">
   <mu1>1.0</mu1>
@@ -338,4 +403,3 @@
   <maxVel>1.0</maxVel>
 </gazebo>
-</xacro:if>
 </robot>
