Commit message: lizi description

File: robotican_lizi/description/models/lizi.xacro (robot description, xacro)
@@ -1,406 +1,436 @@
-<?xml version="1.0"?>
-<robot xmlns:xacro="http://www.ros.org/wiki/xacro" name="lizi">
-	<xacro:property name="M_PI" value="3.1415926535897931" />
-	<xacro:property name="lizi_color" value="0 0.517 0.26 1" />
-	<xacro:arg name="pan_tilt" default="false"/>
-	<!-- Load all the links  -->
-	<link name="base_link">
-			<inertial>
-				<origin rpy="0 0 0" xyz="-0.036889 0.00027038 0.069426" />
-				<mass value="4.706" />
-				<inertia ixx="0.032024" ixy="0.00038846" ixz="-0.0046108" iyy="0.065583" iyz="2.8552E-06" izz="0.076391" />
-			</inertial>
-			<visual>
-				<origin rpy="0 0 0" xyz="0 0 0" />
-				<geometry>
-					<mesh filename="package://robotican_lizi/description/meshes/base_link.STL" />
-				</geometry>
-				<material name="">
-					<color rgba="${lizi_color}" />
-				</material>
-			</visual>
-			<collision>
-				<origin rpy="0 0 0" xyz="0 0 0" />
-				<geometry>
-					<mesh filename="package://robotican_lizi/description/meshes/base_link.STL" />
-				</geometry>
-			</collision>
-	</link>
-	<link name="fl_wheel_link">
-			<inertial>
-				<origin rpy="0 0 0" xyz="2.9411E-11 -0.0075967 5.8231E-11" />
-				<mass value="0.4084" />
-				<inertia ixx="0.00059356" ixy="3.4979E-14" ixz="-4.6514E-14" iyy="0.0011268" iyz="5.6928E-14" izz="0.00059356" />
-			</inertial>
-			<visual>
-				<origin rpy="0 0 0" xyz="0 0 0" />
-				<geometry>
-					<mesh filename="package://robotican_lizi/description/meshes/fl_wheel_link.STL" />
-				</geometry>
-				<material name="">
-					<color rgba="0.2 0.2 0.2 1" />
-				</material>
-			</visual>
-			<collision>
-				<origin rpy="${M_PI/2} 0 0" xyz="0 0 0" />
-				<geometry>
-<!-- 					<mesh filename="package://robotican_lizi/description/meshes/fl_wheel_link.STL" /> -->
-				  <cylinder  length="0.02" radius="0.065"/>
-				</geometry>
-			</collision>
-	</link>
-	<link name="fr_wheel_link">
-			<inertial>
-				<origin rpy="0 0 0" xyz="-2.9052E-11 0.0035967 5.8411E-11" />
-				<mass value="0.4084" />
-				<inertia ixx="0.00059356" ixy="3.4627E-14" ixz="4.9977E-14" iyy="0.0011268" iyz="-5.7142E-14" izz="0.00059356" />
-			</inertial>
-			<visual>
-				<origin rpy="0 0 0" xyz="0 0 0" />
-				<geometry>
-					<mesh filename="package://robotican_lizi/description/meshes/fr_wheel_link.STL" />
-				</geometry>
-				<material name="">
-					<color rgba="0.2 0.2 0.2 1" />
-				</material>
-			</visual>
-			<collision>
-				<origin rpy="${M_PI/2} 0 0" xyz="0 0 0" />
-				<geometry>
-<!-- 					<mesh filename="package://robotican_lizi/description/meshes/fr_wheel_link.STL" /> -->
-				  <cylinder  length="0.02" radius="0.065"/>
-				</geometry>
-			</collision>
-	</link>
-	<link name="rl_wheel_link">
-			<inertial>
-				<origin rpy="0 0 0" xyz="2.9411E-11 -0.0035967 5.8231E-11" />
-				<mass value="0.4084" />
-				<inertia ixx="0.00059356" ixy="3.4979E-14" ixz="-4.6514E-14" iyy="0.0011268" iyz="5.6928E-14" izz="0.00059356" />
-			</inertial>
-			<visual>
-				<origin rpy="0 0 0" xyz="0 0 0" />
-				<geometry>
-					<mesh filename="package://robotican_lizi/description/meshes/rl_wheel_link.STL" />
-				</geometry>
-				<material name="">
-					<color rgba="0.2 0.2 0.2 1" />
-				</material>
-			</visual>
-			<collision>
-				<origin rpy="${M_PI/2} 0 0" xyz="0 0 0" />
-				<geometry>
-<!-- 					<mesh filename="package://robotican_lizi/description/meshes/rl_wheel_link.STL" /> -->
-				  <cylinder  length="0.02" radius="0.065"/>
-				</geometry>
-			</collision>
-	</link>
-	<link name="rr_wheel_link">
-		<inertial>
-			<origin rpy="0 0 0" xyz="-2.9411E-11 0.0035967 5.8231E-11" />
-			<mass value="0.4084" />
-			<inertia ixx="0.00059356" ixy="3.4979E-14" ixz="4.6514E-14" iyy="0.0011268" iyz="-5.6928E-14" izz="0.00059356" />
-		</inertial>
-		<visual>
-			<origin rpy="0 0 0" xyz="0 0 0" />
-			<geometry>
-				<mesh filename="package://robotican_lizi/description/meshes/rr_wheel_link.STL" />
-			</geometry>
-			<material name="">
-				<color rgba="0.2 0.2 0.2 1" />
-			</material>
-		</visual>
-		<collision>
-			<origin rpy="${M_PI/2} 0 0" xyz="0 0 0" />
-			<geometry>
-<!-- 				<mesh filename="package://robotican_lizi/description/meshes/rr_wheel_link.STL" /> -->
-			  <cylinder  length="0.02" radius="0.065"/>
-			</geometry>
-		</collision>
-  	</link>
-	<link name="right_urf_link">
-		<inertial>
-			<origin rpy="0 0 0" xyz="1.6494E-05 0.012085 -1.486E-07" />
-			<mass value="0.0020317" />
-			<inertia ixx="8.4324E-08" ixy="1.1443E-10" ixz="1.6171E-09" iyy="9.8652E-08" iyz="-1.0309E-12" izz="7.8496E-08" />
-		</inertial>
-		<visual>
-			<origin rpy="0 0 1.57" xyz="0 0 0" />
-			<geometry>
-				<mesh filename="package://robotican_lizi/description/meshes/right_urf_link.STL" />
-			</geometry>
-			<material name="">
-				<color rgba="0.19216 0.11961 0.13333 1" />
-			</material>
-		</visual>
-		<collision>
-			<origin rpy="0 0 0" xyz="0 0 0" />
-			<geometry>
-				<mesh filename="package://robotican_lizi/description/meshes/right_urf_link.STL" />
-			</geometry>
-		</collision>
-	</link>
-	<link name="rear_urf_link">
-		<inertial>
-			<origin rpy="0 0 0" xyz="0.012085 -1.486E-07 1.6494E-05" />
-			<mass value="0.0020317" />
-			<inertia ixx="9.8652E-08" ixy="-1.0309E-12" ixz="1.1443E-10" iyy="7.8496E-08" iyz="1.6171E-09" izz="8.4324E-08" />
-		</inertial>
-		<visual>
-			<origin rpy="0 0 ${M_PI}" xyz="0 0 0" />
-			<geometry>
-				<mesh filename="package://robotican_lizi/description/meshes/rear_urf_link.STL" />
-			</geometry>
-			<material name="">
-				<color rgba="0.19216 0.11961 0.13333 1" />
-			</material>
-		</visual>
-		<collision>
-			<origin rpy="0 0 ${M_PI}" xyz="0 0 0" />
-			<geometry>
-				<mesh filename="package://robotican_lizi/description/meshes/rear_urf_link.STL" />
-			</geometry>
-		</collision>
-	</link>
-	<link name="left_urf_link">
-		<inertial>
-			<origin rpy="0 0 0" xyz="1.6494E-05 -0.012085 1.486E-07" />
-			<mass value="0.0020317" />
-			<inertia ixx="8.4324E-08" ixy="-1.1443E-10" ixz="-1.6171E-09" iyy="9.8652E-08" iyz="-1.0309E-12" izz="7.8496E-08" />
-		</inertial>
-		<visual>
-			<origin rpy="0 0 -1.57" xyz="0 0 0" />
-			<geometry>
-				<mesh filename="package://robotican_lizi/description/meshes/left_urf_link.STL" />
-			</geometry>
-			<material name="">
-				<color rgba="0.19216 0.11961 0.13333 1" />
-			</material>
-		</visual>
-		<collision>
-			<origin rpy="0 0 0" xyz="0 0 0" />
-			<geometry>
-				<mesh filename="package://robotican_lizi/description/meshes/left_urf_link.STL" />
-			</geometry>
-		</collision>
-	</link>
-	<link name="laser_link">
-		<inertial>
-			<origin rpy="0 0 0" xyz="0.00079194 -0.00016941 -0.032844" />
-			<mass value="0.13934" />
-			<inertia ixx="7.4677E-05" ixy="-1.0667E-07" ixz="-9.0925E-07" iyy="7.7824E-05" iyz="5.076E-07" izz="5.1196E-05" />
-		</inertial>
-		<visual>
-			<origin rpy="0 0 ${M_PI}" xyz="0 0 0" />
-			<geometry>
-				<mesh filename="package://robotican_lizi/description/meshes/laser_link.STL" />
-			</geometry>
-			<material name="">
-				<color rgba="0.25294 0.25294 0.25294 1" />
-			</material>
-		</visual>
-		<collision>
-			<origin rpy="0 0 0" xyz="0 0 0" />
-			<geometry>
-				<mesh filename="package://robotican_lizi/description/meshes/laser_link.STL" />
-			</geometry>
-		</collision>
-	</link>
-	<link name="camera_link">
-			<inertial>
-				<origin rpy="0 0 0" xyz="-0.010925 -4.5428E-06 0.00024772" />
-				<mass value="0.033156" />
-				<inertia ixx="9.3903E-06" ixy="-1.4061E-09" ixz="5.0587E-08" iyy="5.845E-06" iyz="-2.4174E-09" izz="5.8692E-06" />
-			</inertial>
-			<visual>
-				<origin rpy="0 0 0" xyz="0 0 0" />
-				<geometry>
-					<mesh filename="package://robotican_lizi/description/meshes/camera_link.STL" />
-				</geometry>
-				<material name="">
-					<color rgba="0.2 0.2 0.2 1" />
-				</material>
-			</visual>
-			<collision>
-				<origin rpy="0 0 0" xyz="0 0 0" />
-				<geometry>
-					<mesh filename="package://robotican_lizi/description/meshes/camera_link.STL" />
-				</geometry>
-			</collision>
-		</link>
-	<xacro:if value="$(arg pan_tilt)">
-		<link name="pan_link">
-			<inertial>
-				<origin rpy="0 0 0" xyz="-0.015533 -0.010751 0.019512" />
-				<mass value="0.016162" />
-				<inertia ixx="5.2781E-06" ixy="1.178E-06" ixz="1.1286E-06" iyy="6.0052E-06" iyz="7.9421E-07" izz="4.7257E-06" />
-			</inertial>
-			<visual>
-				<origin rpy="0 0 0" xyz="0 0 0" />
-				<geometry>
-					<mesh filename="package://robotican_lizi/description/meshes/pan_link.STL" />
-				</geometry>
-				<material name="">
-					<color rgba="0.2 0.2 0.2 1" />
-				</material>
-			</visual>
-			<collision>
-				<origin rpy="0 0 0" xyz="0 0 0" />
-				<geometry>
-					<mesh filename="package://robotican_lizi/description/meshes/pan_link.STL" />
-				</geometry>
-			</collision>
-		</link>
-		<link name="asus_camera_link">
-			<inertial>
-				<origin rpy="0 0 0" xyz="0 0 0" />
-				<mass value="0.14689" />
-				<inertia ixx="0.00037709" ixy="-2.2879E-08" ixz="1.0241E-05" iyy="0.00038351" iyz="1.2981E-08" izz="2.2432E-05" />
-			</inertial>
-			<visual>
-				<origin rpy="${M_PI/2} 0 0" xyz="-0.007 0 0" />
-				<geometry>
-					<mesh filename="package://robotican_lizi/description/meshes/asus_camera_link.STL" />
-				</geometry>
-				<material name="">
-					<color rgba="0.2 0.2 0.2 1" />
-				</material>
-			</visual>
-			<collision>
-				<origin rpy="${M_PI/2} 0 0" xyz="0 0 0" />
-				<geometry>
-					<mesh filename="package://robotican_lizi/description/meshes/asus_camera_link.STL" />
-				</geometry>
-			</collision>
-		</link>
-		  <joint name="asus_rgb_joint" type="fixed">
-      <origin xyz="0 0.022 0" rpy="0 0 0"/>
-      <parent link="asus_camera_link"/>
-      <child link="asus_camera_rgb_frame" />
-    </joint>
-    <link name="asus_camera_rgb_frame">
-      <inertial>
-	<mass value="0.001" />
-	<origin xyz="0 0 0" />
-	<inertia ixx="0.0001" ixy="0.0" ixz="0.0"
-	  iyy="0.0001" iyz="0.0"
-	  izz="0.0001" />
-	</inertial>
-      </link>
-      <joint name="asus_camera_rgb_optical_joint" type="fixed">
-	<origin xyz="0 0 0" rpy="${-M_PI/2} 0 ${-M_PI/2}" />
-	<parent link="asus_camera_rgb_frame" />
-	<child link="asus_camera_rgb_optical_frame" />
-      </joint>
-      <link name="asus_camera_rgb_optical_frame">
-	<inertial>
-	  <mass value="0.001" />
-	  <origin xyz="0 0 0" />
-	  <inertia ixx="0.0001" ixy="0.0" ixz="0.0"
-	    iyy="0.0001" iyz="0.0"
-	    izz="0.0001" />
-	  </inertial>
-	</link>
-	<joint name="asus_camera_depth_joint" type="fixed">
-	  <origin xyz="0 0.049 0" rpy="0 0 0" />
-	  <parent link="asus_camera_link" />
-	  <child link="asus_camera_depth_frame" />
-	</joint>
-	<link name="asus_camera_depth_frame">
-	  <inertial>
-	    <mass value="0.001" />
-	    <origin xyz="0 0 0" />
-	    <inertia ixx="0.0001" ixy="0.0" ixz="0.0"
-	      iyy="0.0001" iyz="0.0"
-	      izz="0.0001" />
-	    </inertial>
-	  </link>
-	  <joint name="asus_camera_depth_optical_joint" type="fixed">
-	    <origin xyz="0 0 0" rpy="${-M_PI/2} 0 ${-M_PI/2}" />
-	    <parent link="asus_camera_depth_frame" />
-	    <child link="asus_camera_depth_optical_frame" />
-	  </joint>
-	  <link name="asus_camera_depth_optical_frame">
-	    <inertial>
-	      <mass value="0.001" />
-	      <origin xyz="0 0 0" />
-	      <inertia ixx="0.0001" ixy="0.0" ixz="0.0"
-		iyy="0.0001" iyz="0.0"
-		izz="0.0001" />
-	      </inertial>
-	    </link>
-	</xacro:if>
-	<!--         END         -->
-	<!-- Load all the joints -->
-	<joint name="fl_wheel_joint" type="continuous">
-    		<origin xyz="0.118 0.1338 0.026" rpy="0 0 -1.3371E-16" />
-    		<parent link="base_link" />
-    		<child link="fl_wheel_link" />
-    		<axis xyz="0 1 0" />
-  	</joint>
-	<joint name="rl_wheel_joint" type="continuous">
-    		<origin xyz="-0.118 0.1338 0.026" rpy="0 0 -6.6853E-16" />
-    		<parent link="base_link" />
-    		<child link="rl_wheel_link" />
-    		<axis xyz="0 1 0" />
-  	</joint>
-	<joint name="rr_wheel_joint" type="continuous">
-    		<origin xyz="-0.118 -0.1338 0.026" rpy="-1.2938E-16 -1.2938E-15 -6.6853E-16" />
-    		<parent link="base_link" />
-    		<child link="rr_wheel_link" />
-    		<axis xyz="0 1 0" />
-  	</joint>
-	<joint name="fr_wheel_joint" type="continuous">
-    		<origin xyz="0.118 -0.1338 0.026" rpy="4.4216E-16 -0.0061583 -2.6824E-16" />
-    		<parent link="base_link" />
-    		<child link="fr_wheel_link" />
-    		<axis xyz="0 1 0" />
-  	</joint>
-	<xacro:if value="$(arg pan_tilt)">
-		<joint name="pan_joint" type="revolute">
-				<origin xyz="0.081249 0 0.092091" rpy="2.1253E-16 8.5011E-16 0" />
-				<parent link="base_link" />
-				<child link="pan_link" />
-				<axis xyz="0 0 1" />
-				<limit upper="0.610865" lower="-0.610865" effort="1.11" velocity="5.3" />
-		</joint>
-		<joint name="tilt_joint" type="revolute">
-				<origin xyz="-0.0004889 -0.00041349 0.08" rpy="0 0 0" />
-				<parent link="pan_link" />
-				<child link="asus_camera_link" />
-				<axis xyz="0 1 0" />
-				<limit upper="0.523599" lower="-0.523599" effort="1.11" velocity="5.3" />
-		</joint>
-	</xacro:if>
-	<joint name="right_urf_joint" type="fixed">
-    		<origin xyz="-0.0074577 -0.11 0.07895" rpy="0 0 ${-M_PI/2}" />
-    		<parent link="base_link" />
-    		<child link="right_urf_link" />
-    		<axis xyz="0 0 0" />
-  	</joint>
-	<joint name="left_urf_joint" type="fixed">
-    		<origin xyz="-0.0074577 0.11 0.07895" rpy="0 0 ${M_PI/2}" />
-    		<parent link="base_link" />
-    		<child link="left_urf_link" />
-    		<axis xyz="0 0 0" />
-  	</joint>
-	<joint name="rear_urf_joint" type="fixed">
-    		<origin xyz="-0.187 0.085 0.093934" rpy="0 0 ${M_PI}" />
-    		<parent link="base_link" />
-    		<child link="rear_urf_link" />
-    		<axis xyz="0 0 0" />
-  	</joint>
-	<joint name="laser_joint" type="fixed">
-    		<origin xyz="0.14276 -1.1564E-05 0.10781" rpy="2.1253E-16 8.5011E-16 -2.6741E-16" />
-    		<parent link="base_link" />
-    		<child link="laser_link" />
-    		<axis xyz="0 0 0" />
-  	</joint>
-	<joint name="camera_joint" type="fixed">
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
Commit message: slip factor

File: robotican_lizi/description/models/lizi.xacro (robot description, xacro)
@@ -1,4 +1,5 @@
-<robot
-  name="robotican_lizi">
+<?xml version="1.0"?>
+<robot xmlns:xacro="http://www.ros.org/wiki/xacro" name="lizi_robot" description="lizi Robot">
+<xacro:property name="M_PI" value="3.1415926535897931"/>
   <link
     name="base_link">
@@ -134,7 +135,7 @@
       </geometry>
       <material
-        name="">
-        <color
-          rgba="0.29804 0.29804 0.29804 1" />
+        name="black">
+        <color
+          rgba="0.0 0.0 0.0 1" />
       </material>
     </visual>
@@ -229,5 +230,5 @@
       <geometry>
         <mesh
-          filename="package://robotican_lizi/description/meshes/FL_wheel_link.STL" />
+          filename="package://robotican_lizi/description/meshes/wheel_link.STL" />
       </geometry>
       <material
@@ -240,8 +241,8 @@
       <origin
         xyz="0 0 0"
-        rpy="0 0 0" />
-      <geometry>
-        <mesh
-          filename="package://robotican_lizi/description/meshes/FL_wheel_link.STL" />
+        rpy="${M_PI/2} 0 0" />
+      <geometry>
+       <!--    <mesh filename="package://robotican_lizi/description/meshes/wheel_link.STL" /> -->
+  <cylinder  length="0.02" radius="0.0762"/>
       </geometry>
     </collision>
@@ -282,5 +283,5 @@
       <geometry>
         <mesh
-          filename="package://robotican_lizi/description/meshes/RL_wheel_link.STL" />
+          filename="package://robotican_lizi/description/meshes/wheel_link.STL" />
       </geometry>
       <material
@@ -293,8 +294,8 @@
       <origin
         xyz="0 0 0"
-        rpy="0 0 0" />
-      <geometry>
-        <mesh
-          filename="package://robotican_lizi/description/meshes/RL_wheel_link.STL" />
+         rpy="${M_PI/2} 0 0" />
+      <geometry>
+       <!--    <mesh filename="package://robotican_lizi/description/meshes/wheel_link.STL" /> -->
+  <cylinder  length="0.02" radius="0.0762"/>
       </geometry>
     </collision>
@@ -335,5 +336,5 @@
       <geometry>
         <mesh
-          filename="package://robotican_lizi/description/meshes/FR_wheel_link.STL" />
+          filename="package://robotican_lizi/description/meshes/wheel_link.STL" />
       </geometry>
       <material
@@ -346,8 +347,8 @@
       <origin
         xyz="0 0 0"
-        rpy="0 0 0" />
-      <geometry>
-        <mesh
-          filename="package://robotican_lizi/description/meshes/FR_wheel_link.STL" />
+     rpy="${M_PI/2} 0 0" />
+      <geometry>
+       <!--    <mesh filename="package://robotican_lizi/description/meshes/wheel_link.STL" /> -->
+  <cylinder  length="0.02" radius="0.0762"/>
       </geometry>
     </collision>
@@ -388,5 +389,5 @@
       <geometry>
         <mesh
-          filename="package://robotican_lizi/description/meshes/RR_wheel_link.STL" />
+          filename="package://robotican_lizi/description/meshes/wheel_link.STL" />
       </geometry>
       <material
@@ -399,8 +400,8 @@
       <origin
         xyz="0 0 0"
-        rpy="0 0 0" />
-      <geometry>
-        <mesh
-          filename="package://robotican_lizi/description/meshes/RR_wheel_link.STL" />
+        rpy="${M_PI/2} 0 0" />
+      <geometry>
+       <!--    <mesh filename="package://robotican_lizi/description/meshes/wheel_link.STL" /> -->
+  <cylinder  length="0.02" radius="0.0762"/>
       </geometry>
     </collision>

File: robotican_lizi/description/models/lizi_gazebo.xacro (robot description, xacro)
@@ -9,47 +9,8 @@
   <xacro:arg name="lidar" default="false"/>
   <xacro:arg name="sr300" default="false"/>
-  <xacro:arg name="pan_tilt" default='false'/>
   <xacro:arg name="asus_hz" default="10.0"/>
   <xacro:property name="URF_FOV" value="${10.0*M_PI/180}" />
-  <xacro:if value="$(arg pan_tilt)">
-    <gazebo reference="asus_camera_rgb_frame">
-      <sensor type="depth" name="asus_camera">
-        <always_on>true</always_on>
-        <update_rate>$(arg asus_hz)</update_rate>
-      <camera>
-        <horizontal_fov>${57.0*M_PI/180.0}</horizontal_fov>
-        <image>
-          <format>R8G8B8</format>
-          <height>640</height>
-          <width>480</width>
-        </image>
-        <clip>
-          <near>0.01</near>
-          <far>5.0</far>
-        </clip>
-      </camera>
-        <plugin name="asus_camera_controller" filename="libgazebo_ros_openni_kinect.so">
-          <cameraName>asus_camera</cameraName>
-          <alwaysOn>true</alwaysOn>
-          <updateRate>$(arg asus_hz)</updateRate>
-            <imageTopicName>rgb/image_raw</imageTopicName>
-            <cameraInfoTopicName>rgb/camera_info</cameraInfoTopicName>
-            <depthImageTopicName>depth/image_raw</depthImageTopicName>
-            <depthImageCameraInfoTopicName>depth/camera_info</depthImageCameraInfoTopicName>
-            <pointCloudTopicName>depth/points</pointCloudTopicName>
-          <frameName>asus_camera_depth_optical_frame</frameName>
-    <distortion_k1>-0.02</distortion_k1>
-            <distortion_k2>0.04</distortion_k2>
-            <distortion_k3>-0.06</distortion_k3>
-            <distortion_t1>0.0</distortion_t1>
-            <distortion_t2>0.0</distortion_t2>
-          <pointCloudCutoff>0.01</pointCloudCutoff>
-    <pointCloudCutoffMax>5.0</pointCloudCutoffMax>
-        </plugin>
-      </sensor>
-    </gazebo>
-  </xacro:if>
-  <xacro:if value="$(arg urf)">
-    <gazebo reference="left_urf_link">
+ <xacro:if value="$(arg urf)">
+      <gazebo reference="left_urf_link">
        <material>Gazebo/Black</material>
       <sensor type="ray" name="range">
@@ -154,6 +115,6 @@
       </sensor>
     </gazebo>
-  </xacro:if>
-  <xacro:if value="$(arg lidar)">
+ </xacro:if>
+ <xacro:if value="$(arg lidar)">
     <gazebo reference="laser_link">
       <sensor type="ray" name="head_hokuyo_sensor">
@@ -312,25 +273,7 @@
       </actuator>
     </transmission>
-    <xacro:if value="$(arg pan_tilt)">
-      <transmission name="pan_joint_trans">
-        <type>transmission_interface/SimpleTransmission</type>
-        <joint name="pan_joint">
-          <hardwareInterface>PositionJointInterface</hardwareInterface>
-        </joint>
-        <actuator name="pan_joint_motor">
-          <mechanicalReduction>1</mechanicalReduction>
-        </actuator>
-      </transmission>
-      <transmission name="tilt_joint_trans">
-        <type>transmission_interface/SimpleTransmission</type>
-        <joint name="tilt_joint">
-          <hardwareInterface>PositionJointInterface</hardwareInterface>
-        </joint>
-        <actuator name="tilt_joint_motor">
-          <mechanicalReduction>1</mechanicalReduction>
-        </actuator>
-      </transmission>
-    </xacro:if>
-  </xacro:if>
+  <gazebo reference="sr300_link">
+    <material>Gazebo/FlatBlack</material>
+   </gazebo>
 <gazebo reference="right_urf_link">
     <material>Gazebo/Black</material>
@@ -363,12 +306,4 @@
     <material>Gazebo/FlatBlack</material>
    </gazebo>
-   <xacro:if value="$(arg pan_tilt)">
-     <gazebo reference="asus_camera_link">
-    <material>Gazebo/FlatBlack</material>
-     </gazebo>
-     <gazebo reference="pan_link">
-    <material>Gazebo/Grey</material>
-     </gazebo>
-   </xacro:if>
   <gazebo reference="FR_wheel_link">
   <mu1>1.0</mu1>
@@ -403,3 +338,4 @@
   <maxVel>1.0</maxVel>
 </gazebo>
+</xacro:if>
 </robot>
