Commit message: lizi modifications

File: robotican_lizi/description/models/lizi.xacro (robot description, xacro)
@@ -9,5 +9,5 @@
         rpy="0 0 0" />
       <mass
-        value="0.47025" />
+        value="20.47025" />
       <inertia
         ixx="0.004176"
@@ -84,5 +84,5 @@
         name="">
         <color
-          rgba="0.75294 0.75294 0.75294 1" />
+          rgba="0.0 0.0 0.0 1" />
       </material>
     </visual>
@@ -235,5 +235,5 @@
         name="">
         <color
-          rgba="0.79216 0.81961 0.93333 1" />
+          rgba="0.0 0.0 0.0 1" />
       </material>
     </visual>
@@ -288,5 +288,5 @@
         name="">
         <color
-          rgba="0.79216 0.81961 0.93333 1" />
+          rgba="0.0 0.0 0.0 1" />
       </material>
     </visual>
@@ -341,5 +341,5 @@
         name="">
         <color
-          rgba="0.79216 0.81961 0.93333 1" />
+          rgba="0.0 0.0 0.0 1" />
       </material>
     </visual>
@@ -394,5 +394,5 @@
         name="">
         <color
-          rgba="0.79216 0.81961 0.93333 1" />
+          rgba="0.0 0.0 0.0 1" />
       </material>
     </visual>

File: robotican_lizi/description/models/lizi_gazebo.xacro (robot description, xacro)
@@ -306,36 +306,48 @@
     <material>Gazebo/FlatBlack</material>
    </gazebo>
-  <gazebo reference="FR_wheel_link">
-  <mu1>1.0</mu1>
-  <mu2>1.0</mu2>
-  <kp>1000000.0</kp>
-  <kd>100.0</kd>
-  <minDepth>0.001</minDepth>
-  <maxVel>1.0</maxVel>
-</gazebo>
-  <gazebo reference="FL_wheel_link">
-  <mu1>1.0</mu1>
-  <mu2>1.0</mu2>
-  <kp>1000000.0</kp>
-  <kd>100.0</kd>
-  <minDepth>0.001</minDepth>
-  <maxVel>1.0</maxVel>
-</gazebo>
-  <gazebo reference="RR_wheel_link">
-  <mu1>1.0</mu1>
-  <mu2>1.0</mu2>
-  <kp>1000000.0</kp>
-  <kd>100.0</kd>
-  <minDepth>0.001</minDepth>
-  <maxVel>1.0</maxVel>
-</gazebo>
-  <gazebo reference="RL_wheel_link">
-  <mu1>1.0</mu1>
-  <mu2>1.0</mu2>
-  <kp>1000000.0</kp>
-  <kd>100.0</kd>
-  <minDepth>0.001</minDepth>
-  <maxVel>1.0</maxVel>
-</gazebo>
+ <gazebo reference="FL_wheel_link">
+    <!-- kp and kd for rubber -->
+    <kp>1000000.0</kp>
+    <kd>100.0</kd>
+    <mu1>1.5</mu1>
+    <mu2>1.5</mu2>
+    <fdir1>1 0 0</fdir1>
+    <maxVel>1.0</maxVel>
+    <minDepth>0.00</minDepth>
+        <material>Gazebo/Black</material>
+  </gazebo>
+   <gazebo reference="FR_wheel_link">
+    <!-- kp and kd for rubber -->
+    <kp>1000000.0</kp>
+    <kd>100.0</kd>
+    <mu1>1.5</mu1>
+    <mu2>1.5</mu2>
+    <fdir1>1 0 0</fdir1>
+    <maxVel>1.0</maxVel>
+    <minDepth>0.00</minDepth>
+        <material>Gazebo/Black</material>
+  </gazebo>
+   <gazebo reference="RL_wheel_link">
+    <!-- kp and kd for rubber -->
+    <kp>1000000.0</kp>
+    <kd>100.0</kd>
+    <mu1>1.5</mu1>
+    <mu2>1.5</mu2>
+    <fdir1>1 0 0</fdir1>
+    <maxVel>1.0</maxVel>
+    <minDepth>0.00</minDepth>
+        <material>Gazebo/Black</material>
+  </gazebo>
+   <gazebo reference="RR_wheel_link">
+    <!-- kp and kd for rubber -->
+    <kp>1000000.0</kp>
+    <kd>100.0</kd>
+    <mu1>1.5</mu1>
+    <mu2>1.5</mu2>
+    <fdir1>1 0 0</fdir1>
+    <maxVel>1.0</maxVel>
+    <minDepth>0.00</minDepth>
+        <material>Gazebo/Black</material>
+  </gazebo>
 </xacro:if>
 </robot>

Commit message: lizi fixes

File: robotican_lizi/description/models/lizi.xacro (robot description, xacro)
@@ -6,8 +6,8 @@
     <inertial>
       <origin
-        xyz="0.0041783 0.0052424 0.04047"
+        xyz="0.0 0.0 0.04047"
         rpy="0 0 0" />
       <mass
-        value="20.47025" />
+        value="5.47025" />
       <inertia
         ixx="0.004176"
@@ -59,18 +59,4 @@
   <link
     name="laser_link">
-    <inertial>
-      <origin
-        xyz="-3.976E-05 0.00016529 -0.022904"
-        rpy="0 0 0" />
-      <mass
-        value="0.13302" />
-      <inertia
-        ixx="6.9591E-05"
-        ixy="-6.1652E-08"
-        ixz="-1.627E-07"
-        iyy="7.0066E-05"
-        iyz="-4.9495E-07"
-        izz="4.5841E-05" />
-    </inertial>
     <visual>
       <origin
@@ -112,18 +98,4 @@
   <link
     name="sr300_link">
-    <inertial>
-      <origin
-        xyz="-0.019521 -4.9406E-07 0.0028518"
-        rpy="0 0 0" />
-      <mass
-        value="0.064787" />
-      <inertia
-        ixx="5.9362E-05"
-        ixy="-6.331E-10"
-        ixz="-5.1662E-06"
-        iyy="2.5368E-05"
-        iyz="4.3621E-11"
-        izz="7.6483E-05" />
-    </inertial>
     <visual>
       <origin
@@ -244,5 +216,5 @@
       <geometry>
        <!--    <mesh filename="package://robotican_lizi/description/meshes/wheel_link.STL" /> -->
-  <cylinder  length="0.02" radius="0.0762"/>
+  <cylinder  length="0.05" radius="0.0762"/>
       </geometry>
     </collision>
@@ -297,5 +269,5 @@
       <geometry>
        <!--    <mesh filename="package://robotican_lizi/description/meshes/wheel_link.STL" /> -->
-  <cylinder  length="0.02" radius="0.0762"/>
+  <cylinder  length="0.05" radius="0.0762"/>
       </geometry>
     </collision>
@@ -350,5 +322,5 @@
       <geometry>
        <!--    <mesh filename="package://robotican_lizi/description/meshes/wheel_link.STL" /> -->
-  <cylinder  length="0.02" radius="0.0762"/>
+  <cylinder  length="0.05" radius="0.0762"/>
       </geometry>
     </collision>
@@ -403,5 +375,5 @@
       <geometry>
        <!--    <mesh filename="package://robotican_lizi/description/meshes/wheel_link.STL" /> -->
-  <cylinder  length="0.02" radius="0.0762"/>
+  <cylinder  length="0.05" radius="0.0762"/>
       </geometry>
     </collision>

Commit message: init branch

File: robotican_lizi/description/models/lizi.xacro (robot description, xacro)
@@ -2,4 +2,5 @@
 <robot xmlns:xacro="http://www.ros.org/wiki/xacro" name="lizi_robot" description="lizi Robot">
 <xacro:property name="M_PI" value="3.1415926535897931"/>
+<xacro:include filename="$(find robotican_common)/models/softkinetic_camera_ds325/model.xacro" />
   <link
     name="base_link">
@@ -97,58 +98,4 @@
   </joint>
   <link
-    name="sr300_link">
-    <visual>
-      <origin
-        xyz="0 0 0"
-        rpy="0 0 0" />
-      <geometry>
-        <mesh
-          filename="package://robotican_lizi/description/meshes/sr300_link.STL" />
-      </geometry>
-      <material
-        name="black">
-        <color
-          rgba="0.0 0.0 0.0 1" />
-      </material>
-    </visual>
-    <collision>
-      <origin
-        xyz="0 0 0"
-        rpy="0 0 0" />
-      <geometry>
-        <mesh
-          filename="package://robotican_lizi/description/meshes/sr300_link.STL" />
-      </geometry>
-    </collision>
-  </link>
-  <joint
-    name="sr300_joint"
-    type="fixed">
-    <origin
-      xyz="0.19382 0 0.10646"
-      rpy="0 0 0" />
-    <parent
-      link="base_link" />
-    <child
-      link="sr300_link" />
-    <axis
-      xyz="0 0 0" />
-  </joint>
-  <link
-    name="left_urf_link" />
-  <joint
-    name="left_urf_joint"
-    type="fixed">
-    <origin
-      xyz="0.014542 0.1055 0.0902"
-      rpy="0 0 1.5708" />
-    <parent
-      link="base_link" />
-    <child
-      link="left_urf_link" />
-    <axis
-      xyz="0 0 0" />
-  </joint>
-  <link
     name="rear_urf_link" />
   <joint
@@ -407,3 +354,6 @@
       xyz="0 0 0" />
   </joint>
+  <sensor_senz3d parent="base_link" name="softkinetic_camera">
+    <origin xyz="0.16122 0.0 0.13223" rpy="0.0 0.0 0.0"/>
+  </sensor_senz3d>
 </robot>

File: robotican_lizi/description/models/lizi_gazebo.xacro (robot description, xacro)
@@ -2,4 +2,5 @@
 <robot xmlns:xacro="http://www.ros.org/wiki/xacro" name="lizi" description="lizi robot">
   <xacro:include filename="$(find robotican_lizi)/description/models/lizi.xacro" />
+  <xacro:include filename="$(find robotican_common)/gazebo/softkinetic_camera_ds325.xacro" />
   <xacro:arg name="controllers" default="true"/>
   <xacro:arg name="urf" default="false"/>
@@ -8,5 +9,5 @@
   <xacro:arg name="front_camera" default="false"/>
   <xacro:arg name="lidar" default="false"/>
-  <xacro:arg name="sr300" default="false"/>
+  <xacro:arg name="depth_camera" default="false"/>
   <xacro:arg name="asus_hz" default="10.0"/>
   <xacro:property name="URF_FOV" value="${10.0*M_PI/180}" />
@@ -230,4 +231,7 @@
       </sensor>
     </gazebo>
+  </xacro:if>
+  <xacro:if value="$(arg depth_camera)">
+	  <xacro:softkinetic_gazebo name="softkinetic_camera_rgb" ros_topic="softkinetic_camera"/>
   </xacro:if>
   <xacro:if value="$(arg controllers)">

Commit message: left urf link fix

File: robotican_lizi/description/models/lizi.xacro (robot description, xacro)
@@ -127,4 +127,19 @@
       xyz="0 0 0" />
   </joint>
+<link
+    name="left_urf_link" />
+  <joint
+    name="left_urf_joint"
+    type="fixed">
+    <origin
+      xyz="0.014542 0.1055 0.0902"
+      rpy="0 0 1.5708" />
+    <parent
+      link="base_link" />
+    <child
+      link="left_urf_link" />
+    <axis
+      xyz="0 0 0" />
+  </joint>
   <link
     name="FL_wheel_link">

Commit message: urf left xacro fix2

File: robotican_lizi/description/models/lizi.xacro (robot description, xacro)
@@ -3,12 +3,14 @@
 <xacro:property name="M_PI" value="3.1415926535897931"/>
 <xacro:include filename="$(find robotican_common)/models/softkinetic_camera_ds325/model.xacro" />
+<robot
+  name="robotican_lizi">
   <link
     name="base_link">
     <inertial>
       <origin
-        xyz="0.0 0.0 0.04047"
-        rpy="0 0 0" />
-      <mass
-        value="5.47025" />
+        xyz="0.0041783 0.0052424 0.04047"
+        rpy="0 0 0" />
+      <mass
+        value="0.47025" />
       <inertia
         ixx="0.004176"
@@ -25,34 +27,34 @@
       <geometry>
         <mesh
-          filename="package://robotican_lizi/description/meshes/base_link.STL" />
-      </geometry>
-      <material
-        name="">
-        <color
-          rgba="0.0 1.0 0.0 1" />
-      </material>
-    </visual>
-    <collision>
-      <origin
-        xyz="0 0 0"
-        rpy="0 0 0" />
-      <geometry>
-        <mesh
-          filename="package://robotican_lizi/description/meshes/base_link.STL" />
-      </geometry>
-    </collision>
-  </link>
-  <link
-    name="base_footprint" />
+          filename="package://robotican_lizi/meshes/base_link.STL" />
+      </geometry>
+      <material
+        name="">
+        <color
+          rgba="0.79216 0.81961 0.93333 1" />
+      </material>
+    </visual>
+    <collision>
+      <origin
+        xyz="0 0 0"
+        rpy="0 0 0" />
+      <geometry>
+        <mesh
+          filename="package://robotican_lizi/meshes/base_link.STL" />
+      </geometry>
+    </collision>
+  </link>
+  <link
+    name="footprint_link" />
   <joint
     name="footprint_joint"
     type="fixed">
     <origin
-      xyz="0 0 0.0762"
-      rpy="0 0 0" />
-    <parent
-      link="base_footprint" />
-    <child
-      link="base_link" />
+      xyz="0 0 -0.0762"
+      rpy="0 0 0" />
+    <parent
+      link="base_link" />
+    <child
+      link="footprint_link" />
     <axis
       xyz="0 0 0" />
@@ -60,25 +62,39 @@
   <link
     name="laser_link">
-    <visual>
-      <origin
-        xyz="0 0 0"
-        rpy="0 0 0" />
-      <geometry>
-        <mesh
-          filename="package://robotican_lizi/description/meshes/laser_link.STL" />
-      </geometry>
-      <material
-        name="">
-        <color
-          rgba="0.0 0.0 0.0 1" />
-      </material>
-    </visual>
-    <collision>
-      <origin
-        xyz="0 0 0"
-        rpy="0 0 0" />
-      <geometry>
-        <mesh
-          filename="package://robotican_lizi/description/meshes/laser_link.STL" />
+    <inertial>
+      <origin
+        xyz="-3.976E-05 0.00016529 -0.022904"
+        rpy="0 0 0" />
+      <mass
+        value="0.13302" />
+      <inertia
+        ixx="6.9591E-05"
+        ixy="-6.1652E-08"
+        ixz="-1.627E-07"
+        iyy="7.0066E-05"
+        iyz="-4.9495E-07"
+        izz="4.5841E-05" />
+    </inertial>
+    <visual>
+      <origin
+        xyz="0 0 0"
+        rpy="0 0 0" />
+      <geometry>
+        <mesh
+          filename="package://robotican_lizi/meshes/laser_link.STL" />
+      </geometry>
+      <material
+        name="">
+        <color
+          rgba="0.75294 0.75294 0.75294 1" />
+      </material>
+    </visual>
+    <collision>
+      <origin
+        xyz="0 0 0"
+        rpy="0 0 0" />
+      <geometry>
+        <mesh
+          filename="package://robotican_lizi/meshes/laser_link.STL" />
       </geometry>
     </collision>
@@ -88,5 +104,5 @@
     type="fixed">
     <origin
-      xyz="0.1495 0 0.079"
+      xyz="0.1495 0 0.069005"
       rpy="0 0 0" />
     <parent
@@ -94,4 +110,72 @@
     <child
       link="laser_link" />
+    <axis
+      xyz="0 0 0" />
+  </joint>
+  <link
+    name="sr300_link">
+    <inertial>
+      <origin
+        xyz="-0.019521 -4.9406E-07 0.0028518"
+        rpy="0 0 0" />
+      <mass
+        value="0.064787" />
+      <inertia
+        ixx="5.9362E-05"
+        ixy="-6.331E-10"
+        ixz="-5.1662E-06"
+        iyy="2.5368E-05"
+        iyz="4.3621E-11"
+        izz="7.6483E-05" />
+    </inertial>
+    <visual>
+      <origin
+        xyz="0 0 0"
+        rpy="0 0 0" />
+      <geometry>
+        <mesh
+          filename="package://robotican_lizi/meshes/sr300_link.STL" />
+      </geometry>
+      <material
+        name="">
+        <color
+          rgba="0.29804 0.29804 0.29804 1" />
+      </material>
+    </visual>
+    <collision>
+      <origin
+        xyz="0 0 0"
+        rpy="0 0 0" />
+      <geometry>
+        <mesh
+          filename="package://robotican_lizi/meshes/sr300_link.STL" />
+      </geometry>
+    </collision>
+  </link>
+  <joint
+    name="sr300_joint"
+    type="fixed">
+    <origin
+      xyz="0.19382 0 0.10646"
+      rpy="0 0 0" />
+    <parent
+      link="base_link" />
+    <child
+      link="sr300_link" />
+    <axis
+      xyz="0 0 0" />
+  </joint>
+  <link
+    name="left_urf_link" />
+  <joint
+    name="left_urf_joint"
+    type="fixed">
+    <origin
+      xyz="0.014542 0.1055 0.0902"
+      rpy="0 0 1.5708" />
+    <parent
+      link="base_link" />
+    <child
+      link="left_urf_link" />
     <axis
       xyz="0 0 0" />
@@ -124,19 +208,4 @@
     <child
       link="right_urf_link" />
-    <axis
-      xyz="0 0 0" />
-  </joint>
-<link
-    name="left_urf_link" />
-  <joint
-    name="left_urf_joint"
-    type="fixed">
-    <origin
-      xyz="0.014542 0.1055 0.0902"
-      rpy="0 0 1.5708" />
-    <parent
-      link="base_link" />
-    <child
-      link="left_urf_link" />
     <axis
       xyz="0 0 0" />
@@ -164,19 +233,19 @@
       <geometry>
         <mesh
-          filename="package://robotican_lizi/description/meshes/wheel_link.STL" />
-      </geometry>
-      <material
-        name="">
-        <color
-          rgba="0.0 0.0 0.0 1" />
-      </material>
-    </visual>
-    <collision>
-      <origin
-        xyz="0 0 0"
-        rpy="${M_PI/2} 0 0" />
-      <geometry>
-       <!--    <mesh filename="package://robotican_lizi/description/meshes/wheel_link.STL" /> -->
-  <cylinder  length="0.05" radius="0.0762"/>
+          filename="package://robotican_lizi/meshes/FL_wheel_link.STL" />
+      </geometry>
+      <material
+        name="">
+        <color
+          rgba="0.79216 0.81961 0.93333 1" />
+      </material>
+    </visual>
+    <collision>
+      <origin
+        xyz="0 0 0"
+        rpy="0 0 0" />
+      <geometry>
+        <mesh
+          filename="package://robotican_lizi/meshes/FL_wheel_link.STL" />
       </geometry>
     </collision>
@@ -217,19 +286,19 @@
       <geometry>
         <mesh
-          filename="package://robotican_lizi/description/meshes/wheel_link.STL" />
-      </geometry>
-      <material
-        name="">
-        <color
-          rgba="0.0 0.0 0.0 1" />
-      </material>
-    </visual>
-    <collision>
-      <origin
-        xyz="0 0 0"
-         rpy="${M_PI/2} 0 0" />
-      <geometry>
-       <!--    <mesh filename="package://robotican_lizi/description/meshes/wheel_link.STL" /> -->
-  <cylinder  length="0.05" radius="0.0762"/>
+          filename="package://robotican_lizi/meshes/RL_wheel_link.STL" />
+      </geometry>
+      <material
+        name="">
+        <color
+          rgba="0.79216 0.81961 0.93333 1" />
+      </material>
+    </visual>
+    <collision>
+      <origin
+        xyz="0 0 0"
+        rpy="0 0 0" />
+      <geometry>
+        <mesh
+          filename="package://robotican_lizi/meshes/RL_wheel_link.STL" />
       </geometry>
     </collision>
@@ -246,5 +315,5 @@
       link="RL_wheel_link" />
     <axis
-      xyz="0 1 0" />
+      xyz="0 -1 0" />
   </joint>
   <link
@@ -270,24 +339,24 @@
       <geometry>
         <mesh
-          filename="package://robotican_lizi/description/meshes/wheel_link.STL" />
-      </geometry>
-      <material
-        name="">
-        <color
-          rgba="0.0 0.0 0.0 1" />
-      </material>
-    </visual>
-    <collision>
-      <origin
-        xyz="0 0 0"
-     rpy="${M_PI/2} 0 0" />
-      <geometry>
-       <!--    <mesh filename="package://robotican_lizi/description/meshes/wheel_link.STL" /> -->
-  <cylinder  length="0.05" radius="0.0762"/>
-      </geometry>
-    </collision>
-  </link>
-  <joint
-    name="FR_wheel_joint"
+          filename="package://robotican_lizi/meshes/FR_wheel_link.STL" />
+      </geometry>
+      <material
+        name="">
+        <color
+          rgba="0.79216 0.81961 0.93333 1" />
+      </material>
+    </visual>
+    <collision>
+      <origin
+        xyz="0 0 0"
+        rpy="0 0 0" />
+      <geometry>
+        <mesh
+          filename="package://robotican_lizi/meshes/FR_wheel_link.STL" />
+      </geometry>
+    </collision>
+  </link>
+  <joint
+    name="FR_wheell_joint"
     type="continuous">
     <origin
@@ -323,19 +392,19 @@
       <geometry>
         <mesh
-          filename="package://robotican_lizi/description/meshes/wheel_link.STL" />
-      </geometry>
-      <material
-        name="">
-        <color
-          rgba="0.0 0.0 0.0 1" />
-      </material>
-    </visual>
-    <collision>
-      <origin
-        xyz="0 0 0"
-        rpy="${M_PI/2} 0 0" />
-      <geometry>
-       <!--    <mesh filename="package://robotican_lizi/description/meshes/wheel_link.STL" /> -->
-  <cylinder  length="0.05" radius="0.0762"/>
+          filename="package://robotican_lizi/meshes/RR_wheel_link.STL" />
+      </geometry>
+      <material
+        name="">
+        <color
+          rgba="0.79216 0.81961 0.93333 1" />
+      </material>
+    </visual>
+    <collision>
+      <origin
+        xyz="0 0 0"
+        rpy="0 0 0" />
+      <geometry>
+        <mesh
+          filename="package://robotican_lizi/meshes/RR_wheel_link.STL" />
       </geometry>
     </collision>
@@ -352,5 +421,5 @@
       link="RR_wheel_link" />
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