Commit message: Update lizi.xacro

File: robotican_lizi/description/models/lizi.xacro (robot description, xacro)
@@ -7,8 +7,8 @@
     <inertial>
       <origin
-        xyz="0.0041783 0.0052424 0.04047"
-        rpy="0 0 0" />
-      <mass
-        value="0.47025" />
+        xyz="0.0 0.0 0.04047"
+        rpy="0 0 0" />
+      <mass
+        value="5.47025" />
       <inertia
         ixx="0.004176"
@@ -25,34 +25,34 @@
       <geometry>
         <mesh
-          filename="package://robotican_lizi/meshes/base_link.STL" />
-      </geometry>
-      <material
-        name="">
-        <color
-          rgba="0.79216 0.81961 0.93333 1" />
-      </material>
-    </visual>
-    <collision>
-      <origin
-        xyz="0 0 0"
-        rpy="0 0 0" />
-      <geometry>
-        <mesh
-          filename="package://robotican_lizi/meshes/base_link.STL" />
-      </geometry>
-    </collision>
-  </link>
-  <link
-    name="footprint_link" />
+          filename="package://robotican_lizi/description/meshes/base_link.STL" />
+      </geometry>
+      <material
+        name="">
+        <color
+          rgba="0.0 1.0 0.0 1" />
+      </material>
+    </visual>
+    <collision>
+      <origin
+        xyz="0 0 0"
+        rpy="0 0 0" />
+      <geometry>
+        <mesh
+          filename="package://robotican_lizi/description/meshes/base_link.STL" />
+      </geometry>
+    </collision>
+  </link>
+  <link
+    name="base_footprint" />
   <joint
     name="footprint_joint"
     type="fixed">
     <origin
-      xyz="0 0 -0.0762"
-      rpy="0 0 0" />
-    <parent
-      link="base_link" />
-    <child
-      link="footprint_link" />
+      xyz="0 0 0.0762"
+      rpy="0 0 0" />
+    <parent
+      link="base_footprint" />
+    <child
+      link="base_link" />
     <axis
       xyz="0 0 0" />
@@ -60,39 +60,25 @@
   <link
     name="laser_link">
-    <inertial>
-      <origin
-        xyz="-3.976E-05 0.00016529 -0.022904"
-        rpy="0 0 0" />
-      <mass
-        value="0.13302" />
-      <inertia
-        ixx="6.9591E-05"
-        ixy="-6.1652E-08"
-        ixz="-1.627E-07"
-        iyy="7.0066E-05"
-        iyz="-4.9495E-07"
-        izz="4.5841E-05" />
-    </inertial>
-    <visual>
-      <origin
-        xyz="0 0 0"
-        rpy="0 0 0" />
-      <geometry>
-        <mesh
-          filename="package://robotican_lizi/meshes/laser_link.STL" />
-      </geometry>
-      <material
-        name="">
-        <color
-          rgba="0.75294 0.75294 0.75294 1" />
-      </material>
-    </visual>
-    <collision>
-      <origin
-        xyz="0 0 0"
-        rpy="0 0 0" />
-      <geometry>
-        <mesh
-          filename="package://robotican_lizi/meshes/laser_link.STL" />
+    <visual>
+      <origin
+        xyz="0 0 0"
+        rpy="0 0 0" />
+      <geometry>
+        <mesh
+          filename="package://robotican_lizi/description/meshes/laser_link.STL" />
+      </geometry>
+      <material
+        name="">
+        <color
+          rgba="0.0 0.0 0.0 1" />
+      </material>
+    </visual>
+    <collision>
+      <origin
+        xyz="0 0 0"
+        rpy="0 0 0" />
+      <geometry>
+        <mesh
+          filename="package://robotican_lizi/description/meshes/laser_link.STL" />
       </geometry>
     </collision>
@@ -102,5 +88,5 @@
     type="fixed">
     <origin
-      xyz="0.1495 0 0.069005"
+      xyz="0.1495 0 0.079"
       rpy="0 0 0" />
     <parent
@@ -112,57 +98,19 @@
   </joint>
   <link
-    name="sr300_link">
-    <inertial>
-      <origin
-        xyz="-0.019521 -4.9406E-07 0.0028518"
-        rpy="0 0 0" />
-      <mass
-        value="0.064787" />
-      <inertia
-        ixx="5.9362E-05"
-        ixy="-6.331E-10"
-        ixz="-5.1662E-06"
-        iyy="2.5368E-05"
-        iyz="4.3621E-11"
-        izz="7.6483E-05" />
-    </inertial>
-    <visual>
-      <origin
-        xyz="0 0 0"
-        rpy="0 0 0" />
-      <geometry>
-        <mesh
-          filename="package://robotican_lizi/meshes/sr300_link.STL" />
-      </geometry>
-      <material
-        name="">
-        <color
-          rgba="0.29804 0.29804 0.29804 1" />
-      </material>
-    </visual>
-    <collision>
-      <origin
-        xyz="0 0 0"
-        rpy="0 0 0" />
-      <geometry>
-        <mesh
-          filename="package://robotican_lizi/meshes/sr300_link.STL" />
-      </geometry>
-    </collision>
-  </link>
-  <joint
-    name="sr300_joint"
-    type="fixed">
-    <origin
-      xyz="0.19382 0 0.10646"
-      rpy="0 0 0" />
-    <parent
-      link="base_link" />
-    <child
-      link="sr300_link" />
-    <axis
-      xyz="0 0 0" />
-  </joint>
-  <link
+    name="rear_urf_link" />
+  <joint
+    name="rear_urf_joint"
+    type="fixed">
+    <origin
+      xyz="-0.18 0 0.0902"
+      rpy="0 0 3.1416" />
+    <parent
+      link="base_link" />
+    <child
+      link="rear_urf_link" />
+    <axis
+      xyz="0 0 0" />
+  </joint>
+<link
     name="left_urf_link" />
   <joint
@@ -176,19 +124,4 @@
     <child
       link="left_urf_link" />
-    <axis
-      xyz="0 0 0" />
-  </joint>
-  <link
-    name="rear_urf_link" />
-  <joint
-    name="rear_urf_joint"
-    type="fixed">
-    <origin
-      xyz="-0.18 0 0.0902"
-      rpy="0 0 3.1416" />
-    <parent
-      link="base_link" />
-    <child
-      link="rear_urf_link" />
     <axis
       xyz="0 0 0" />
@@ -231,19 +164,19 @@
       <geometry>
         <mesh
-          filename="package://robotican_lizi/meshes/FL_wheel_link.STL" />
-      </geometry>
-      <material
-        name="">
-        <color
-          rgba="0.79216 0.81961 0.93333 1" />
-      </material>
-    </visual>
-    <collision>
-      <origin
-        xyz="0 0 0"
-        rpy="0 0 0" />
-      <geometry>
-        <mesh
-          filename="package://robotican_lizi/meshes/FL_wheel_link.STL" />
+          filename="package://robotican_lizi/description/meshes/wheel_link.STL" />
+      </geometry>
+      <material
+        name="">
+        <color
+          rgba="0.0 0.0 0.0 1" />
+      </material>
+    </visual>
+    <collision>
+      <origin
+        xyz="0 0 0"
+        rpy="${M_PI/2} 0 0" />
+      <geometry>
+       <!--    <mesh filename="package://robotican_lizi/description/meshes/wheel_link.STL" /> -->
+  <cylinder  length="0.05" radius="0.0762"/>
       </geometry>
     </collision>
@@ -284,19 +217,19 @@
       <geometry>
         <mesh
-          filename="package://robotican_lizi/meshes/RL_wheel_link.STL" />
-      </geometry>
-      <material
-        name="">
-        <color
-          rgba="0.79216 0.81961 0.93333 1" />
-      </material>
-    </visual>
-    <collision>
-      <origin
-        xyz="0 0 0"
-        rpy="0 0 0" />
-      <geometry>
-        <mesh
-          filename="package://robotican_lizi/meshes/RL_wheel_link.STL" />
+          filename="package://robotican_lizi/description/meshes/wheel_link.STL" />
+      </geometry>
+      <material
+        name="">
+        <color
+          rgba="0.0 0.0 0.0 1" />
+      </material>
+    </visual>
+    <collision>
+      <origin
+        xyz="0 0 0"
+         rpy="${M_PI/2} 0 0" />
+      <geometry>
+       <!--    <mesh filename="package://robotican_lizi/description/meshes/wheel_link.STL" /> -->
+  <cylinder  length="0.05" radius="0.0762"/>
       </geometry>
     </collision>
@@ -313,5 +246,5 @@
       link="RL_wheel_link" />
     <axis
-      xyz="0 -1 0" />
+      xyz="0 1 0" />
   </joint>
   <link
@@ -337,24 +270,24 @@
       <geometry>
         <mesh
-          filename="package://robotican_lizi/meshes/FR_wheel_link.STL" />
-      </geometry>
-      <material
-        name="">
-        <color
-          rgba="0.79216 0.81961 0.93333 1" />
-      </material>
-    </visual>
-    <collision>
-      <origin
-        xyz="0 0 0"
-        rpy="0 0 0" />
-      <geometry>
-        <mesh
-          filename="package://robotican_lizi/meshes/FR_wheel_link.STL" />
-      </geometry>
-    </collision>
-  </link>
-  <joint
-    name="FR_wheell_joint"
+          filename="package://robotican_lizi/description/meshes/wheel_link.STL" />
+      </geometry>
+      <material
+        name="">
+        <color
+          rgba="0.0 0.0 0.0 1" />
+      </material>
+    </visual>
+    <collision>
+      <origin
+        xyz="0 0 0"
+     rpy="${M_PI/2} 0 0" />
+      <geometry>
+       <!--    <mesh filename="package://robotican_lizi/description/meshes/wheel_link.STL" /> -->
+  <cylinder  length="0.05" radius="0.0762"/>
+      </geometry>
+    </collision>
+  </link>
+  <joint
+    name="FR_wheel_joint"
     type="continuous">
     <origin
@@ -390,19 +323,19 @@
       <geometry>
         <mesh
-          filename="package://robotican_lizi/meshes/RR_wheel_link.STL" />
-      </geometry>
-      <material
-        name="">
-        <color
-          rgba="0.79216 0.81961 0.93333 1" />
-      </material>
-    </visual>
-    <collision>
-      <origin
-        xyz="0 0 0"
-        rpy="0 0 0" />
-      <geometry>
-        <mesh
-          filename="package://robotican_lizi/meshes/RR_wheel_link.STL" />
+          filename="package://robotican_lizi/description/meshes/wheel_link.STL" />
+      </geometry>
+      <material
+        name="">
+        <color
+          rgba="0.0 0.0 0.0 1" />
+      </material>
+    </visual>
+    <collision>
+      <origin
+        xyz="0 0 0"
+        rpy="${M_PI/2} 0 0" />
+      <geometry>
+       <!--    <mesh filename="package://robotican_lizi/description/meshes/wheel_link.STL" /> -->
+  <cylinder  length="0.05" radius="0.0762"/>
       </geometry>
     </collision>
@@ -419,5 +352,5 @@
       link="RR_wheel_link" />
     <axis
-      xyz="0 -1 0" />
+      xyz="0 1 0" />
   </joint>
   <link

Commit message: lizi xacro

File: robotican_lizi/description/models/lizi.xacro (robot description, xacro)
@@ -112,4 +112,19 @@
       xyz="0 0 0" />
   </joint>
+<link
+    name="left_urf_link" />
+  <joint
+    name="left_urf_joint"
+    type="fixed">
+    <origin
+      xyz="0.014542 0.1055 0.0902"
+      rpy="0 0 1.5708" />
+    <parent
+      link="base_link" />
+    <child
+      link="left_urf_link" />
+    <axis
+      xyz="0 0 0" />
+  </joint>
   <link
     name="right_urf_link" />

Commit message: fixing lizi errors, deleting robotican_gui

File: robotican_lizi/description/models/lizi.xacro (robot description, xacro)
@@ -369,6 +369,3 @@
       xyz="0 0 0" />
   </joint>
-  <sensor_senz3d parent="base_link" name="softkinetic_camera">
-    <origin xyz="0.16122 0.0 0.13223" rpy="0.0 0.0 0.0"/>
-  </sensor_senz3d>
 </robot>
