Commit message: fixes

File: robotican_common/gazebo/sr300.xacro (robot description, xacro)
@@ -1,4 +1,29 @@
+<?xml version="1.0"?>
 <robot xmlns:xacro="http://www.ros.org/wiki/xacro" name="SR300" description="SR300 sensor">
  	<xacro:arg name="sr300_hz" default="10.0"/>
+<link name="sr300_rgb_frame" />
+		<joint name="sr300_rgb_joint" type="fixed">
+		  <origin xyz="0 0 0" rpy="0 0 0" />
+		  <parent link="sr300_link" />
+		  <child link="sr300_rgb_frame" />
+		</joint>
+		 <link name="sr300_rgb_optical_frame" />
+		<joint name="sr300_rgb_optical_joint" type="fixed">
+		  <origin xyz="0 0 0" rpy="${-M_PI/2} 0 ${-M_PI/2}" />
+		  <parent link="sr300_rgb_frame" />
+		  <child link="sr300_rgb_optical_frame" />
+		</joint>
+		<link name="sr300_depth_frame" />
+		<joint name="sr300_depth_joint" type="fixed">
+		  <origin xyz="0 -0.0257 0" rpy="0 0 0" />
+		  <parent link="sr300_link" />
+		  <child link="sr300_depth_frame" />
+		</joint>
+		<link name="sr300_depth_optical_frame" />
+		<joint name="sr300_depth_optical_joint" type="fixed">
+		  <origin xyz="0 0 0" rpy="${-M_PI/2} 0 ${-M_PI/2}" />
+		  <parent link="sr300_depth_frame" />
+		  <child link="sr300_depth_optical_frame" />
+		</joint>
 	<gazebo reference="sr300_rgb_frame">
 		<sensor type="depth" name="sr300">
@@ -6,5 +31,6 @@
 			<update_rate>$(arg sr300_hz)</update_rate>
 			<camera>
-				<horizontal_fov>1.20772254</horizontal_fov>
+				<horizontal_fov>1.18682</horizontal_fov>
+				<!-- <vetrical_fov>0.9424</vetrical_fov> -->
 				<image>
 					<format>B8G8R8</format>
@@ -13,6 +39,6 @@
 				</image>
 				<clip>
-					<near>0.1</near>
-					<far>1.2</far>
+					<near>0.05</near>
+					<far>1.5</far>
 				</clip>
 			</camera>

File: robotican_manipulator_h/models/manipulator_h.xacro (robot description, xacro)
@@ -567,27 +567,3 @@
       xyz="0 0 0" />
   </joint>
-  		<link name="sr300_rgb_frame" />
-		<joint name="sr300_rgb_joint" type="fixed">
-		  <origin xyz="0 0 0" rpy="0 0 0" />
-		  <parent link="sr300_link" />
-		  <child link="sr300_rgb_frame" />
-		</joint>
-		 <link name="sr300_rgb_optical_frame" />
-		<joint name="sr300_rgb_optical_joint" type="fixed">
-		  <origin xyz="0 0 0" rpy="${-M_PI/2} 0 ${-M_PI/2}" />
-		  <parent link="sr300_rgb_frame" />
-		  <child link="sr300_rgb_optical_frame" />
-		</joint>
-		<link name="sr300_depth_frame" />
-		<joint name="sr300_depth_joint" type="fixed">
-		  <origin xyz="0 -0.0235 0" rpy="0 0 0" />
-		  <parent link="sr300_link" />
-		  <child link="sr300_depth_frame" />
-		</joint>
-		<link name="sr300_depth_optical_frame" />
-		<joint name="sr300_depth_optical_joint" type="fixed">
-		  <origin xyz="0 0 0" rpy="${-M_PI/2} 0 ${-M_PI/2}" />
-		  <parent link="sr300_depth_frame" />
-		  <child link="sr300_depth_optical_frame" />
-		</joint>
 </robot>
