Commit message: trying to fix model

File: robotican_common/models/softkinetic_camera_ds325/model.xacro (robot description, xacro)
@@ -1,4 +1,4 @@
 <robot xmlns:xacro="http://www.ros.org/wiki/xacro" name="lizi_robot" description="lizi Robot">
-  <xacro:macro name="sensor_senz3d" params="parent name *origin">
+  <xacro:macro name="sensor_senz3d" params="parent name *origin v_offset_x v_offset_y v_offset_z">
       <joint name="${name}_joint" type="fixed">
         <insert_block name="origin"/>
@@ -8,5 +8,5 @@
       <link name="${name}_link">
         <visual>
-          <origin xyz="-0.01 0.0 0.0" rpy="${-M_PI/2} -${M_PI} ${-M_PI/2}"/>
+          <origin xyz="${-0.01-v_offset_x} ${0.0-v_offset_y} ${0.0-v_offset_z}" rpy="${-M_PI/2} -${M_PI} ${-M_PI/2}"/>
           <geometry>
             <!-- As we don't have a Senz3D mesh, use a deformed Asus Xtion Pro instead -->
@@ -16,5 +16,5 @@
         </visual>
         <collision>
-          <origin xyz="-0.01 0.0 0.0" rpy="0 0 0"/>
+          <origin xyz="${-0.01-v_offset_x} ${0.0-v_offset_y} ${0.0-v_offset_z}" rpy="0 0 0"/>
           <geometry>
           <box size="0.04 0.11 0.04"/>

File: robotican_manipulator_h/models/manipulator_h.xacro (robot description, xacro)
@@ -570,6 +570,6 @@
   </joint>
 -->
-  <sensor_senz3d parent="wrist_link" name="softkinetic_camera">
-    <origin xyz="-0.05905 0 0.0303" rpy="0.0 -${M_PI/2} 0.0"/>
+  <sensor_senz3d parent="wrist_link" name="softkinetic_camera" v_offset_x="0.035" v_offset_y="0.0" v_offset_z="0.0">
+    <origin xyz="-0.05905 0 0.0653" rpy="0.0 -${M_PI/2} 0.0"/>
   </sensor_senz3d>
 </robot>
