Commit message: komodo

File: robotican_komodo/description/models/komodo.xacro (robot description, xacro)
@@ -1,4 +1,4 @@
 <?xml version="1.0"?>
-	<robot xmlns:xacro="http://www.ros.org/wiki/xacro" name="armadillo_robot" description="ARMadillo Robot">
+	<robot xmlns:xacro="http://www.ros.org/wiki/xacro" name="komodo_robot" description="Komodo Robot">
 	<xacro:property name="M_PI" value="3.1415926535897931" />
 	<!--    BASE      -->
@@ -8,5 +8,5 @@
 	<xacro:include filename="$(find robotican_manipulator_h)/models/manipulator_h.xacro" />
 	<!--      END          -->
-<link
+ <link
     name="arm_link">
     <inertial>
@@ -15,12 +15,12 @@
         rpy="0 0 0" />
       <mass
-        value="1.3188" />
+        value="0.16757" />
       <inertia
-        ixx="0.0049508"
-        ixy="-6.559E-09"
-        ixz="-0.0011709"
-        iyy="0.0084361"
-        iyz="1.3268E-08"
-        izz="0.010567" />
+        ixx="0.00062908"
+        ixy="-8.3342E-10"
+        ixz="-0.00014877"
+        iyy="0.0010719"
+        iyz="1.6859E-09"
+        izz="0.0013427" />
     </inertial>
     <visual>
@@ -35,5 +35,5 @@
         name="">
         <color
-          rgba="0.27843 0.2902 0.31765 1" />
+          rgba="0.79216 0.81961 0.93333 1" />
       </material>
     </visual>
@@ -53,5 +53,5 @@
     <origin
       xyz="-0.11925 0 0.16716"
-      rpy="9.68E-16 -2.5959E-15 -1.3587E-14" />
+      rpy="0 0 0" />
     <parent
       link="base_link" />
@@ -62,9 +62,8 @@
   </joint>
 	<joint name="base_arm_joint" type="fixed">
-		<origin xyz="0.033 0 0.03575" rpy="0 0 0" />
+		<origin xyz="-0.091 0 0.093" rpy="0 0 0" />
 		<parent link="arm_link" />
 		<child link="base_arm_link" />
 		<axis xyz="0 0 0" />
 	</joint>
-	<!--      END          -->
 </robot>

File: robotican_komodo/description/models/komodo_base.xacro (robot description, xacro)
@@ -1,20 +1,20 @@
 <?xml version="1.0"?>
 <robot
-  name="Komodo_base">
+  name="robotican_komodo">
   <link
     name="base_link">
     <inertial>
       <origin
-        xyz="-0.029184 -0.0003442 0.0086835"
-        rpy="0 0 0" />
-      <mass
-        value="0.87157" />
-      <inertia
-        ixx="0.012492"
-        ixy="7.0693E-05"
-        ixz="-0.0019088"
-        iyy="0.027664"
-        iyz="-1.6685E-05"
-        izz="0.036797" />
+        xyz="0.0030152 0.00057861 0.0749"
+        rpy="0 0 0" />
+      <mass
+        value="2.0058" />
+      <inertia
+        ixx="0.025582"
+        ixy="0.0010034"
+        ixz="-0.0041152"
+        iyy="0.086418"
+        iyz="-3.8058E-05"
+        izz="0.091994" />
     </inertial>
     <visual>
@@ -43,7 +43,7 @@
   </link>
   <link
-    name="base_footprint_link" />
-  <joint
-    name="base_footprint_joint"
+    name="base_footprint" />
+  <joint
+    name="footprint_joint"
     type="fixed">
     <origin
@@ -53,7 +53,113 @@
       link="base_link" />
     <child
-      link="base_footprint_link" />
-    <axis
-      xyz="0 0 0" />
+      link="base_footprint" />
+    <axis
+      xyz="0 0 0" />
+  </joint>
+  <link
+    name="RL_wheel_link">
+    <inertial>
+      <origin
+        xyz="9.8684E-07 -9.3003E-05 -1.8753E-05"
+        rpy="0 0 0" />
+      <mass
+        value="2.6829" />
+      <inertia
+        ixx="0.012758"
+        ixy="8.7952E-09"
+        ixz="-1.0406E-07"
+        iyy="0.023277"
+        iyz="2.0115E-06"
+        izz="0.012755" />
+    </inertial>
+    <visual>
+      <origin
+        xyz="0 0 0"
+        rpy="0 0 0" />
+      <geometry>
+        <mesh
+          filename="package://robotican_komodo/description/meshes/wheel_link.STL" />
+      </geometry>
+      <material
+        name="">
+        <color
+          rgba="0.79216 0.81961 0.93333 1" />
+      </material>
+    </visual>
+    <collision>
+      <origin
+        xyz="0 0 0"
+        rpy="${M_PI/2} 0 0" />
+      <geometry>
+	<!--  <mesh filename="package://robotican_komodo/description/meshes/wheel_link.STL" /> -->
+	  <cylinder  length="0.05" radius="0.127"/>
+      </geometry>
+    </collision>
+  </link>
+  <joint
+    name="RL_wheel_joint"
+    type="continuous">
+    <origin
+      xyz="-0.165 0.18955 0"
+      rpy="0 0 0" />
+    <parent
+      link="base_link" />
+    <child
+      link="RL_wheel_link" />
+    <axis
+      xyz="0 1 0" />
+  </joint>
+  <link
+    name="FL_wheel_link">
+    <inertial>
+      <origin
+        xyz="9.8687E-07 -9.3003E-05 -1.8753E-05"
+        rpy="0 0 0" />
+      <mass
+        value="2.6829" />
+      <inertia
+        ixx="0.012758"
+        ixy="8.7932E-09"
+        ixz="-1.0406E-07"
+        iyy="0.023277"
+        iyz="2.0115E-06"
+        izz="0.012755" />
+    </inertial>
+    <visual>
+      <origin
+        xyz="0 0 0"
+        rpy="0 0 0" />
+      <geometry>
+        <mesh
+          filename="package://robotican_komodo/description/meshes/wheel_link.STL" />
+      </geometry>
+      <material
+        name="">
+        <color
+          rgba="0.79216 0.81961 0.93333 1" />
+      </material>
+    </visual>
+    <collision>
+      <origin
+        xyz="0 0 0"
+        rpy="${M_PI/2} 0 0" />
+      <geometry>
+	<!--  <mesh filename="package://robotican_komodo/description/meshes/wheel_link.STL" /> -->
+	  <cylinder  length="0.05" radius="0.127"/>
+      </geometry>
+    </collision>
+  </link>
+  <joint
+    name="FL_wheel_joint"
+    type="continuous">
+    <origin
+      xyz="0.165 0.18955 0"
+      rpy="0 0 0" />
+    <parent
+      link="base_link" />
+    <child
+      link="FL_wheel_link" />
+    <axis
+      xyz="0 1 0" />
   </joint>
   <link
@@ -61,37 +167,37 @@
     <inertial>
       <origin
-        xyz="1.2974E-05 -0.00017781 -1.1646E-05"
-        rpy="0 0 0" />
-      <mass
-        value="3.5882" />
-      <inertia
-        ixx="0.016234"
-        ixy="1.9586E-06"
-        ixz="-1.7465E-06"
-        iyy="0.029573"
-        iyz="-1.5657E-06"
-        izz="0.016234" />
-    </inertial>
-    <visual>
-      <origin
-        xyz="0 0 0"
-        rpy="0 0 1.57" />
-      <geometry>
-        <mesh
-          filename="package://robotican_komodo/description/meshes/RR_wheel_link.STL" />
-      </geometry>
-      <material
-        name="">
-        <color
-          rgba="0.75294 0.75294 0.75294 1" />
-      </material>
-    </visual>
-    <collision>
-      <origin
-        xyz="0 0 0"
-        rpy="0 0 0" />
-      <geometry>
-        <mesh
-          filename="package://robotican_komodo/description/meshes/RR_wheel_link.STL" />
+        xyz="-9.8675E-07 9.3004E-05 -1.8753E-05"
+        rpy="0 0 0" />
+      <mass
+        value="2.6829" />
+      <inertia
+        ixx="0.012758"
+        ixy="8.801E-09"
+        ixz="1.0405E-07"
+        iyy="0.023277"
+        iyz="-2.0115E-06"
+        izz="0.012755" />
+    </inertial>
+    <visual>
+      <origin
+        xyz="0 0 0"
+        rpy="0 0 0" />
+      <geometry>
+        <mesh
+          filename="package://robotican_komodo/description/meshes/wheel_link.STL" />
+      </geometry>
+      <material
+        name="">
+        <color
+          rgba="0.79216 0.81961 0.93333 1" />
+      </material>
+    </visual>
+    <collision>
+      <origin
+        xyz="0 0 0"
+        rpy="${M_PI/2} 0 0" />
+      <geometry>
+	<!--  <mesh filename="package://robotican_komodo/description/meshes/wheel_link.STL" /> -->
+	  <cylinder  length="0.05" radius="0.127"/>
       </geometry>
     </collision>
@@ -101,5 +207,5 @@
     type="continuous">
     <origin
-      xyz="-0.165 -0.1893 0"
+      xyz="-0.165 -0.18955 0"
       rpy="0 0 0" />
     <parent
@@ -111,93 +217,40 @@
   </joint>
   <link
-    name="RL_wheel_link">
-    <inertial>
-      <origin
-        xyz="-1.2974E-05 0.00017781 -1.1646E-05"
-        rpy="0 0 0" />
-      <mass
-        value="3.5882" />
-      <inertia
-        ixx="0.016234"
-        ixy="1.9586E-06"
-        ixz="1.7465E-06"
-        iyy="0.029573"
-        iyz="1.5657E-06"
-        izz="0.016234" />
-    </inertial>
-    <visual>
-      <origin
-        xyz="0 0 0"
-        rpy="0 0 1.57" />
-      <geometry>
-        <mesh
-          filename="package://robotican_komodo/description/meshes/RL_wheel_link.STL" />
-      </geometry>
-      <material
-        name="">
-        <color
-          rgba="0.75294 0.75294 0.75294 1" />
-      </material>
-    </visual>
-    <collision>
-      <origin
-        xyz="0 0 0"
-        rpy="0 0 0" />
-      <geometry>
-        <mesh
-          filename="package://robotican_komodo/description/meshes/RL_wheel_link.STL" />
-      </geometry>
-    </collision>
-  </link>
-  <joint
-    name="RL_wheel_joint"
-    type="continuous">
-    <origin
-      xyz="-0.165 0.1893 0"
-      rpy="0 0 0" />
-    <parent
-      link="base_link" />
-    <child
-      link="RL_wheel_link" />
-    <axis
-      xyz="0 1 0" />
-  </joint>
-  <link
     name="FR_wheel_link">
     <inertial>
       <origin
-        xyz="1.2974E-05 -0.00017781 -1.1646E-05"
-        rpy="0 0 0" />
-      <mass
-        value="3.5882" />
-      <inertia
-        ixx="0.016234"
-        ixy="1.9586E-06"
-        ixz="-1.7465E-06"
-        iyy="0.029573"
-        iyz="-1.5657E-06"
-        izz="0.016234" />
-    </inertial>
-    <visual>
-      <origin
-        xyz="0 0 0"
-        rpy="0 0 1.57" />
-      <geometry>
-        <mesh
-          filename="package://robotican_komodo/description/meshes/FR_wheel_link.STL" />
-      </geometry>
-      <material
-        name="">
-        <color
-          rgba="0.75294 0.75294 0.75294 1" />
-      </material>
-    </visual>
-    <collision>
-      <origin
-        xyz="0 0 0"
-        rpy="0 0 0" />
-      <geometry>
-        <mesh
-          filename="package://robotican_komodo/description/meshes/FR_wheel_link.STL" />
+        xyz="-9.867E-07 9.3004E-05 -1.8753E-05"
+        rpy="0 0 0" />
+      <mass
+        value="2.6829" />
+      <inertia
+        ixx="0.012758"
+        ixy="8.8036E-09"
+        ixz="1.0405E-07"
+        iyy="0.023277"
+        iyz="-2.0115E-06"
+        izz="0.012755" />
+    </inertial>
+    <visual>
+      <origin
+        xyz="0 0 0"
+        rpy="0 0 0" />
+      <geometry>
+        <mesh
+          filename="package://robotican_komodo/description/meshes/wheel_link.STL" />
+      </geometry>
+      <material
+        name="">
+        <color
+          rgba="0.79216 0.81961 0.93333 1" />
+      </material>
+    </visual>
+    <collision>
+      <origin
+        xyz="0 0 0"
+        rpy="${M_PI/2} 0 0" />
+      <geometry>
+	<!--  <mesh filename="package://robotican_komodo/description/meshes/wheel_link.STL" /> -->
+	  <cylinder  length="0.05" radius="0.127"/>
       </geometry>
     </collision>
@@ -207,5 +260,5 @@
     type="continuous">
     <origin
-      xyz="0.165 -0.1893 0"
+      xyz="0.165 -0.18955 0"
       rpy="0 0 0" />
     <parent
@@ -217,157 +270,88 @@
   </joint>
   <link
-    name="FL_wheel_link">
-    <inertial>
-      <origin
-        xyz="-1.2974E-05 0.00017781 -1.1646E-05"
-        rpy="0 0 0" />
-      <mass
-        value="3.5882" />
-      <inertia
-        ixx="0.016234"
-        ixy="1.9586E-06"
-        ixz="1.7466E-06"
-        iyy="0.029573"
-        iyz="1.5657E-06"
-        izz="0.016234" />
-    </inertial>
-    <visual>
-      <origin
-        xyz="0 0 0"
-        rpy="0 0 1.57" />
-      <geometry>
-        <mesh
-          filename="package://robotican_komodo/description/meshes/FL_wheel_link.STL" />
-      </geometry>
-      <material
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
Commit message: KOMODO REV ARM

File: robotican_komodo/description/models/komodo.xacro (robot description, xacro)
@@ -55,5 +55,5 @@
     <origin
       xyz="-0.11925 0 0.16716"
-      rpy="0 0 0" />
+      rpy="0 0 ${M_PI}" />
     <parent
       link="base_link" />
@@ -64,5 +64,5 @@
   </joint>
 	<joint name="base_arm_joint" type="fixed">
-		<origin xyz="-0.091 0 0.093" rpy="0 0 0" />
+		<origin xyz="-0.091 0 0.093" rpy="0 0 ${M_PI}" />
 		<parent link="arm_link" />
 		<child link="base_arm_link" />

Commit message: init branch

File: robotican_komodo/description/models/komodo.xacro (robot description, xacro)
@@ -6,7 +6,10 @@
 	<!--      END          -->
 	<!--    ARM     -->
-	<xacro:include filename="$(find robotican_manipulator_h)/models/manipulator_h.xacro" />
+	<!-- <xacro:include filename="$(find robotican_manipulator_h)/models/manipulator_h.xacro" /> -->
 	<!--      END          -->
- <link
+  <!--    TORSO     -->
+  <xacro:include filename="$(find robotican_komodo)/description/models/komodo_torso.xacro" />
+  <!--     END      -->
+<!--  <link
     name="arm_link">
     <inertial>  <gazebo reference="base_arm_link">
@@ -62,10 +65,10 @@
     <axis
       xyz="0 0 0" />
-  </joint>
-	<joint name="base_arm_joint" type="fixed">
+  </joint> -->
+<!-- 	<joint name="base_arm_joint" type="fixed">
 		<origin xyz="-0.091 0 0.093" rpy="0 0 ${M_PI}" />
 		<parent link="arm_link" />
 		<child link="base_arm_link" />
 		<axis xyz="0 0 0" />
-	</joint>
+	</joint> -->
 </robot>

Commit message: changes

File: robotican_komodo/description/models/komodo.xacro (robot description, xacro)
@@ -11,64 +11,3 @@
   <xacro:include filename="$(find robotican_komodo)/description/models/komodo_torso.xacro" />
   <!--     END      -->
-<!--  <link
-    name="arm_link">
-    <inertial>  <gazebo reference="base_arm_link">
-    <material>Gazebo/Grey</material>
-  </gazebo>
-      <origin
-        xyz="-0.022197 -1.9122E-07 0.044251"
-        rpy="0 0 0" />
-      <mass
-        value="0.16757" />
-      <inertia
-        ixx="0.00062908"
-        ixy="-8.3342E-10"
-        ixz="-0.00014877"
-        iyy="0.0010719"
-        iyz="1.6859E-09"
-        izz="0.0013427" />
-    </inertial>
-    <visual>
-      <origin
-        xyz="0 0 0"
-        rpy="0 0 0" />
-      <geometry>
-        <mesh
-          filename="package://robotican_komodo/description/meshes/arm_link.STL" />
-      </geometry>
-      <material
-        name="">
-        <color
-          rgba="0.79216 0.81961 0.93333 1" />
-      </material>
-    </visual>
-    <collision>
-      <origin
-        xyz="0 0 0"
-        rpy="0 0 0" />
-      <geometry>
-        <mesh
-          filename="package://robotican_komodo/description/meshes/arm_link.STL" />
-      </geometry>
-    </collision>
-  </link>
-  <joint
-    name="arm_joint"
-    type="fixed">
-    <origin
-      xyz="-0.11925 0 0.16716"
-      rpy="0 0 ${M_PI}" />
-    <parent
-      link="base_link" />
-    <child
-      link="arm_link" />
-    <axis
-      xyz="0 0 0" />
-  </joint> -->
-<!-- 	<joint name="base_arm_joint" type="fixed">
-		<origin xyz="-0.091 0 0.093" rpy="0 0 ${M_PI}" />
-		<parent link="arm_link" />
-		<child link="base_arm_link" />
-		<axis xyz="0 0 0" />
-	</joint> -->
 </robot>
