Commit message: finish fix

File: robotican_komodo/description/models/komodo_base.xacro (robot description, xacro)
@@ -261,5 +261,23 @@
   </joint>
   <link
-    name="laser_link" />
+    name="laser_link" >
+    <visual>
+      <origin
+        xyz="-0.22 0.0 -0.165"
+        rpy="0 0 0" />
+      <material
+        name="">
+        <color
+          rgba="0.79216 0.81961 0.93333 1" />
+      </material>
+      <geometry>
+        <mesh
+          filename="package://robotican_komodo/description/meshes/laser_link.STL" />
+      </geometry>
+      <material
+        name="">
+      </material>
+    </visual>
+  </link>
   <joint
     name="laser_joint"

Commit message: asus

File: robotican_komodo/description/models/komodo_base.xacro (robot description, xacro)
@@ -368,3 +368,59 @@
       xyz="0 0 0" />
   </joint>
+<joint name="depth_camera_rgb_joint" type="fixed">
+      <origin xyz="0 0.0185 0" rpy="0 0 0"/>
+      <parent link="depth_camera_link"/>
+      <child link="depth_camera_rgb_frame" />
+    </joint>
+    <link name="depth_camera_rgb_frame">
+      <inertial>
+	<mass value="0.001" />
+	<origin xyz="0 0 0" />
+	<inertia ixx="0.0001" ixy="0.0" ixz="0.0"
+	  iyy="0.0001" iyz="0.0"
+	  izz="0.0001" />
+	</inertial>
+      </link>
+      <joint name="depth_camera_rgb_optical_joint" type="fixed">
+	<origin xyz="0 0 0" rpy="${-M_PI/2} 0 ${-M_PI/2}" />
+	<parent link="depth_camera_rgb_frame" />
+	<child link="depth_camera_rgb_optical_frame" />
+      </joint>
+      <link name="depth_camera_rgb_optical_frame">
+	<inertial>
+	  <mass value="0.001" />
+	  <origin xyz="0 0 0" />
+	  <inertia ixx="0.0001" ixy="0.0" ixz="0.0"
+	    iyy="0.0001" iyz="0.0"
+	    izz="0.0001" />
+	  </inertial>
+	</link>
+	<joint name="depth_camera_depth_joint" type="fixed">
+	  <origin xyz="0 0.0445 0" rpy="0 0 0" />
+	  <parent link="depth_camera_link" />
+	  <child link="depth_camera_depth_frame" />
+	</joint>
+	<link name="depth_camera_depth_frame">
+	  <inertial>
+	    <mass value="0.001" />
+	    <origin xyz="0 0 0" />
+	    <inertia ixx="0.0001" ixy="0.0" ixz="0.0"
+	      iyy="0.0001" iyz="0.0"
+	      izz="0.0001" />
+	    </inertial>
+	  </link>
+	  <joint name="depth_camera_depth_optical_joint" type="fixed">
+	    <origin xyz="0 0 0" rpy="${-M_PI/2} 0 ${-M_PI/2}" />
+	    <parent link="depth_camera_depth_frame" />
+	    <child link="depth_camera_depth_optical_frame" />
+	  </joint>
+	  <link name="depth_camera_depth_optical_frame">
+	    <inertial>
+	      <mass value="0.001" />
+	      <origin xyz="0 0 0" />
+	      <inertia ixx="0.0001" ixy="0.0" ixz="0.0"
+		iyy="0.0001" iyz="0.0"
+		izz="0.0001" />
+	      </inertial>
+	    </link>
 </robot>

File: robotican_komodo/description/models/komodo_gazebo.xacro (robot description, xacro)
@@ -10,4 +10,5 @@
   <xacro:arg name="lidar" default="false"/>
   <xacro:arg name="sr300" default="false"/>
+  <xacro:arg name="depth_camera" default="false"/>
   <xacro:include filename="$(find robotican_manipulator_h)/models/manipulator_h_gazebo_plugins.xacro" />
   	    <!-- SR300 -->
@@ -16,4 +17,7 @@
   </xacro:if>
   <!-- TODO: Asus -->
+  <xacro:if value="$(arg depth_camera)">
+    <xacro:include filename="$(find robotican_common)/gazebo/asus_xtion_pro_live.xacro" />
+  </xacro:if>
   <!-- Sonars -->
   <xacro:if value="$(arg urf)">

Commit message: tom's last commit

File: robotican_komodo/description/models/komodo_base.xacro (robot description, xacro)
@@ -83,5 +83,4 @@
         rpy="${M_PI/2} 0 0" />
       <geometry>
-	<!--  <mesh filename="package://robotican_komodo/description/meshes/wheel_link.STL" /> -->
 	  <cylinder  length="0.05" radius="0.127"/>
       </geometry>
@@ -136,5 +135,4 @@
         rpy="${M_PI/2} 0 0" />
       <geometry>
-	<!--  <mesh filename="package://robotican_komodo/description/meshes/wheel_link.STL" /> -->
 	  <cylinder  length="0.05" radius="0.127"/>
       </geometry>
@@ -189,5 +187,4 @@
         rpy="${M_PI/2} 0 0" />
       <geometry>
-	<!--  <mesh filename="package://robotican_komodo/description/meshes/wheel_link.STL" /> -->
 	  <cylinder  length="0.05" radius="0.127"/>
       </geometry>
@@ -242,5 +239,4 @@
         rpy="${M_PI/2} 0 0" />
       <geometry>
-	<!--  <mesh filename="package://robotican_komodo/description/meshes/wheel_link.STL" /> -->
 	  <cylinder  length="0.05" radius="0.127"/>
       </geometry>

File: robotican_komodo/description/models/komodo_gazebo.xacro (robot description, xacro)
@@ -167,5 +167,5 @@
           <type>transmission_interface/SimpleTransmission</type>
           <joint name="base_rotation_joint">
-            <hardwareInterface>PositionJointInterface</hardwareInterface>
+            <hardwareInterface>PosVelJointInterface</hardwareInterface>
           </joint>
           <actuator name="base_rotation_joint_motor">
@@ -176,5 +176,5 @@
           <type>transmission_interface/SimpleTransmission</type>
           <joint name="shoulder_joint">
-            <hardwareInterface>PositionJointInterface</hardwareInterface>
+            <hardwareInterface>PosVelJointInterface</hardwareInterface>
           </joint>
           <actuator name="shoulder_joint_motor">
@@ -185,5 +185,5 @@
           <type>transmission_interface/SimpleTransmission</type>
           <joint name="elbow1_joint">
-            <hardwareInterface>PositionJointInterface</hardwareInterface>
+            <hardwareInterface>PosVelJointInterface</hardwareInterface>
           </joint>
           <actuator name="elbow1_joint_motor">
@@ -194,5 +194,5 @@
           <type>transmission_interface/SimpleTransmission</type>
           <joint name="elbow2_joint">
-            <hardwareInterface>PositionJointInterface</hardwareInterface>
+            <hardwareInterface>PosVelJointInterface</hardwareInterface>
           </joint>
           <actuator name="elbow2_joint_motor">
@@ -203,5 +203,5 @@
           <type>transmission_interface/SimpleTransmission</type>
           <joint name="wrist_joint">
-            <hardwareInterface>PositionJointInterface</hardwareInterface>
+            <hardwareInterface>PosVelJointInterface</hardwareInterface>
           </joint>
           <actuator name="wrist_joint_motor">

File: robotican_komodo/description/models/komodo_torso.xacro (robot description, xacro)
@@ -22,5 +22,5 @@
       </material>
     </visual>
-    <collision>
+  <collision>
       <origin xyz="0 0 0" rpy="0 0 0" />
       <geometry>
@@ -91,5 +91,5 @@
 	upper="0.45"
 	effort="70"
-	velocity="0.062" />
+	velocity="0.012" />
   </joint>
   <joint
@@ -109,5 +109,5 @@
       upper="3.14"
       effort="10"
-      velocity="0" />
+      velocity="1.0" />
   </joint>
   <link name="base_rotation_link">
@@ -161,5 +161,4 @@
       <geometry>
         <mesh filename="package://robotican_arm/meshes/shoulder_link.STL"/>
-        <!-- Simplified -->
       </geometry>
     </collision>
@@ -170,5 +169,5 @@
     <child link="shoulder_link"/>
     <axis xyz="0 1 0"/>
-    <limit effort="2000" lower="0.0" upper="1.57" velocity="0"/>
+    <limit effort="2000" lower="0.0" upper="1.57" velocity="1.0"/>
   </joint>
   <link name="elbow1_link">
@@ -192,5 +191,4 @@
       <geometry>
         <mesh filename="package://robotican_arm/meshes/elbow1_link.STL"/>
-        <!-- Simplified -->
       </geometry>
     </collision>
@@ -201,5 +199,5 @@
     <child link="elbow1_link"/>
     <axis xyz="-0.999999999998754 0 0"/>
-    <limit effort="100" lower="-3.14" upper="3.14" velocity="0"/>
+    <limit effort="100" lower="-3.14" upper="3.14" velocity="1.0"/>
   </joint>
   <link name="elbow2_link">
@@ -223,5 +221,4 @@
       <geometry>
         <mesh filename="package://robotican_arm/meshes/elbow2_link.STL"/>
-        <!-- Simplified -->
       </geometry>
     </collision>
@@ -232,5 +229,5 @@
     <child link="elbow2_link"/>
     <axis xyz="0 1 0"/>
-    <limit effort="10" lower="-3.14" upper="3.14" velocity="0"/>
+    <limit effort="10" lower="-3.14" upper="3.14" velocity="1.0"/>
   </joint>
   <link name="wrist_link">
@@ -254,5 +251,4 @@
       <geometry>
         <mesh filename="package://robotican_arm/meshes/wrist_link.STL"/>
-        <!-- Simplified -->
       </geometry>
     </collision>
@@ -263,5 +259,5 @@
     <child link="wrist_link"/>
     <axis xyz="0 0 0.999999999998754"/>
-    <limit effort="10" lower="-3.14" upper="3.14" velocity="0"/>
+    <limit effort="10" lower="-3.14" upper="3.14" velocity="1.0"/>
   </joint>
   <link name="gripper_link"/>
@@ -291,5 +287,4 @@
       <geometry>
         <mesh filename="package://robotican_arm/meshes/left_finger_link.STL"/>
-        <!-- Simplified -->
       </geometry>
     </collision>
@@ -322,5 +317,4 @@
       <geometry>
         <mesh filename="package://robotican_arm/meshes/right_finger_link.STL"/>
-        <!-- Simplified -->
       </geometry>
     </collision>
@@ -599,5 +593,5 @@
       xyz="0 0 0" />
   </joint>
-<joint name="torso_camera_rgb_joint" type="fixed">
+  <joint name="torso_camera_rgb_joint" type="fixed">
       <origin xyz="0 0.0185 0" rpy="0 0 0"/>
       <parent link="torso_camera_link"/>
