Commit message: update

File: robotican_komodo/description/models/komodo_torso.xacro (robot description, xacro)
@@ -35,12 +35,70 @@
     <axis xyz="0 0 0" />
   </joint>
+   <link
+    name="torso_link">
+    <inertial>
+      <origin
+        xyz="0.0954671716579415 1.91586249009607E-06 -0.0185743175743276"
+        rpy="0 0 0" />
+      <mass
+        value="1.09057945344451" />
+      <inertia
+        ixx="0.000835857275985966"
+        ixy="5.81870910353681E-08"
+        ixz="-3.13493979506258E-05"
+        iyy="0.00128840659932805"
+        iyz="1.45397132642805E-07"
+        izz="0.00136461371089342" />
+    </inertial>
+    <visual>
+      <origin
+        xyz="0 0 0"
+        rpy="0 0 0" />
+      <geometry>
+        <mesh
+          filename="package://robotican_komodo/description/meshes/torso_link.STL" />
+      </geometry>
+      <material
+        name="">
+        <color
+          rgba="0.35 0.35 0.35 1" />
+      </material>
+    </visual>
+    <collision>
+      <origin
+        xyz="0 0 0"
+        rpy="0 0 0" />
+      <geometry>
+        <mesh
+          filename="package://robotican_komodo/description/meshes/torso_link.STL" />
+      </geometry>
+    </collision>
+  </link>
+  <joint
+    name="torso_joint"
+    type="fixed"> <!--prismatic-->
+    <origin
+      xyz="0.101457996026178 0 0.0740000000000002"
+      rpy="0 0 0" />
+    <parent
+      link="arm_base_link" />
+    <child
+      link="torso_link" />
+    <axis
+      xyz="0 0 1" />
+   <limit
+	lower="0"
+	upper="0.45"
+	effort="0"
+	velocity="0" />
+  </joint>
   <joint
     name="base_rotation_joint"
     type="revolute">
     <origin
-      xyz="-0.096277996026178 0 0.0549000000000002"
-      rpy="-5.46369598732866E-16 1.34659130519145E-15 -2.1922983760752E-31" />
+      xyz="0.113 0 -0.00400000000000003"
+      rpy="0 0 0" />
     <parent
-      link="arm_base_link" />
+      link="torso_link" />
     <child
       link="base_rotation_link" />

Commit message: gezebo update

File: robotican_komodo/description/models/komodo_torso.xacro (robot description, xacro)
@@ -333,3 +333,215 @@
     <limit effort="10" lower="-3.14" upper="3.14" velocity="0"/>
   </joint>
+  <link
+    name="Creative_Camera_link">
+    <inertial>
+      <origin
+        xyz="0.000246466472824558 6.40214461760665E-06 -3.77569804070194E-05"
+        rpy="0 0 0" />
+      <mass
+        value="0.0917411732955106" />
+      <inertia
+        ixx="9.42830385924344E-05"
+        ixy="7.20275321596364E-09"
+        ixz="-9.53710985095244E-09"
+        iyy="1.31046061468615E-05"
+        iyz="2.49172946580444E-11"
+        izz="9.18985906934582E-05" />
+    </inertial>
+    <visual>
+      <origin
+        xyz="0 0 0"
+        rpy="0 0 0" />
+      <geometry>
+        <mesh
+          filename="package://robotican_komodo/description/meshes/creative_camera_link.STL" />
+      </geometry>
+      <material
+        name="">
+        <color
+          rgba="0.2 0.2 0.2 1" />
+      </material>
+    </visual>
+    <collision>
+      <origin
+        xyz="0 0 0"
+        rpy="0 0 0" />
+      <geometry>
+        <mesh
+          filename="package://robotican_komodo/description/meshes/creative_camera_link.STL" />
+      </geometry>
+    </collision>
+  </link>
+  <joint
+    name="Creative_Camera_joint"
+    type="fixed">
+    <origin
+      xyz="-0.05 0 0.0255"
+      rpy="0 -1.57 0" />
+    <parent
+      link="wrist_link" />
+    <child
+      link="Creative_Camera_link" />
+    <axis
+      xyz="0 0 0" />
+  </joint>
+  <link
+      name="torso_camera_link">
+      <inertial>
+        <origin
+          xyz="-0.0186787128878999 -0.000250455424978622 -0.00418879037489228"
+          rpy="0 0 0" />
+        <mass
+          value="0.172317738459302" />
+        <inertia
+          ixx="0.00043258025617677"
+          ixy="-5.30549374358253E-07"
+          ixz="-4.88064241259027E-07"
+          iyy="4.50251290386955E-05"
+          iyz="-1.80788928482687E-07"
+          izz="0.000422864751433858" />
+      </inertial>
+      <visual>
+        <origin
+          xyz="0 0 0"
+          rpy="0 0 0" />
+        <geometry>
+          <mesh
+            filename="package://robotican_komodo/description/meshes/torso_camera_link.STL" />
+        </geometry>
+        <material
+          name="">
+          <color
+            rgba="0.1792156862745098 0.1819607843137255 0.1933333333333333 1" />
+        </material>
+      </visual>
+      <collision>
+        <origin
+          xyz="0 0 0"
+          rpy="0 0 0" />
+        <geometry>
+          <mesh
+            filename="package://robotican_komodo/description/meshes/torso_camera_link.STL" />
+        </geometry>
+      </collision>
+    </link>
+    <joint
+      name="torso_camera_joint"
+      type="fixed">
+      <origin
+        xyz="0.143457996026181 0 0.696234376944339"
+        rpy="0 0 0" />
+      <parent
+        link="arm_base_link" />
+      <child
+        link="torso_camera_link" />
+      <axis
+        xyz="0 0 0" />
+    </joint>
+    <link
+    name="rear_camera_link">
+    <inertial>
+      <origin
+        xyz="3.63553471786722E-06 0.000213443852905448 -0.00979905092954501"
+        rpy="0 0 0" />
+      <mass
+        value="0.0346828331927957" />
+      <inertia
+        ixx="6.28790547336403E-06"
+        ixy="-2.06834495042828E-09"
+        ixz="1.17994816083997E-09"
+        iyy="6.08020816375982E-06"
+        iyz="3.61787794070637E-08"
+        izz="9.95214453956502E-06" />
+    </inertial>
+    <visual>
+      <origin
+        xyz="0 0 0"
+        rpy="1.57 0 1.57" />
+      <geometry>
+        <mesh
+          filename="package://robotican_komodo/description/meshes/rear_camera_link.STL" />
+      </geometry>
+      <material
+        name="">
+        <color
+          rgba="0.1 0.1 0.1 1" />
+      </material>
+    </visual>
+    <collision>
+      <origin
+        xyz="0 0 0"
+        rpy="0 0 0" />
+      <geometry>
+        <mesh
+          filename="package://robotican_komodo/description/meshes/rear_camera_link.STL" />
+      </geometry>
+    </collision>
+  </link>
+  <joint
+    name="rear_camera_joint"
+    type="fixed">
+    <origin
+      xyz="0.0329579960261737 0 0.354500000000001"
+      rpy="0 0 -3.15" />
+    <parent
+      link="arm_base_link" />
+    <child
+      link="rear_camera_link" />
+    <axis
+      xyz="0 0 0" />
+  </joint>
+  <link
+    name="top_camera_link">
+    <inertial>
+      <origin
+        xyz="4.37351127445876E-06 0.000213430006923504 -0.00979905092954436"
+        rpy="0 0 0" />
+      <mass
+        value="0.0346828331927942" />
+      <inertia
+        ixx="6.28791729321072E-06"
+        ixy="-1.35017062474835E-09"
+        ixz="1.30503198120059E-09"
+        iyy="6.08019634391293E-06"
+        iyz="3.61744833904195E-08"
+        izz="9.95214453956468E-06" />
+    </inertial>
+    <visual>
+      <origin
+        xyz="0 0 0"
+        rpy="5.38354147863953E-15 1.55701850396119E-12 -1.56733874423455" />
+      <geometry>
+        <mesh
+          filename="package://robotican_komodo/description/meshes/top_camera_link.STL" />
+      </geometry>
+      <material
+        name="">
+        <color
+          rgba="0.1 0.1 0.1 1" />
+      </material>
+    </visual>
+    <collision>
+      <origin
+        xyz="0 0 0"
+        rpy="0 0 0" />
+      <geometry>
+        <mesh
+          filename="package://robotican_komodo/description/meshes/top_camera_link.STL" />
+      </geometry>
+    </collision>
+  </link>
+  <joint
+    name="top_camera_joint"
+    type="fixed">
+    <origin
+      xyz="0.0622079960261761 0.0152829991418538 0.660000000000001"
+      rpy="0 0.0 0" />
+    <parent
+      link="arm_base_link" />
+    <child
+      link="top_camera_link" />
+    <axis
+      xyz="0 0 0" />
+  </joint>
 </robot>

Commit message: update

File: robotican_komodo/description/models/komodo_torso.xacro (robot description, xacro)
@@ -170,5 +170,5 @@
     <child link="shoulder_link"/>
     <axis xyz="0 1 0"/>
-    <limit effort="2000" lower="-1.57" upper="1.57" velocity="0"/>
+    <limit effort="2000" lower="0.0" upper="1.57" velocity="0"/>
   </joint>
   <link name="elbow1_link">

Commit message: update

File: robotican_komodo/description/models/komodo_torso.xacro (robot description, xacro)
@@ -299,5 +299,5 @@
     <parent link="wrist_link"/>
     <child link="left_finger_link"/>
-    <axis xyz="1 0 0"/>
+    <axis xyz="0.5 0 0"/>
     <limit effort="3.1" lower="-1.57" upper="1.57" velocity="2.0"/>
   </joint>
@@ -330,5 +330,5 @@
     <parent link="wrist_link"/>
     <child link="right_finger_link"/>
-    <axis xyz="1 0 0"/>
+    <axis xyz="0.5 0 0"/>
     <limit effort="3.1" lower="-1.57" upper="1.57" velocity="2.0"/>
   </joint>

Commit message: update

File: robotican_komodo/description/models/komodo_torso.xacro (robot description, xacro)
@@ -299,5 +299,5 @@
     <parent link="wrist_link"/>
     <child link="left_finger_link"/>
-    <axis xyz="0.5 0 0"/>
+    <axis xyz="1.5 0 0"/>
     <limit effort="3.1" lower="-1.57" upper="1.57" velocity="2.0"/>
   </joint>
@@ -330,5 +330,5 @@
     <parent link="wrist_link"/>
     <child link="right_finger_link"/>
-    <axis xyz="0.5 0 0"/>
+    <axis xyz="1.5 0 0"/>
     <limit effort="3.1" lower="-1.57" upper="1.57" velocity="2.0"/>
   </joint>

Commit message: update

File: robotican_komodo/description/models/komodo_torso.xacro (robot description, xacro)
@@ -299,5 +299,5 @@
     <parent link="wrist_link"/>
     <child link="left_finger_link"/>
-    <axis xyz="1.5 0 0"/>
+    <axis xyz="3 0 0"/>
     <limit effort="3.1" lower="-1.57" upper="1.57" velocity="2.0"/>
   </joint>
@@ -330,5 +330,5 @@
     <parent link="wrist_link"/>
     <child link="right_finger_link"/>
-    <axis xyz="1.5 0 0"/>
+    <axis xyz="3 0 0"/>
     <limit effort="3.1" lower="-1.57" upper="1.57" velocity="2.0"/>
   </joint>

Commit message: update

File: robotican_komodo/description/models/komodo_torso.xacro (robot description, xacro)
@@ -296,8 +296,8 @@
   </link>
   <joint name="left_finger_joint" type="revolute">
-    <origin rpy="2.85979682697881E-15 1.01870746742143E-16 3.19235832636806E-21" xyz="-0.000250000000000111 0.021 0.0422500000000001"/>
+    <origin rpy="0.0 0.3 0.0" xyz="-0.000250000000000111 0.021 0.0422500000000001"/>
     <parent link="wrist_link"/>
     <child link="left_finger_link"/>
-    <axis xyz="3 0 0"/>
+    <axis xyz="1 0 0"/>
     <limit effort="3.1" lower="-1.57" upper="1.57" velocity="2.0"/>
   </joint>
@@ -327,8 +327,8 @@
   </link>
   <joint name="right_finger_joint" type="revolute">
-    <origin rpy="0 3.19686557214722E-37 0" xyz="-0.00024999999999889 -0.021 0.0422499999999999"/>
+    <origin rpy="0 0.3 0" xyz="-0.00024999999999889 -0.021 0.0422499999999999"/>
     <parent link="wrist_link"/>
     <child link="right_finger_link"/>
-    <axis xyz="3 0 0"/>
+    <axis xyz="1 0 0"/>
     <limit effort="3.1" lower="-1.57" upper="1.57" velocity="2.0"/>
   </joint>

Commit message: update

File: robotican_komodo/description/models/komodo_torso.xacro (robot description, xacro)
@@ -296,5 +296,5 @@
   </link>
   <joint name="left_finger_joint" type="revolute">
-    <origin rpy="0.0 0.3 0.0" xyz="-0.000250000000000111 0.021 0.0422500000000001"/>
+    <origin rpy="0.0 2 0.0" xyz="-0.000250000000000111 0.021 0.0422500000000001"/>
     <parent link="wrist_link"/>
     <child link="left_finger_link"/>
@@ -327,5 +327,5 @@
   </link>
   <joint name="right_finger_joint" type="revolute">
-    <origin rpy="0 0.3 0" xyz="-0.00024999999999889 -0.021 0.0422499999999999"/>
+    <origin rpy="0 2 0" xyz="-0.00024999999999889 -0.021 0.0422499999999999"/>
     <parent link="wrist_link"/>
     <child link="right_finger_link"/>

Commit message: update

File: robotican_komodo/description/models/komodo_torso.xacro (robot description, xacro)
@@ -296,5 +296,5 @@
   </link>
   <joint name="left_finger_joint" type="revolute">
-    <origin rpy="0.0 2 0.0" xyz="-0.000250000000000111 0.021 0.0422500000000001"/>
+    <origin rpy="2 0 0.0" xyz="-0.000250000000000111 0.021 0.0422500000000001"/>
     <parent link="wrist_link"/>
     <child link="left_finger_link"/>
@@ -327,5 +327,5 @@
   </link>
   <joint name="right_finger_joint" type="revolute">
-    <origin rpy="0 2 0" xyz="-0.00024999999999889 -0.021 0.0422499999999999"/>
+    <origin rpy="2 0 0" xyz="-0.00024999999999889 -0.021 0.0422499999999999"/>
     <parent link="wrist_link"/>
     <child link="right_finger_link"/>

Commit message: update

File: robotican_komodo/description/models/komodo_torso.xacro (robot description, xacro)
@@ -296,5 +296,5 @@
   </link>
   <joint name="left_finger_joint" type="revolute">
-    <origin rpy="2 0 0.0" xyz="-0.000250000000000111 0.021 0.0422500000000001"/>
+    <origin rpy="0.3 0 0.0" xyz="-0.000250000000000111 0.021 0.0422500000000001"/>
     <parent link="wrist_link"/>
     <child link="left_finger_link"/>
@@ -327,5 +327,5 @@
   </link>
   <joint name="right_finger_joint" type="revolute">
-    <origin rpy="2 0 0" xyz="-0.00024999999999889 -0.021 0.0422499999999999"/>
+    <origin rpy="-0.3 0 0" xyz="-0.00024999999999889 -0.021 0.0422499999999999"/>
     <parent link="wrist_link"/>
     <child link="right_finger_link"/>

Commit message: update

File: robotican_komodo/description/models/komodo_torso.xacro (robot description, xacro)
@@ -296,5 +296,5 @@
   </link>
   <joint name="left_finger_joint" type="revolute">
-    <origin rpy="0.3 0 0.0" xyz="-0.000250000000000111 0.021 0.0422500000000001"/>
+    <origin rpy="0.1 0 0.0" xyz="-0.000250000000000111 0.021 0.0422500000000001"/>
     <parent link="wrist_link"/>
     <child link="left_finger_link"/>
@@ -327,5 +327,5 @@
   </link>
   <joint name="right_finger_joint" type="revolute">
-    <origin rpy="-0.3 0 0" xyz="-0.00024999999999889 -0.021 0.0422499999999999"/>
+    <origin rpy="-0.1 0 0" xyz="-0.00024999999999889 -0.021 0.0422499999999999"/>
     <parent link="wrist_link"/>
     <child link="right_finger_link"/>

Commit message: update

File: robotican_komodo/description/models/komodo_torso.xacro (robot description, xacro)
@@ -296,5 +296,5 @@
   </link>
   <joint name="left_finger_joint" type="revolute">
-    <origin rpy="0.1 0 0.0" xyz="-0.000250000000000111 0.021 0.0422500000000001"/>
+    <origin rpy="0.2 0 0.0" xyz="-0.000250000000000111 0.021 0.0422500000000001"/>
     <parent link="wrist_link"/>
     <child link="left_finger_link"/>
@@ -327,5 +327,5 @@
   </link>
   <joint name="right_finger_joint" type="revolute">
-    <origin rpy="-0.1 0 0" xyz="-0.00024999999999889 -0.021 0.0422499999999999"/>
+    <origin rpy="-0.2 0 0" xyz="-0.00024999999999889 -0.021 0.0422499999999999"/>
     <parent link="wrist_link"/>
     <child link="right_finger_link"/>

Commit message: update

File: robotican_komodo/description/models/komodo_torso.xacro (robot description, xacro)
@@ -296,5 +296,5 @@
   </link>
   <joint name="left_finger_joint" type="revolute">
-    <origin rpy="0.2 0 0.0" xyz="-0.000250000000000111 0.021 0.0422500000000001"/>
+    <origin rpy="0.25 0 0.0" xyz="-0.000250000000000111 0.021 0.0422500000000001"/>
     <parent link="wrist_link"/>
     <child link="left_finger_link"/>
@@ -327,5 +327,5 @@
   </link>
   <joint name="right_finger_joint" type="revolute">
-    <origin rpy="-0.2 0 0" xyz="-0.00024999999999889 -0.021 0.0422499999999999"/>
+    <origin rpy="-0.25 0 0" xyz="-0.00024999999999889 -0.021 0.0422499999999999"/>
     <parent link="wrist_link"/>
     <child link="right_finger_link"/>

Commit message: update

File: robotican_komodo/description/models/komodo_torso.xacro (robot description, xacro)
@@ -296,5 +296,5 @@
   </link>
   <joint name="left_finger_joint" type="revolute">
-    <origin rpy="0.25 0 0.0" xyz="-0.000250000000000111 0.021 0.0422500000000001"/>
+    <origin rpy="0.22 0 0.0" xyz="-0.000250000000000111 0.021 0.0422500000000001"/>
     <parent link="wrist_link"/>
     <child link="left_finger_link"/>
@@ -327,5 +327,5 @@
   </link>
   <joint name="right_finger_joint" type="revolute">
-    <origin rpy="-0.25 0 0" xyz="-0.00024999999999889 -0.021 0.0422499999999999"/>
+    <origin rpy="-0.22 0 0" xyz="-0.00024999999999889 -0.021 0.0422499999999999"/>
     <parent link="wrist_link"/>
     <child link="right_finger_link"/>

Commit message: update

File: robotican_komodo/description/models/komodo_torso.xacro (robot description, xacro)
@@ -296,5 +296,5 @@
   </link>
   <joint name="left_finger_joint" type="revolute">
-    <origin rpy="0.22 0 0.0" xyz="-0.000250000000000111 0.021 0.0422500000000001"/>
+    <origin rpy="0.21 0 0.0" xyz="-0.000250000000000111 0.021 0.0422500000000001"/>
     <parent link="wrist_link"/>
     <child link="left_finger_link"/>
@@ -327,5 +327,5 @@
   </link>
   <joint name="right_finger_joint" type="revolute">
-    <origin rpy="-0.22 0 0" xyz="-0.00024999999999889 -0.021 0.0422499999999999"/>
+    <origin rpy="-0.21 0 0" xyz="-0.00024999999999889 -0.021 0.0422499999999999"/>
     <parent link="wrist_link"/>
     <child link="right_finger_link"/>

Commit message: update

File: robotican_komodo/description/models/komodo_torso.xacro (robot description, xacro)
@@ -296,5 +296,5 @@
   </link>
   <joint name="left_finger_joint" type="revolute">
-    <origin rpy="0.21 0 0.0" xyz="-0.000250000000000111 0.021 0.0422500000000001"/>
+    <origin rpy="0.205 0 0.0" xyz="-0.000250000000000111 0.021 0.0422500000000001"/>
     <parent link="wrist_link"/>
     <child link="left_finger_link"/>
@@ -327,5 +327,5 @@
   </link>
   <joint name="right_finger_joint" type="revolute">
-    <origin rpy="-0.21 0 0" xyz="-0.00024999999999889 -0.021 0.0422499999999999"/>
+    <origin rpy="-0.205 0 0" xyz="-0.00024999999999889 -0.021 0.0422499999999999"/>
     <parent link="wrist_link"/>
     <child link="right_finger_link"/>

Commit message: komodo effort limit fix for gazebo

File: robotican_komodo/description/models/komodo_torso.xacro (robot description, xacro)
@@ -169,5 +169,5 @@
     <child link="shoulder_link"/>
     <axis xyz="0 1 0"/>
-    <limit effort="2000" lower="0.0" upper="1.57" velocity="1.0"/>
+    <limit effort="2000" lower="-9.9E-07" upper="1.57" velocity="1.0"/>
   </joint>
   <link name="elbow1_link">

Commit message: creative deletion

File: robotican_komodo/description/models/komodo_torso.xacro (robot description, xacro)
@@ -328,5 +328,5 @@
   </joint>
   <link
-    name="creative_camera_link">
+    name="softkinetic_camera_link">
     <inertial>
       <origin
@@ -368,5 +368,5 @@
   </link>
   <joint
-    name="creative_camera_joint"
+    name="softkinetic_camera_joint"
     type="fixed">
     <origin
@@ -376,14 +376,14 @@
       link="wrist_link" />
     <child
-      link="creative_camera_link" />
+      link="softkinetic_camera_link" />
     <axis
       xyz="0 0 0" />
   </joint>
-<joint name="creative_camera_rgb_joint" type="fixed">
+<joint name="softkinetic_camera_rgb_joint" type="fixed">
       <origin xyz="0 0.0185 0" rpy="0 0 0"/>
-      <parent link="creative_camera_link"/>
-      <child link="creative_camera_rgb_frame" />
+      <parent link="softkinetic_camera_link"/>
+      <child link="softkinetic_camera_rgb_frame" />
     </joint>
-    <link name="creative_camera_rgb_frame">
+    <link name="softkinetic_camera_rgb_frame">
       <inertial>
   <mass value="0.001" />
@@ -394,10 +394,10 @@
   </inertial>
       </link>
-      <joint name="creative_camera_rgb_optical_joint" type="fixed">
+      <joint name="softkinetic_camera_rgb_optical_joint" type="fixed">
   <origin xyz="0 0 0" rpy="${-M_PI/2} 0 ${-M_PI/2}" />
-  <parent link="creative_camera_rgb_frame" />
-  <child link="creative_camera_rgb_optical_frame" />
+  <parent link="softkinetic_camera_rgb_frame" />
+  <child link="softkinetic_camera_rgb_optical_frame" />
       </joint>
-      <link name="creative_camera_rgb_optical_frame">
+      <link name="softkinetic_camera_rgb_optical_frame">
   <inertial>
     <mass value="0.001" />
@@ -408,10 +408,10 @@
     </inertial>
   </link>
-  <joint name="creative_camera_depth_joint" type="fixed">
+  <joint name="softkinetic_camera_depth_joint" type="fixed">
     <origin xyz="0 0.0445 0" rpy="0 0 0" />
-    <parent link="creative_camera_link" />
-    <child link="creative_camera_depth_frame" />
-  </joint>
-  <link name="creative_camera_depth_frame">
+    <parent link="softkinetic_camera_link" />
+    <child link="softkinetic_camera_depth_frame" />
+  </joint>
+  <link name="softkinetic_camera_depth_frame">
     <inertial>
       <mass value="0.001" />
@@ -422,10 +422,10 @@
       </inertial>
     </link>
-    <joint name="creative_camera_depth_optical_joint" type="fixed">
+    <joint name="softkinetic_camera_depth_optical_joint" type="fixed">
       <origin xyz="0 0 0" rpy="${-M_PI/2} 0 ${-M_PI/2}" />
-      <parent link="creative_camera_depth_frame" />
-      <child link="creative_camera_depth_optical_frame" />
+      <parent link="softkinetic_camera_depth_frame" />
+      <child link="softkinetic_camera_depth_optical_frame" />
     </joint>
-    <link name="creative_camera_depth_optical_frame">
+    <link name="softkinetic_camera_depth_optical_frame">
       <inertial>
         <mass value="0.001" />
