Commit message: update

File: robotican_komodo/description/models/komodo_gazebo.xacro (robot description, xacro)
@@ -2,4 +2,5 @@
 <robot xmlns:xacro="http://www.ros.org/wiki/xacro" name="Komodo" description="Komodo robot">
   <xacro:include filename="$(find robotican_komodo)/description/models/komodo.xacro" />
+  <xacro:include filename="$(find robotican_common)/gazebo/softkinetic_camera_ds325.xacro" />
   <xacro:property name="URF_FOV" value="${10.0*M_PI/180}" />
   <xacro:arg name="controllers" default="true"/>
@@ -19,5 +20,5 @@
     <!-- softkinetic -->
   <xacro:if value="$(arg softkinetic)">
-     <xacro:include filename="$(find robotican_common)/gazebo/softkinetic_camera_ds325.xacro" />
+     <xacro:softkinetic_gazebo name="softkinetic_camera_rgb" ros_topic="softkinetic_camera"/>
   </xacro:if>
   <!-- TODO: Asus -->

File: robotican_manipulator_h/models/manipulator_h.xacro (robot description, xacro)
@@ -3,4 +3,5 @@
   name="robotican_manipulator_h" description="Manipulator H Arm" xmlns:xacro="http://www.ros.org/wiki/xacro">
   <xacro:property name="M_PI" value="3.1415926535897931" />
+  <xacro:include filename="$(find robotican_common)/models/softkinetic_camera_ds325/model.xacro" />
   <link
     name="base_arm_link">
@@ -515,4 +516,5 @@
       <dynamics friction ="1000" damping="100"/>
   </joint>
+<!--
   <link
     name="sr300_link">
@@ -567,3 +569,7 @@
       xyz="0 0 0" />
   </joint>
+-->
+  <sensor_senz3d parent="wrist_link" name="softkinetic_camera">
+    <origin xyz="-0.06355 0 0.041852" rpy="0.0 -${M_PI/2} 0.0"/>
+  </sensor_senz3d>
 </robot>

Commit message: strange gazebo

File: robotican_komodo/description/models/komodo_gazebo.xacro (robot description, xacro)
@@ -10,17 +10,6 @@
   <xacro:arg name="gps" default="false"/>
   <xacro:arg name="lidar" default="false"/>
-  <xacro:arg name="sr300" default="false"/>
-    <xacro:arg name="softkinetic" default="false"/>
   <xacro:arg name="depth_camera" default="false"/>
-  <xacro:include filename="$(find robotican_manipulator_h)/models/manipulator_h_gazebo_plugins.xacro" />
-  <!-- SR300 -->
-  <xacro:if value="$(arg sr300)">
-    <xacro:include filename="$(find robotican_common)/gazebo/sr300.xacro" />
-  </xacro:if>
-    <!-- softkinetic -->
-  <xacro:if value="$(arg softkinetic)">
-     <xacro:softkinetic_gazebo name="softkinetic_camera_rgb" ros_topic="softkinetic_camera"/>
-  </xacro:if>
-  <!-- TODO: Asus -->
+  <!-- Asus -->
   <xacro:if value="$(arg depth_camera)">
     <xacro:include filename="$(find robotican_common)/gazebo/asus_xtion_pro_live.xacro" />
@@ -54,6 +43,5 @@
     <xacro:include filename="$(find robotican_common)/gazebo/camera.xacro" />
     <xacro:if value="$(arg front_camera)">
-      <xacro:Camera name="front_camera" link="front_cam_link" image_width="640" image_height="480"
-        image_format="R8G8B8" clip_near="0.02" clip_far="300" />
+      <xacro:Camera name="front_camera" link="front_cam_link" image_width="640" image_height="480"  image_format="R8G8B8" clip_near="0.02" clip_far="300" />
       </xacro:if>
       <!-- controller manager and hardware interfaces -->
@@ -146,4 +134,7 @@
         <material>Gazebo/Black</material>
       </gazebo>
+      <gazebo reference="arm_base_link">
+        <gravity>false</gravity>
+      </gazebo>
       <gazebo reference="base_link">
         <material>Gazebo/Grey</material>
@@ -164,6 +155,3 @@
         <material>Gazebo/Black</material>
       </gazebo>
-      <gazebo reference="sr300_link">
-        <material>Gazebo/Black</material>
-      </gazebo>
 </robot>

Commit message: change komodo moveit

File: robotican_komodo/description/models/komodo_gazebo.xacro (robot description, xacro)
@@ -89,4 +89,67 @@
           </actuator>
         </transmission>
+        <transmission name="base_rotation_joint_trans">
+          <type>transmission_interface/SimpleTransmission</type>
+          <joint name="base_rotation_joint">
+            <hardwareInterface>PosVelJointInterface</hardwareInterface>
+          </joint>
+          <actuator name="base_rotation_joint_motor">
+            <mechanicalReduction>1</mechanicalReduction>
+          </actuator>
+        </transmission>
+        <transmission name="shoulder_joint_trans">
+          <type>transmission_interface/SimpleTransmission</type>
+          <joint name="shoulder_joint">
+            <hardwareInterface>PosVelJointInterface</hardwareInterface>
+          </joint>
+          <actuator name="shoulder_joint_motor">
+            <mechanicalReduction>1</mechanicalReduction>
+          </actuator>
+        </transmission>
+        <transmission name="elbow1_joint_trans">
+          <type>transmission_interface/SimpleTransmission</type>
+          <joint name="elbow1_joint">
+            <hardwareInterface>PosVelJointInterface</hardwareInterface>
+          </joint>
+          <actuator name="elbow1_joint_motor">
+            <mechanicalReduction>1</mechanicalReduction>
+          </actuator>
+        </transmission>
+        <transmission name="elbow2_joint_trans">
+          <type>transmission_interface/SimpleTransmission</type>
+          <joint name="elbow2_joint">
+            <hardwareInterface>PosVelJointInterface</hardwareInterface>
+          </joint>
+          <actuator name="elbow2_joint_motor">
+            <mechanicalReduction>1</mechanicalReduction>
+          </actuator>
+        </transmission>
+        <transmission name="wrist_joint_trans">
+          <type>transmission_interface/SimpleTransmission</type>
+          <joint name="wrist_joint">
+            <hardwareInterface>PosVelJointInterface</hardwareInterface>
+          </joint>
+          <actuator name="wrist_joint_motor">
+            <mechanicalReduction>1</mechanicalReduction>
+          </actuator>
+        </transmission>
+        <transmission name="left_finger_joint_trans">
+          <type>transmission_interface/SimpleTransmission</type>
+          <joint name="left_finger_joint">
+            <hardwareInterface>PositionJointInterface</hardwareInterface>
+          </joint>
+          <actuator name="left_finger_joint_motor">
+            <mechanicalReduction>1</mechanicalReduction>
+          </actuator>
+        </transmission>
+        <transmission name="right_finger_joint_trans">
+          <type>transmission_interface/SimpleTransmission</type>
+          <joint name="right_finger_joint">
+            <hardwareInterface>PositionJointInterface</hardwareInterface>
+          </joint>
+          <actuator name="right_finger_joint_motor">
+            <mechanicalReduction>1</mechanicalReduction>
+          </actuator>
+        </transmission>
       </xacro:if>
       <gazebo reference="FL_wheel_link">

File: robotican_komodo/description/models/komodo_torso.xacro (robot description, xacro)
@@ -35,3 +35,243 @@
     <axis xyz="0 0 0" />
   </joint>
+  <joint
+    name="base_rotation_joint"
+    type="revolute">
+    <origin
+      xyz="-0.096277996026178 0 0.0549000000000002"
+      rpy="-5.46369598732866E-16 1.34659130519145E-15 -2.1922983760752E-31" />
+    <parent
+      link="arm_base_link" />
+    <child
+      link="base_rotation_link" />
+    <axis
+      xyz="0 0 1" />
+    <limit
+      lower="-3.14"
+      upper="3.14"
+      effort="10"
+      velocity="0" />
+  </joint>
+  <link name="base_rotation_link">
+    <inertial>
+      <origin
+        rpy="0 0 0"
+        xyz="-1.11022302462516E-16 -7.80223872637444E-17 0.0660708417371112"/>
+      <mass
+        value="1.4054258533062"/>
+      <inertia
+        ixx="0.00159425912810341"
+        ixy="-8.40269196653518E-08"
+        ixz="-1.60925604895535E-19"
+        iyy="0.000605522001732049"
+        iyz="-6.08768470792684E-19"
+        izz="0.00123388334665811"/>
+    </inertial>
+    <visual>
+      <origin rpy="0 0 0" xyz="0 0 0"/>
+      <geometry>
+        <mesh filename="package://robotican_arm/meshes/base_rotation_link.STL"/>
+      </geometry>
+      <material name="">
+        <color rgba="0.3 0.3 0.3 1"/>
+      </material>
+    </visual>
+    <collision>
+      <origin rpy="0 0 0" xyz="0 0 0"/>
+      <geometry>
+        <mesh filename="package://robotican_arm/meshes/base_rotation_link.STL"/>
+      </geometry>
+    </collision>
+  </link>
+  <link name="shoulder_link">
+    <inertial>
+      <origin rpy="0 0 0" xyz="-4.66231481405233E-06 -9.82289126283389E-05 0.0772888499682157"/>
+      <mass value="0.191480823048406"/>
+      <inertia ixx="0.00107301595696304" ixy="-2.9789063890745E-07" ixz="-2.01216953964121E-08" iyy="0.000975953125213584" iyz="-1.19601921452086E-06" izz="0.000217659789393094"/>
+    </inertial>
+    <visual>
+      <origin rpy="0 0 0" xyz="0 0 0"/>
+      <geometry>
+        <mesh filename="package://robotican_arm/meshes/shoulder_link.STL"/>
+      </geometry>
+      <material name="">
+        <color rgba="0.4 0.4 0.4 1"/>
+      </material>
+    </visual>
+    <collision>
+      <origin rpy="0 0 0" xyz="0 0 0"/>
+      <geometry>
+        <mesh filename="package://robotican_arm/meshes/shoulder_link.STL"/>
+        <!-- Simplified -->
+      </geometry>
+    </collision>
+  </link>
+  <joint name="shoulder_joint" type="revolute">
+    <origin rpy="-4.20159904047482E-15 -5.97509793174248E-16 9.93431320775303E-15" xyz="0 0 0.0834999999999999"/>
+    <parent link="base_rotation_link"/>
+    <child link="shoulder_link"/>
+    <axis xyz="0 1 0"/>
+    <limit effort="2000" lower="-1.57" upper="1.57" velocity="0"/>
+  </joint>
+  <link name="elbow1_link">
+    <inertial>
+      <origin rpy="0 0 0" xyz="3.38561240652013E-05 2.66604610292575E-06 0.0239321015909688"/>
+      <mass value="0.759959116000226"/>
+      <inertia ixx="0.0011156254663426" ixy="3.16193221175592E-07" ixz="2.89169705133133E-06" iyy="0.00114606034071406" iyz="-8.11914906919631E-08" izz="0.000237163435713384"/>
+    </inertial>
+    <visual>
+      <origin rpy="0 0 0" xyz="0 0 0"/>
+      <geometry>
+        <mesh filename="package://robotican_arm/meshes/elbow1_link.STL"/>
+        <!-- Simplified -->
+      </geometry>
+      <material name="">
+        <color rgba="0.3 0.3 0.3 1"/>
+      </material>
+    </visual>
+    <collision>
+      <origin rpy="0 0 0" xyz="0 0 0"/>
+      <geometry>
+        <mesh filename="package://robotican_arm/meshes/elbow1_link.STL"/>
+        <!-- Simplified -->
+      </geometry>
+    </collision>
+  </link>
+  <joint name="elbow1_joint" type="revolute">
+    <origin rpy="1.44504380352115E-15 1.11628850952447E-06 -9.93431159466724E-15" xyz="0 -0.000251155668932789 0.266305434894181"/>
+    <parent link="shoulder_link"/>
+    <child link="elbow1_link"/>
+    <axis xyz="-0.999999999998754 0 0"/>
+    <limit effort="100" lower="-3.14" upper="3.14" velocity="0"/>
+  </joint>
+  <link name="elbow2_link">
+    <inertial>
+      <origin rpy="0 0 0" xyz="-2.29085121194481E-05 -0.000512185919169572 0.0885118786028204"/>
+      <mass value="1.12138857800426"/>
+      <inertia ixx="0.0011156254663426" ixy="3.04261287700186E-07" ixz="-1.22468079415109E-06" iyy="0.0110437302875007" iyz="-7.91547787630536E-05" izz="0.000331598270284794"/>
+    </inertial>
+    <visual>
+      <origin rpy="0 0 0" xyz="0 0 0"/>
+      <geometry>
+        <mesh filename="package://robotican_arm/meshes/elbow2_link.STL"/>
+        <!-- Simplified -->
+      </geometry>
+      <material name="">
+        <color rgba="0.4 0.4 0.4 1"/>
+      </material>
+    </visual>
+    <collision>
+      <origin rpy="0 0 0" xyz="0 0 0"/>
+      <geometry>
+        <mesh filename="package://robotican_arm/meshes/elbow2_link.STL"/>
+        <!-- Simplified -->
+      </geometry>
+    </collision>
+  </link>
+  <joint name="elbow2_joint" type="revolute">
+    <origin rpy="-4.51048856041191E-16 3.35869632765754E-16 0" xyz="0 0 0.223999999999899"/>
+    <parent link="elbow1_link"/>
+    <child link="elbow2_link"/>
+    <axis xyz="0 1 0"/>
+    <limit effort="10" lower="-3.14" upper="3.14" velocity="0"/>
+  </joint>
+  <link name="wrist_link">
+    <inertial>
+      <origin rpy="0 0 0" xyz="0 0 0"/>
+      <mass value="0.717337417215465"/>
+      <inertia ixx="0.000486392340366094" ixy="4.20757000035677E-12" ixz="-3.91843889020299E-06" iyy="0.000211170064630335" iyz="2.79335159568522E-12" izz="0.000437528795624211"/>
+    </inertial>
+    <visual>
+      <origin rpy="0 0 0" xyz="0 0 0"/>
+      <geometry>
+        <mesh filename="package://robotican_arm/meshes/wrist_link.STL"/>
+        <!-- Simplified -->
+      </geometry>
+      <material name="">
+        <color rgba="0.4 0.4 0.4 1"/>
+      </material>
+    </visual>
+    <collision>
+      <origin rpy="0 0 0" xyz="0 0 0"/>
+      <geometry>
+        <mesh filename="package://robotican_arm/meshes/wrist_link.STL"/>
+        <!-- Simplified -->
+      </geometry>
+    </collision>
+  </link>
+  <joint name="wrist_joint" type="revolute">
+    <origin rpy="0 0 0" xyz="0.0137 0 0.244749999999997"/>
+    <parent link="elbow2_link"/>
+    <child link="wrist_link"/>
+    <axis xyz="0 0 0.999999999998754"/>
+    <limit effort="10" lower="-3.14" upper="3.14" velocity="0"/>
+  </joint>
+  <link name="gripper_link"/>
+  <joint name="gripper_joint" type="fixed">
+  <origin xyz="0 0 0.06" rpy="0 1.570796327 0"/>
+  <parent link="wrist_link"/>
+  <child link="gripper_link"/>
+  </joint>
+  <link name="left_finger_link">
+    <inertial>
+      <origin rpy="0 0 0" xyz="-6.10622663543836E-16 0.0205697573116852 0.0301832532936965"/>
+      <mass value="0.0111981711598485"/>
+      <inertia ixx="0.000486392340366094" ixy="4.20757000035677E-12" ixz="-3.91843889020299E-06" iyy="0.000211170064630335" iyz="2.79335159568522E-12" izz="0.000437528795624211"/>
+    </inertial>
+    <visual>
+      <origin rpy="0 0 0" xyz="0 0 0"/>
+      <geometry>
+        <mesh filename="package://robotican_arm/meshes/left_finger_link.STL"/>
+        <!-- Simplified -->
+      </geometry>
+      <material name="">
+        <color rgba="0.4 0.4 0.4 1"/>
+      </material>
+    </visual>
+    <collision>
+      <origin rpy="0 0 0" xyz="0 0 0"/>
+      <geometry>
+        <mesh filename="package://robotican_arm/meshes/left_finger_link.STL"/>
+        <!-- Simplified -->
+      </geometry>
+    </collision>
+  </link>
+  <joint name="left_finger_joint" type="revolute">
+    <origin rpy="2.85979682697881E-15 1.01870746742143E-16 3.19235832636806E-21" xyz="-0.000250000000000111 0.021 0.0422500000000001"/>
+    <parent link="wrist_link"/>
+    <child link="left_finger_link"/>
+    <axis xyz="1 0 0"/>
+    <limit effort="10" lower="-3.14" upper="3.14" velocity="0"/>
+  </joint>
+  <link name="right_finger_link">
+    <inertial>
+      <origin rpy="0 0 0" xyz="2.77555756156289E-16 -0.0205697573116854 0.0301832532936965"/>
+      <mass value="0.0111981711598485"/>
+      <inertia ixx="0.000486392340366094" ixy="4.20757000035677E-12" ixz="-3.91843889020299E-06" iyy="0.000211170064630335" iyz="2.79335159568522E-12" izz="0.000437528795624211"/>
+    </inertial>
+    <visual>
+      <origin rpy="0 0 0" xyz="0 0 0"/>
+      <geometry>
+        <mesh filename="package://robotican_arm/meshes/right_finger_link.STL"/>
+        <!-- Simplified -->
+      </geometry>
+      <material name="">
+        <color rgba="0.4 0.4 0.4 1"/>
+      </material>
+    </visual>
+    <collision>
+      <origin rpy="0 0 0" xyz="0 0 0"/>
+      <geometry>
+        <mesh filename="package://robotican_arm/meshes/right_finger_link.STL"/>
+        <!-- Simplified -->
+      </geometry>
+    </collision>
+  </link>
+  <joint name="right_finger_joint" type="revolute">
+    <origin rpy="0 3.19686557214722E-37 0" xyz="-0.00024999999999889 -0.021 0.0422499999999999"/>
+    <parent link="wrist_link"/>
+    <child link="right_finger_link"/>
+    <axis xyz="1 0 0"/>
+    <limit effort="10" lower="-3.14" upper="3.14" velocity="0"/>
+  </joint>
 </robot>

Commit message: update

File: robotican_komodo/description/models/komodo_gazebo.xacro (robot description, xacro)
@@ -152,4 +152,13 @@
           </actuator>
         </transmission>
+        <transmission name="torso_joint_joint_trans">
+          <type>transmission_interface/SimpleTransmission</type>
+          <joint name="torso_joint">
+            <hardwareInterface>VelocityJointInterface</hardwareInterface>
+          </joint>
+          <actuator name="torso_joint_joint_motor">
+            <mechanicalReduction>1</mechanicalReduction>
+          </actuator>
+        </transmission>
       </xacro:if>
       <gazebo reference="FL_wheel_link">

File: robotican_komodo/description/models/komodo_torso.xacro (robot description, xacro)
@@ -77,5 +77,5 @@
   <joint
     name="torso_joint"
-    type="fixed"> <!--prismatic-->
+    type="prismatic"> <!--prismatic-->
     <origin
       xyz="0.101457996026178 0 0.0740000000000002"
@@ -90,6 +90,6 @@
 	lower="0"
 	upper="0.45"
-	effort="0"
-	velocity="0" />
+	effort="70"
+	velocity="0.0012" />
   </joint>
   <joint
