Commit message: update gazebo release

File: robotican_komodo/description/models/komodo_gazebo.xacro (robot description, xacro)
@@ -6,4 +6,6 @@
   <xacro:arg name="controllers" default="true"/>
   <xacro:arg name="front_camera" default="false"/>
+  <xacro:arg name="rear_camera" default="false"/>
+  <xacro:arg name="top_camera" default="false"/>
   <xacro:arg name="urf" default="false"/>
   <xacro:arg name="imu" default="false"/>
@@ -11,7 +13,74 @@
   <xacro:arg name="lidar" default="false"/>
   <xacro:arg name="depth_camera" default="false"/>
-  <!-- Asus -->
-  <xacro:if value="$(arg depth_camera)">
-    <xacro:include filename="$(find robotican_common)/gazebo/asus_xtion_pro_live.xacro" />
+  <xacro:arg name="torso_camera" default="false"/>
+  <xacro:arg name="arm_camera" default="false"/>
+  <!-- torso_camera -->
+  <xacro:if value="$(arg torso_camera)">
+    <gazebo reference="torso_camera_link">
+        <sensor type="depth" name="torso_camera">
+          <update_rate>20</update_rate>
+          <camera>
+            <horizontal_fov>${62.8 * M_PI/180.0}</horizontal_fov>
+            <image>
+              <format>B8G8R8</format>
+              <width>640</width>
+              <height>480</height>
+            </image>
+            <clip>
+              <near>0.5</near>
+              <far>9</far>
+            </clip>
+          </camera>
+          <plugin name="depth_camera_controller" filename="libgazebo_ros_openni_kinect.so">
+            <alwaysOn>true</alwaysOn>
+            <updateRate>20</updateRate>
+            <imageTopicName>torso_camera/rgb/image_raw</imageTopicName>
+            <cameraInfoTopicName>torso_camera/rgb/camera_info</cameraInfoTopicName>
+            <depthImageTopicName>torso_camera/depth_registered/image_raw</depthImageTopicName>
+            <depthImageCameraInfoTopicName>torso_camera/depth_registered/camera_info</depthImageCameraInfoTopicName>
+            <pointCloudTopicName>torso_camera/depth_registered/points</pointCloudTopicName>
+            <frameName>torso_camera_depth_optical_frame</frameName>
+            <distortion_k1>0.0</distortion_k1>
+            <distortion_k2>0.0</distortion_k2>
+            <distortion_k3>0.0</distortion_k3>
+            <distortion_t1>0.0</distortion_t1>
+            <distortion_t2>0.0</distortion_t2>
+          </plugin>
+        </sensor>
+		</gazebo>
+  </xacro:if>
+    <xacro:if value="$(arg arm_camera)">
+    <gazebo reference="creative_camera_link">
+        <sensor type="depth" name="creative_camera">
+          <update_rate>20</update_rate>
+          <camera>
+            <horizontal_fov>${62.8 * M_PI/180.0}</horizontal_fov>
+            <image>
+              <format>B8G8R8</format>
+              <width>640</width>
+              <height>480</height>
+            </image>
+            <clip>
+              <near>0.5</near>
+              <far>9</far>
+            </clip>
+          </camera>
+          <plugin name="depth_camera_controller" filename="libgazebo_ros_openni_kinect.so">
+            <alwaysOn>true</alwaysOn>
+            <updateRate>20</updateRate>
+            <imageTopicName>arm_camera/rgb/image_raw</imageTopicName>
+            <cameraInfoTopicName>arm_camera/rgb/camera_info</cameraInfoTopicName>
+            <depthImageTopicName>arm_camera/depth_registered/image_raw</depthImageTopicName>
+            <depthImageCameraInfoTopicName>arm_camera/depth_registered/camera_info</depthImageCameraInfoTopicName>
+            <pointCloudTopicName>arm_camera/depth_registered/points</pointCloudTopicName>
+            <frameName>creative_camera_depth_optical_frame</frameName>
+            <distortion_k1>0.0</distortion_k1>
+            <distortion_k2>0.0</distortion_k2>
+            <distortion_k3>0.0</distortion_k3>
+            <distortion_t1>0.0</distortion_t1>
+            <distortion_t2>0.0</distortion_t2>
+          </plugin>
+        </sensor>
+    </gazebo>
   </xacro:if>
   <!-- Sonars -->
@@ -43,6 +112,12 @@
     <xacro:include filename="$(find robotican_common)/gazebo/camera.xacro" />
     <xacro:if value="$(arg front_camera)">
-      <xacro:Camera name="front_camera" link="front_cam_link" image_width="640" image_height="480"  image_format="R8G8B8" clip_near="0.02" clip_far="300" />
-      </xacro:if>
+		<xacro:Camera name="front_camera" link="front_cam_link" image_width="640" image_height="480"  image_format="R8G8B8" clip_near="0.02" clip_far="300" />
+    </xacro:if>
+    <xacro:if value="$(arg rear_camera)">
+		<xacro:Camera name="rear_camera" link="rear_camera_link" image_width="640" image_height="480"  image_format="R8G8B8" clip_near="0.02" clip_far="300" />
+    </xacro:if>
+    <xacro:if value="$(arg top_camera)">
+		<xacro:Camera name="top_camera" link="top_camera_link" image_width="640" image_height="480"  image_format="R8G8B8" clip_near="0.02" clip_far="300" />
+    </xacro:if>
       <!-- controller manager and hardware interfaces -->
       <xacro:if value="$(arg controllers)">

File: robotican_komodo/description/models/komodo_torso.xacro (robot description, xacro)
@@ -300,5 +300,5 @@
     <child link="left_finger_link"/>
     <axis xyz="1 0 0"/>
-    <limit effort="10" lower="-3.14" upper="3.14" velocity="0"/>
+    <limit effort="3.1" lower="-1.57" upper="1.57" velocity="2.0"/>
   </joint>
   <link name="right_finger_link">
@@ -331,8 +331,8 @@
     <child link="right_finger_link"/>
     <axis xyz="1 0 0"/>
-    <limit effort="10" lower="-3.14" upper="3.14" velocity="0"/>
+    <limit effort="3.1" lower="-1.57" upper="1.57" velocity="2.0"/>
   </joint>
   <link
-    name="Creative_Camera_link">
+    name="creative_camera_link">
     <inertial>
       <origin
@@ -374,5 +374,5 @@
   </link>
   <joint
-    name="Creative_Camera_joint"
+    name="creative_camera_joint"
     type="fixed">
     <origin
@@ -382,8 +382,62 @@
       link="wrist_link" />
     <child
-      link="Creative_Camera_link" />
+      link="creative_camera_link" />
     <axis
       xyz="0 0 0" />
   </joint>
+<joint name="creative_camera_rgb_joint" type="fixed">
+      <origin xyz="0 0.0185 0" rpy="0 0 0"/>
+      <parent link="creative_camera_link"/>
+      <child link="creative_camera_rgb_frame" />
+    </joint>
+    <link name="creative_camera_rgb_frame">
+      <inertial>
+  <mass value="0.001" />
+  <origin xyz="0 0 0" />
+  <inertia ixx="0.0001" ixy="0.0" ixz="0.0"
+    iyy="0.0001" iyz="0.0"
+    izz="0.0001" />
+  </inertial>
+      </link>
+      <joint name="creative_camera_rgb_optical_joint" type="fixed">
+  <origin xyz="0 0 0" rpy="${-M_PI/2} 0 ${-M_PI/2}" />
+  <parent link="creative_camera_rgb_frame" />
+  <child link="creative_camera_rgb_optical_frame" />
+      </joint>
+      <link name="creative_camera_rgb_optical_frame">
+  <inertial>
+    <mass value="0.001" />
+    <origin xyz="0 0 0" />
+    <inertia ixx="0.0001" ixy="0.0" ixz="0.0"
+      iyy="0.0001" iyz="0.0"
+      izz="0.0001" />
+    </inertial>
+  </link>
+  <joint name="creative_camera_depth_joint" type="fixed">
+    <origin xyz="0 0.0445 0" rpy="0 0 0" />
+    <parent link="creative_camera_link" />
+    <child link="creative_camera_depth_frame" />
+  </joint>
+  <link name="creative_camera_depth_frame">
+    <inertial>
+      <mass value="0.001" />
+      <origin xyz="0 0 0" />
+      <inertia ixx="0.0001" ixy="0.0" ixz="0.0"
+        iyy="0.0001" iyz="0.0"
+        izz="0.0001" />
+      </inertial>
+    </link>
+    <joint name="creative_camera_depth_optical_joint" type="fixed">
+      <origin xyz="0 0 0" rpy="${-M_PI/2} 0 ${-M_PI/2}" />
+      <parent link="creative_camera_depth_frame" />
+      <child link="creative_camera_depth_optical_frame" />
+    </joint>
+    <link name="creative_camera_depth_optical_frame">
+      <inertial>
+        <mass value="0.001" />
+        <origin xyz="0 0 0" />
+        <inertia ixx="0.0001" ixy="0.0" ixz="0.0" iyy="0.0001" iyz="0.0" izz="0.0001" />
+        </inertial>
+      </link>
   <link
       name="torso_camera_link">
@@ -511,5 +565,5 @@
       <origin
         xyz="0 0 0"
-        rpy="5.38354147863953E-15 1.55701850396119E-12 -1.56733874423455" />
+        rpy="0 1.57 0" />
       <geometry>
         <mesh
@@ -537,5 +591,5 @@
     <origin
       xyz="0.0622079960261761 0.0152829991418538 0.660000000000001"
-      rpy="0 0.0 0" />
+      rpy="0 -1.57 0" />
     <parent
       link="arm_base_link" />
@@ -545,3 +599,57 @@
       xyz="0 0 0" />
   </joint>
+<joint name="torso_camera_rgb_joint" type="fixed">
+      <origin xyz="0 0.0185 0" rpy="0 0 0"/>
+      <parent link="torso_camera_link"/>
+      <child link="torso_camera_rgb_frame" />
+    </joint>
+    <link name="torso_camera_rgb_frame">
+      <inertial>
+  <mass value="0.001" />
+  <origin xyz="0 0 0" />
+  <inertia ixx="0.0001" ixy="0.0" ixz="0.0"
+    iyy="0.0001" iyz="0.0"
+    izz="0.0001" />
+  </inertial>
+      </link>
+      <joint name="torso_camera_rgb_optical_joint" type="fixed">
+  <origin xyz="0 0 0" rpy="${-M_PI/2} 0 ${-M_PI/2}" />
+  <parent link="torso_camera_rgb_frame" />
+  <child link="torso_camera_rgb_optical_frame" />
+      </joint>
+      <link name="torso_camera_rgb_optical_frame">
+  <inertial>
+    <mass value="0.001" />
+    <origin xyz="0 0 0" />
+    <inertia ixx="0.0001" ixy="0.0" ixz="0.0"
+      iyy="0.0001" iyz="0.0"
+      izz="0.0001" />
+    </inertial>
+  </link>
+  <joint name="torso_camera_depth_joint" type="fixed">
+    <origin xyz="0 0.0445 0" rpy="0 0 0" />
+    <parent link="torso_camera_link" />
+    <child link="torso_camera_depth_frame" />
+  </joint>
+  <link name="torso_camera_depth_frame">
+    <inertial>
+      <mass value="0.001" />
+      <origin xyz="0 0 0" />
+      <inertia ixx="0.0001" ixy="0.0" ixz="0.0"
+        iyy="0.0001" iyz="0.0"
+        izz="0.0001" />
+      </inertial>
+    </link>
+    <joint name="torso_camera_depth_optical_joint" type="fixed">
+      <origin xyz="0 0 0" rpy="${-M_PI/2} 0 ${-M_PI/2}" />
+      <parent link="torso_camera_depth_frame" />
+      <child link="torso_camera_depth_optical_frame" />
+    </joint>
+    <link name="torso_camera_depth_optical_frame">
+      <inertial>
+        <mass value="0.001" />
+        <origin xyz="0 0 0" />
+        <inertia ixx="0.0001" ixy="0.0" ixz="0.0" iyy="0.0001" iyz="0.0" izz="0.0001" />
+        </inertial>
+      </link>
 </robot>

Commit message: softkinetic implemetation fix

File: robotican_komodo/description/models/komodo_gazebo.xacro (robot description, xacro)
@@ -12,9 +12,8 @@
   <xacro:arg name="gps" default="false"/>
   <xacro:arg name="lidar" default="false"/>
-  <xacro:arg name="depth_camera" default="false"/>
-  <xacro:arg name="torso_camera" default="false"/>
+  <xacro:arg name="asus_camera" default="false"/>
   <xacro:arg name="arm_camera" default="false"/>
   <!-- torso_camera -->
-  <xacro:if value="$(arg torso_camera)">
+  <xacro:if value="$(arg asus_camera)">
     <gazebo reference="torso_camera_link">
         <sensor type="depth" name="torso_camera">

File: robotican_komodo/description/models/komodo_torso.xacro (robot description, xacro)
@@ -328,4 +328,8 @@
     <limit effort="3.1" lower="-1.57" upper="1.57" velocity="2.0"/>
   </joint>
+<sensor_senz3d parent="wrist_link" name="softkinetic_camera" v_offset_x="0.045" v_offset_y="0.0" v_offset_z="0.0">
+    <origin xyz="-0.05905 0 0.0753" rpy="0.0 -${M_PI/2} 0.0"/>
+  </sensor_senz3d>
+<!--
   <link
     name="softkinetic_camera_link">
@@ -350,5 +354,5 @@
       <geometry>
         <mesh
-          filename="package://robotican_common/description/meshes/creative_camera_link.STL" />
+          filename="package://robotican_common/models/softkinetic_camera_ds325/softkinetic_camera_ds325.STL" />
       </geometry>
       <material
@@ -364,5 +368,5 @@
       <geometry>
         <mesh
-          filename="package://robotican_komodo/description/meshes/creative_camera_link.STL" />
+          filename="package://robotican_common/models/softkinetic_camera_ds325/softkinetic_camera_ds325.STL" />
       </geometry>
     </collision>
@@ -435,4 +439,5 @@
         </inertial>
       </link>
+      -->
   <link
       name="torso_camera_link">

File: robotican_manipulator_h/models/manipulator_h.xacro (robot description, xacro)
@@ -516,5 +516,5 @@
       <dynamics friction ="1000" damping="100"/>
   </joint>
-  <sensor_senz3d parent="wrist_link" name="softkinetic_camera_link" v_offset_x="0.045" v_offset_y="0.0" v_offset_z="0.0">
+  <sensor_senz3d parent="wrist_link" name="softkinetic_camera" v_offset_x="0.045" v_offset_y="0.0" v_offset_z="0.0">
     <origin xyz="-0.05905 0 0.0753" rpy="0.0 -${M_PI/2} 0.0"/>
   </sensor_senz3d>

File: robotican_manipulator_h/models/manipulator_h_gazebo.xacro (robot description, xacro)
@@ -3,8 +3,7 @@
 	<xacro:include filename="$(find robotican_manipulator_h)/models/manipulator_h.xacro" />
 	<xacro:include filename="$(find robotican_manipulator_h)/models/manipulator_h_gazebo_plugins.xacro" />
-	  <xacro:arg name="sr300" default="false"/>
-	    <!-- SR300 -->
-  <xacro:if value="$(arg sr300)">
-    <xacro:include filename="$(find robotican_common)/gazebo/sr300.xacro" />
+	  <xacro:arg name="softkinetic" default="false"/>
+  <xacro:if value="$(arg softkinetic)">
+    <xacro:include filename="$(find robotican_common)/gazebo/softkinetic_camera_ds325.xacro" />
   </xacro:if>
    <link name="world" />
