Commit message: update

File: robotican_manipulator_h/models/manipulator_h.xacro (robot description, xacro)
@@ -3,4 +3,38 @@
   name="robotican_manipulator_h" description="Manipulator H Arm" xmlns:xacro="http://www.ros.org/wiki/xacro">
   <xacro:property name="M_PI" value="3.1415926535897931" />
+  <link name="arm_link">
+    <inertial>
+      <origin xyz="-0.022197 -1.9122E-07 0.044251" rpy="0 0 0" />
+      <mass value="0.16757" />
+      <inertia
+      ixx="0.00062908"
+      ixy="-8.3342E-10"
+      ixz="-0.00014877"
+      iyy="0.0010719"
+      iyz="1.6859E-09"
+      izz="0.0013427" />
+    </inertial>
+    <visual>
+      <origin xyz="0 0 0" rpy="0 0 0" />
+      <geometry>
+        <mesh filename="package://robotican_manipulator_h/meshes/arm_link.STL" />
+      </geometry>
+      <material name="">
+        <color rgba="0.79216 0.81961 0.93333 1" />
+      </material>
+    </visual>
+    <collision>
+      <origin xyz="0 0 0" rpy="0 0 0" />
+      <geometry>
+        <mesh filename="package://robotican_manipulator_h/meshes/arm_link.STL" />
+      </geometry>
+    </collision>
+  </link>
+  <joint name="base_arm_joint" type="fixed">
+    <origin xyz="-0.091 0 0.093" rpy="0 0 0" />
+    <parent link="arm_link" />
+    <child link="base_arm_link" />
+    <axis xyz="0 0 0" />
+  </joint>
   <link
     name="base_arm_link">

Commit message: update

File: robotican_manipulator_h/models/manipulator_h.xacro (robot description, xacro)
@@ -3,38 +3,4 @@
   name="robotican_manipulator_h" description="Manipulator H Arm" xmlns:xacro="http://www.ros.org/wiki/xacro">
   <xacro:property name="M_PI" value="3.1415926535897931" />
-  <link name="arm_link">
-    <inertial>
-      <origin xyz="-0.022197 -1.9122E-07 0.044251" rpy="0 0 0" />
-      <mass value="0.16757" />
-      <inertia
-      ixx="0.00062908"
-      ixy="-8.3342E-10"
-      ixz="-0.00014877"
-      iyy="0.0010719"
-      iyz="1.6859E-09"
-      izz="0.0013427" />
-    </inertial>
-    <visual>
-      <origin xyz="0 0 0" rpy="0 0 0" />
-      <geometry>
-        <mesh filename="package://robotican_manipulator_h/meshes/arm_link.STL" />
-      </geometry>
-      <material name="">
-        <color rgba="0.79216 0.81961 0.93333 1" />
-      </material>
-    </visual>
-    <collision>
-      <origin xyz="0 0 0" rpy="0 0 0" />
-      <geometry>
-        <mesh filename="package://robotican_manipulator_h/meshes/arm_link.STL" />
-      </geometry>
-    </collision>
-  </link>
-  <joint name="base_arm_joint" type="fixed">
-    <origin xyz="-0.091 0 0.093" rpy="0 0 0" />
-    <parent link="arm_link" />
-    <child link="base_arm_link" />
-    <axis xyz="0 0 0" />
-  </joint>
   <link
     name="base_arm_link">

Commit message: update

File: robotican_manipulator_h/models/manipulator_h.xacro (robot description, xacro)
@@ -571,5 +571,5 @@
 -->
   <sensor_senz3d parent="wrist_link" name="softkinetic_camera">
-    <origin xyz="-0.06355 0 0.041852" rpy="0.0 -${M_PI/2} 0.0"/>
+    <origin xyz="-0.05905 0 0.0303" rpy="0.0 -${M_PI/2} 0.0"/>
   </sensor_senz3d>
 </robot>

Commit message: trying to fix model

File: robotican_manipulator_h/models/manipulator_h.xacro (robot description, xacro)
@@ -570,6 +570,6 @@
   </joint>
 -->
-  <sensor_senz3d parent="wrist_link" name="softkinetic_camera" v_offset_x="0.035" v_offset_y="0.0" v_offset_z="0.0">
-    <origin xyz="-0.05905 0 0.0653" rpy="0.0 -${M_PI/2} 0.0"/>
+  <sensor_senz3d parent="wrist_link" name="softkinetic_camera" v_offset_x="0.055" v_offset_y="0.0" v_offset_z="0.0">
+    <origin xyz="-0.05905 0 0.0853" rpy="0.0 -${M_PI/2} 0.0"/>
   </sensor_senz3d>
 </robot>

Commit message: trying to fix model

File: robotican_manipulator_h/models/manipulator_h.xacro (robot description, xacro)
@@ -570,6 +570,6 @@
   </joint>
 -->
-  <sensor_senz3d parent="wrist_link" name="softkinetic_camera" v_offset_x="0.055" v_offset_y="0.0" v_offset_z="0.0">
-    <origin xyz="-0.05905 0 0.0853" rpy="0.0 -${M_PI/2} 0.0"/>
+  <sensor_senz3d parent="wrist_link" name="softkinetic_camera" v_offset_x="0.075" v_offset_y="0.0" v_offset_z="0.0">
+    <origin xyz="-0.05905 0 0.1053" rpy="0.0 -${M_PI/2} 0.0"/>
   </sensor_senz3d>
 </robot>

Commit message: update

File: robotican_manipulator_h/models/manipulator_h.xacro (robot description, xacro)
@@ -570,6 +570,6 @@
   </joint>
 -->
-  <sensor_senz3d parent="wrist_link" name="softkinetic_camera" v_offset_x="0.075" v_offset_y="0.0" v_offset_z="0.0">
-    <origin xyz="-0.05905 0 0.1053" rpy="0.0 -${M_PI/2} 0.0"/>
+  <sensor_senz3d parent="wrist_link" name="softkinetic_camera" v_offset_x="0.055" v_offset_y="0.0" v_offset_z="0.0">
+    <origin xyz="-0.05905 0 0.0853" rpy="0.0 -${M_PI/2} 0.0"/>
   </sensor_senz3d>
 </robot>

Commit message: update fix soft tf;

File: robotican_manipulator_h/models/manipulator_h.xacro (robot description, xacro)
@@ -570,6 +570,6 @@
   </joint>
 -->
-  <sensor_senz3d parent="wrist_link" name="softkinetic_camera" v_offset_x="0.055" v_offset_y="0.0" v_offset_z="0.0">
-    <origin xyz="-0.05905 0 0.0853" rpy="0.0 -${M_PI/2} 0.0"/>
+  <sensor_senz3d parent="wrist_link" name="softkinetic_camera" v_offset_x="0.045" v_offset_y="0.0" v_offset_z="0.0">
+    <origin xyz="-0.05905 0 0.0753" rpy="0.0 -${M_PI/2} 0.0"/>
   </sensor_senz3d>
 </robot>

Commit message: change arm ctrl

File: robotican_manipulator_h/models/manipulator_h.xacro (robot description, xacro)
@@ -3,5 +3,4 @@
   name="robotican_manipulator_h" description="Manipulator H Arm" xmlns:xacro="http://www.ros.org/wiki/xacro">
   <xacro:property name="M_PI" value="3.1415926535897931" />
-  <xacro:include filename="$(find robotican_common)/models/softkinetic_camera_ds325/model.xacro" />
   <link
     name="base_arm_link">
@@ -516,5 +515,4 @@
       <dynamics friction ="1000" damping="100"/>
   </joint>
-<!--
   <link
     name="sr300_link">
@@ -569,7 +567,3 @@
       xyz="0 0 0" />
   </joint>
--->
-  <sensor_senz3d parent="wrist_link" name="softkinetic_camera" v_offset_x="0.045" v_offset_y="0.0" v_offset_z="0.0">
-    <origin xyz="-0.05905 0 0.0753" rpy="0.0 -${M_PI/2} 0.0"/>
-  </sensor_senz3d>
 </robot>

Commit message: softkinetic link changes

File: robotican_manipulator_h/models/manipulator_h.xacro (robot description, xacro)
@@ -3,4 +3,5 @@
   name="robotican_manipulator_h" description="Manipulator H Arm" xmlns:xacro="http://www.ros.org/wiki/xacro">
   <xacro:property name="M_PI" value="3.1415926535897931" />
+  <xacro:include filename="$(find robotican_common)/models/softkinetic_camera_ds325/model.xacro" />
   <link
     name="base_arm_link">
@@ -515,4 +516,5 @@
       <dynamics friction ="1000" damping="100"/>
   </joint>
+<!--
   <link
     name="sr300_link">
@@ -567,3 +569,7 @@
       xyz="0 0 0" />
   </joint>
+-->
+  <sensor_senz3d parent="wrist_link" name="softkinetic_camera" v_offset_x="0.045" v_offset_y="0.0" v_offset_z="0.0">
+    <origin xyz="-0.05905 0 0.0753" rpy="0.0 -${M_PI/2} 0.0"/>
+  </sensor_senz3d>
 </robot>

Commit message: fresh komodo installation

File: robotican_manipulator_h/models/manipulator_h.xacro (robot description, xacro)
@@ -516,59 +516,5 @@
       <dynamics friction ="1000" damping="100"/>
   </joint>
-<!--
-  <link
-    name="sr300_link">
-    <inertial>
-      <origin
-        xyz="-0.015404 -1.7297E-09 -0.007331"
-        rpy="0 0 0" />
-      <mass
-        value="0.092188" />
-      <inertia
-        ixx="0.00012728"
-        ixy="-5.5477E-12"
-        ixz="5.4874E-06"
-        iyy="2.6617E-05"
-        iyz="-4.8961E-11"
-        izz="0.00013363" />
-    </inertial>
-    <visual>
-      <origin
-        xyz="0 0 0"
-        rpy="0 0 0" />
-      <geometry>
-        <mesh
-          filename="package://robotican_manipulator_h/meshes/sr300_optical_link.STL" />
-      </geometry>
-      <material
-        name="">
-        <color
-          rgba="0.1 0.1 0.1 1" />
-      </material>
-    </visual>
-    <collision>
-      <origin
-        xyz="0 0 0"
-        rpy="0 0 0" />
-      <geometry>
-        <mesh filename="package://robotican_manipulator_h/meshes/sr300_optical_link.STL" />
-      </geometry>
-    </collision>
-  </link>
-  <joint
-    name="sr300_joint"
-    type="fixed">
-    <origin
-      xyz="-0.06355 0 0.041852"
-      rpy="0 -1.5708 0" />
-    <parent
-      link="wrist_link" />
-    <child
-      link="sr300_link" />
-    <axis
-      xyz="0 0 0" />
-  </joint>
--->
-  <sensor_senz3d parent="wrist_link" name="softkinetic_camera" v_offset_x="0.045" v_offset_y="0.0" v_offset_z="0.0">
+  <sensor_senz3d parent="wrist_link" name="softkinetic_camera_link" v_offset_x="0.045" v_offset_y="0.0" v_offset_z="0.0">
     <origin xyz="-0.05905 0 0.0753" rpy="0.0 -${M_PI/2} 0.0"/>
   </sensor_senz3d>
