Commit message: update

File: robotican_arm/models/arm.xacro (robot description, xacro)
@@ -1,34 +1,98 @@
 <?xml version="1.0"?>
 <robot xmlns:xacro="http://www.ros.org/wiki/xacro" name="robotican_arm" description="robotican arm">
-	  <link name="arm_base_link">
-    <inertial>
-      <origin rpy="0 0 0" xyz="0.0 0.0 0.0"/>
-      <mass value="1.08982930885161"/>
-      <inertia ixx="0.00311458437968986" ixy="-7.0610782277189E-06" ixz="-0.000262941654993437" iyy="0.00855106134499406" iyz="1.00391927392762E-06" izz="0.0104177337437887"/>
-    </inertial>
-    <visual>
-      <origin rpy="0 0 0" xyz="0 0 0"/>
-      <geometry>
-        <mesh filename="package://robotican_arm/meshes/arm_base_link.STL"/>
-      </geometry>
-      <material name="">
-        <color rgba="0.4 0.4 0.4 1"/>
-      </material>
-    </visual>
-    <collision>
-      <origin rpy="0 0 0" xyz="0 0 0"/>
-      <geometry>
-        <mesh filename="package://robotican_arm/meshes/arm_base_link.STL"/>
-      </geometry>
-    </collision>
-  </link>
-   <joint
+<link name="arm_base_link">
+    <inertial>
+      <origin xyz="0.0787832367713514 1.63894955207658E-05 0.30372182598738" rpy="0 0 0" />
+      <mass value="5.82785061945851" />
+      <inertia
+        ixx="0.262040399352781"
+        ixy="-1.20613586206922E-05"
+        ixz="0.0219696026578"
+        iyy="0.271705564666912"
+        iyz="3.10612186063073E-05"
+        izz="0.0337682852586326" />
+    </inertial>
+    <visual>
+      <origin xyz="0 0 0" rpy="0 0 0" />
+      <geometry>
+        <mesh filename="package://robotican_komodo/description/meshes/arm_base_link.STL" />
+      </geometry>
+      <material name="">
+        <color rgba="0.4 0.4 0.4 1" />
+      </material>
+    </visual>
+    <collision>
+      <origin xyz="0 0 0" rpy="0 0 0" />
+      <geometry>
+        <mesh filename="package://robotican_komodo/description/meshes/arm_base_link.STL" />
+      </geometry>
+    </collision>
+  </link>
+   <link
+    name="torso_link">
+    <inertial>
+      <origin
+        xyz="0.0954671716579415 1.91586249009607E-06 -0.0185743175743276"
+        rpy="0 0 0" />
+      <mass
+        value="1.09057945344451" />
+      <inertia
+        ixx="0.000835857275985966"
+        ixy="5.81870910353681E-08"
+        ixz="-3.13493979506258E-05"
+        iyy="0.00128840659932805"
+        iyz="1.45397132642805E-07"
+        izz="0.00136461371089342" />
+    </inertial>
+    <visual>
+      <origin
+        xyz="0 0 0"
+        rpy="0 0 0" />
+      <geometry>
+        <mesh
+          filename="package://robotican_komodo/description/meshes/torso_link.STL" />
+      </geometry>
+      <material
+        name="">
+        <color
+          rgba="0.35 0.35 0.35 1" />
+      </material>
+    </visual>
+    <collision>
+      <origin
+        xyz="0 0 0"
+        rpy="0 0 0" />
+      <geometry>
+        <mesh
+          filename="package://robotican_komodo/description/meshes/torso_link.STL" />
+      </geometry>
+    </collision>
+  </link>
+  <joint
+    name="torso_joint"
+    type="fixed"> <!--prismatic-->
+    <origin
+      xyz="0.101457996026178 0 0.0740000000000002"
+      rpy="0 0 0" />
+    <parent
+      link="arm_base_link" />
+    <child
+      link="torso_link" />
+    <axis
+      xyz="0 0 1" />
+   <limit
+	lower="0"
+	upper="0.45"
+	effort="0"
+	velocity="0" />
+  </joint>
+  <joint
     name="base_rotation_joint"
     type="revolute">
     <origin
-      xyz="-0.096277996026178 0 0.0549000000000002"
-      rpy="-5.46369598732866E-16 1.34659130519145E-15 -2.1922983760752E-31" />
+      xyz="0.113 0 -0.00400000000000003"
+      rpy="0 0 0" />
     <parent
-      link="arm_base_link" />
+      link="torso_link" />
     <child
       link="base_rotation_link" />
@@ -41,18 +105,18 @@
       velocity="0" />
   </joint>
-	<link name="base_rotation_link">
+  <link name="base_rotation_link">
     <inertial>
       <origin
-      	rpy="0 0 0"
-      	xyz="-1.11022302462516E-16 -7.80223872637444E-17 0.0660708417371112"/>
+        rpy="0 0 0"
+        xyz="-6.93889390390723E-17 1.46538271444029E-17 0.0623331826247039"/>
       <mass
-      	value="1.4054258533062"/>
+        value="1.4054258533062"/>
       <inertia
-      	ixx="0.00159425912810341"
-      	ixy="-8.40269196653518E-08"
-      	ixz="-1.60925604895535E-19"
-      	iyy="0.000605522001732049"
-      	iyz="-6.08768470792684E-19"
-      	izz="0.00123388334665811"/>
+        ixx="0.00159425912810341"
+        ixy="-8.40269196653518E-08"
+        ixz="-1.60925604895535E-19"
+        iyy="0.000605522001732049"
+        iyz="-6.08768470792684E-19"
+        izz="0.00123388334665811"/>
     </inertial>
     <visual>
@@ -74,5 +138,5 @@
   <link name="shoulder_link">
     <inertial>
-      <origin rpy="0 0 0" xyz="-4.66231481405233E-06 -9.82289126283389E-05 0.0772888499682157"/>
+      <origin rpy="0 0 0" xyz="4.66247777455853E-06 -9.82289263772941E-05 0.0772888499398813"/>
       <mass value="0.191480823048406"/>
       <inertia ixx="0.00107301595696304" ixy="-2.9789063890745E-07" ixz="-2.01216953964121E-08" iyy="0.000975953125213584" iyz="-1.19601921452086E-06" izz="0.000217659789393094"/>
@@ -96,5 +160,5 @@
   </link>
   <joint name="shoulder_joint" type="revolute">
-    <origin rpy="-4.20159904047482E-15 -5.97509793174248E-16 9.93431320775303E-15" xyz="0 0 0.0834999999999999"/>
+    <origin rpy="-4.20159904047482E-15 -5.97509793174248E-16 9.93431320775303E-15" xyz="0 0 0.0835"/>
     <parent link="base_rotation_link"/>
     <child link="shoulder_link"/>
@@ -104,5 +168,5 @@
   <link name="elbow1_link">
     <inertial>
-      <origin rpy="0 0 0" xyz="3.38561240652013E-05 2.66604610292575E-06 0.0239321015909688"/>
+      <origin rpy="0 0 0" xyz="3.38829306132937E-05 2.66620552362602E-06 0.0239321015118659"/>
       <mass value="0.759959116000226"/>
       <inertia ixx="0.0011156254663426" ixy="3.16193221175592E-07" ixz="2.89169705133133E-06" iyy="0.00114606034071406" iyz="-8.11914906919631E-08" izz="0.000237163435713384"/>
@@ -127,5 +191,5 @@
   </link>
   <joint name="elbow1_joint" type="revolute">
-    <origin rpy="1.44504380352115E-15 1.11628850952447E-06 -9.93431159466724E-15" xyz="0 -0.000251155668932789 0.266305434894181"/>
+    <origin rpy="1.44504380352115E-15 1.11628850952447E-06 -9.93431159466724E-15" xyz="0 -0.000251155668931501 0.266305434894181"/>
     <parent link="shoulder_link"/>
     <child link="elbow1_link"/>
@@ -135,5 +199,5 @@
   <link name="elbow2_link">
     <inertial>
-      <origin rpy="0 0 0" xyz="-2.29085121194481E-05 -0.000512185919169572 0.0885118786028204"/>
+      <origin rpy="0 0 0" xyz="0.000512284668490459 -2.29084833272284E-05 0.0885118785637893"/>
       <mass value="1.12138857800426"/>
       <inertia ixx="0.0011156254663426" ixy="3.04261287700186E-07" ixz="-1.22468079415109E-06" iyy="0.0110437302875007" iyz="-7.91547787630536E-05" izz="0.000331598270284794"/>
@@ -158,5 +222,5 @@
   </link>
   <joint name="elbow2_joint" type="revolute">
-    <origin rpy="-4.51048856041191E-16 3.35869632765754E-16 0" xyz="0 0 0.223999999999899"/>
+    <origin rpy="-4.51048856041191E-16 3.35869632765754E-16 0" xyz="0 0 0.22399999999847"/>
     <parent link="elbow1_link"/>
     <child link="elbow2_link"/>
@@ -166,5 +230,5 @@
   <link name="wrist_link">
     <inertial>
-      <origin rpy="0 0 0" xyz="0 0 0"/>
+      <origin rpy="0 0 0" xyz="0.0303673809619356 4.00707611352118E-10 0.000140374211043737"/>
       <mass value="0.717337417215465"/>
       <inertia ixx="0.000486392340366094" ixy="4.20757000035677E-12" ixz="-3.91843889020299E-06" iyy="0.000211170064630335" iyz="2.79335159568522E-12" izz="0.000437528795624211"/>
@@ -189,5 +253,5 @@
   </link>
   <joint name="wrist_joint" type="revolute">
-    <origin rpy="0 0 0" xyz="0.0137 0 0.244749999999997"/>
+    <origin rpy="0 0 0" xyz="0.0131002732116043 0 0.244749985376465"/>
     <parent link="elbow2_link"/>
     <child link="wrist_link"/>
@@ -197,7 +261,7 @@
   <link name="gripper_link"/>
   <joint name="gripper_joint" type="fixed">
-	<origin xyz="0 0 0.06" rpy="0 1.570796327 0"/>
-	<parent link="wrist_link"/>
-	<child link="gripper_link"/>
+  <origin xyz="0 0 0.06" rpy="0 1.570796327 0"/>
+  <parent link="wrist_link"/>
+  <child link="gripper_link"/>
   </joint>
   <link name="left_finger_link">

File: robotican_komodo/description/models/komodo_torso.xacro (robot description, xacro)
@@ -115,5 +115,5 @@
       <origin
         rpy="0 0 0"
-        xyz="-1.11022302462516E-16 -7.80223872637444E-17 0.0660708417371112"/>
+        xyz="-6.93889390390723E-17 1.46538271444029E-17 0.0623331826247039"/>
       <mass
         value="1.4054258533062"/>
@@ -144,5 +144,5 @@
   <link name="shoulder_link">
     <inertial>
-      <origin rpy="0 0 0" xyz="-4.66231481405233E-06 -9.82289126283389E-05 0.0772888499682157"/>
+      <origin rpy="0 0 0" xyz="4.66247777455853E-06 -9.82289263772941E-05 0.0772888499398813"/>
       <mass value="0.191480823048406"/>
       <inertia ixx="0.00107301595696304" ixy="-2.9789063890745E-07" ixz="-2.01216953964121E-08" iyy="0.000975953125213584" iyz="-1.19601921452086E-06" izz="0.000217659789393094"/>
@@ -166,5 +166,5 @@
   </link>
   <joint name="shoulder_joint" type="revolute">
-    <origin rpy="-4.20159904047482E-15 -5.97509793174248E-16 9.93431320775303E-15" xyz="0 0 0.0834999999999999"/>
+    <origin rpy="-4.20159904047482E-15 -5.97509793174248E-16 9.93431320775303E-15" xyz="0 0 0.0835"/>
     <parent link="base_rotation_link"/>
     <child link="shoulder_link"/>
@@ -174,5 +174,5 @@
   <link name="elbow1_link">
     <inertial>
-      <origin rpy="0 0 0" xyz="3.38561240652013E-05 2.66604610292575E-06 0.0239321015909688"/>
+      <origin rpy="0 0 0" xyz="3.38829306132937E-05 2.66620552362602E-06 0.0239321015118659"/>
       <mass value="0.759959116000226"/>
       <inertia ixx="0.0011156254663426" ixy="3.16193221175592E-07" ixz="2.89169705133133E-06" iyy="0.00114606034071406" iyz="-8.11914906919631E-08" izz="0.000237163435713384"/>
@@ -197,5 +197,5 @@
   </link>
   <joint name="elbow1_joint" type="revolute">
-    <origin rpy="1.44504380352115E-15 1.11628850952447E-06 -9.93431159466724E-15" xyz="0 -0.000251155668932789 0.266305434894181"/>
+    <origin rpy="1.44504380352115E-15 1.11628850952447E-06 -9.93431159466724E-15" xyz="0 -0.000251155668931501 0.266305434894181"/>
     <parent link="shoulder_link"/>
     <child link="elbow1_link"/>
@@ -205,5 +205,5 @@
   <link name="elbow2_link">
     <inertial>
-      <origin rpy="0 0 0" xyz="-2.29085121194481E-05 -0.000512185919169572 0.0885118786028204"/>
+      <origin rpy="0 0 0" xyz="0.000512284668490459 -2.29084833272284E-05 0.0885118785637893"/>
       <mass value="1.12138857800426"/>
       <inertia ixx="0.0011156254663426" ixy="3.04261287700186E-07" ixz="-1.22468079415109E-06" iyy="0.0110437302875007" iyz="-7.91547787630536E-05" izz="0.000331598270284794"/>
@@ -228,5 +228,5 @@
   </link>
   <joint name="elbow2_joint" type="revolute">
-    <origin rpy="-4.51048856041191E-16 3.35869632765754E-16 0" xyz="0 0 0.223999999999899"/>
+    <origin rpy="-4.51048856041191E-16 3.35869632765754E-16 0" xyz="0 0 0.22399999999847"/>
     <parent link="elbow1_link"/>
     <child link="elbow2_link"/>
@@ -236,5 +236,5 @@
   <link name="wrist_link">
     <inertial>
-      <origin rpy="0 0 0" xyz="0 0 0"/>
+      <origin rpy="0 0 0" xyz="0.0303673809619356 4.00707611352118E-10 0.000140374211043737"/>
       <mass value="0.717337417215465"/>
       <inertia ixx="0.000486392340366094" ixy="4.20757000035677E-12" ixz="-3.91843889020299E-06" iyy="0.000211170064630335" iyz="2.79335159568522E-12" izz="0.000437528795624211"/>
@@ -259,5 +259,5 @@
   </link>
   <joint name="wrist_joint" type="revolute">
-    <origin rpy="0 0 0" xyz="0.0137 0 0.244749999999997"/>
+    <origin rpy="0 0 0" xyz="0.0131002732116043 0 0.244749985376465"/>
     <parent link="elbow2_link"/>
     <child link="wrist_link"/>

Commit message: moveit demo update

File: robotican_arm/models/arm.xacro (robot description, xacro)
@@ -261,5 +261,5 @@
   <link name="gripper_link"/>
   <joint name="gripper_joint" type="fixed">
-  <origin xyz="0 0 0.06" rpy="0 1.570796327 0"/>
+  <origin xyz="0 0 0.06" rpy="0 -1.570796327 0"/>
   <parent link="wrist_link"/>
   <child link="gripper_link"/>

File: robotican_komodo/description/models/komodo.xacro (robot description, xacro)
@@ -5,7 +5,4 @@
 	<xacro:include filename="$(find robotican_komodo)/description/models/komodo_base.xacro" />
 	<!--      END          -->
-	<!--    ARM     -->
-	<!-- <xacro:include filename="$(find robotican_manipulator_h)/models/manipulator_h.xacro" /> -->
-	<!--      END          -->
   <!--    TORSO     -->
   <xacro:include filename="$(find robotican_komodo)/description/models/komodo_torso.xacro" />

File: robotican_komodo/description/models/komodo_torso.xacro (robot description, xacro)
@@ -264,5 +264,5 @@
   <link name="gripper_link"/>
   <joint name="gripper_joint" type="fixed">
-  <origin xyz="0 0 0.06" rpy="0 1.570796327 0"/>
+  <origin xyz="0 0 0.06" rpy="0 -1.570796327 0"/>
   <parent link="wrist_link"/>
   <child link="gripper_link"/>
